Commit message: Resolve "Kamery w modelu urdf Siriusa"

File: src/sirius_description/urdf/materials.urdf.xacro (robot description, xacro)
@@ -14,4 +14,7 @@
   <material name="gray">
     <color rgba=".796 .824 .937 1" />
+  </material>
+  <material name="black">
+    <color rgba="0 0 0 1" />
   </material>
   <xacro:macro name="gold">
@@ -55,3 +58,11 @@
     </material>
   </xacro:macro>
+  <xacro:macro name="black">
+    <material>
+      <ambient>0 0 0 1</ambient>
+      <diffuse>0 0 0 1</diffuse>
+      <specular>0 0 0 1</specular>
+      <emissive>0.0 0.0 0.0 0.0</emissive>
+    </material>
+  </xacro:macro>
 </robot>

File: src/sirius_description/urdf/sirius_2.urdf.xacro (robot description, xacro)
@@ -5,7 +5,10 @@
   <xacro:property name="collisions" value="${xacro.load_yaml('sirius_2/sirius_2_collisions.yaml')}" />
   <xacro:property name="inertial" value="${xacro.load_yaml('sirius_2/sirius_2_inertial.yaml')}" />
+  <xacro:property name="cameras" value="${xacro.load_yaml('cameras/cameras.yaml')}" />
+  <xacro:property name="cameras_inertial" value="${xacro.load_yaml('cameras/cameras_inertial.yaml')}" />
   <xacro:include filename="materials.urdf.xacro" />
   <xacro:include filename="sirius_2/indicator_light.urdf.xacro" />
   <xacro:include filename="sirius_2/platform.urdf.xacro" />
+  <xacro:include filename="cameras/hp_4310.urdf.xacro" />
   <xacro:macro name="drive_system" params="reflect:=false prefix:='' params:=^ direction:=1">
     <xacro:include filename="sirius_2/suspension.urdf.xacro" />
@@ -50,4 +53,10 @@
     <xacro:blue_t/>
   </xacro:indicator_light>
+  <xacro:hp_4310 prefix="left_side" material="black">
+    <xacro:black/>
+  </xacro:hp_4310>
+  <xacro:hp_4310 prefix="right_side" material="black">
+    <xacro:black/>
+  </xacro:hp_4310>
   <xacro:drive_system prefix="right_front" />
   <xacro:drive_system reflect="true" prefix="right_back" direction="-1"/>
@@ -61,5 +70,5 @@
     <parent link="base_link"/>
     <child link="main_platform"/>
-    <origin xyz="0 0 ${params['wheel_radius'] + params['suspension_height'] - params['suspension_z']}" rpy="0 0 ${pi}"/>
+    <origin xyz="0 0 ${params['wheel_radius'] + params['suspension_height'] - params['suspension_z']}" rpy="0 0 0"/>
     <axis xyz="0 0 1"/>
   </joint>
@@ -94,8 +103,18 @@
     <origin xyz="${params['blue_indicator_light_xyz']}" rpy="0 0 ${pi}"/>
   </joint>
+  <joint name="base_to_left_side_camera" type="fixed">
+    <parent link="main_platform"/>
+    <child link="left_side_camera"/>
+    <origin xyz="${params['left_side_camera_xyz']}" rpy="${params['left_side_camera_rpy']}"/>
+  </joint>
+  <joint name="base_to_right_side_camera" type="fixed">
+    <parent link="main_platform"/>
+    <child link="right_side_camera"/>
+    <origin xyz="${params['right_side_camera_xyz']}" rpy="${params['right_side_camera_rpy']}"/>
+  </joint>
   <gazebo>
-  <plugin name="gazebo_ros_control" filename="libgazebo_ros_control.so">
-    <robotNamespace>/</robotNamespace>
-  </plugin>
+    <plugin name="gazebo_ros_control" filename="libgazebo_ros_control.so">
+      <robotNamespace>/</robotNamespace>
+    </plugin>
   </gazebo>
 </robot>
