Commit message: remove zed camera

File: src/sirius_description/urdf/sirius_2.urdf.xacro (robot description, xacro)
@@ -11,5 +11,4 @@
   <xacro:include filename="sirius_2/platform.urdf.xacro" />
   <xacro:include filename="cameras/hp_4310.urdf.xacro" />
-  <xacro:include filename="cameras/zed2i.urdf.xacro" />
   <xacro:include filename="cameras/oak-d-w.urdf.xacro" />
   <xacro:property name="link_prefix" value=""/>
@@ -64,6 +63,5 @@
     <xacro:black/>
   </xacro:hp_4310>
-  <xacro:zed2i prefix="front"/>
-  <xacro:oak-d-w prefix="back"/>
+  <xacro:oak-d-w prefix="front"/>
   <xacro:drive_system prefix="right_front" />
   <xacro:drive_system reflect="true" prefix="right_back" direction="-1"/>
@@ -125,9 +123,4 @@
     <origin xyz="${params['front_camera_xyz']}" rpy="${params['front_camera_rpy']}"/>
   </joint>
-  <joint name="base_to_back_camera" type="fixed">
-    <parent link="main_platform"/>
-    <child link="back_camera_center"/>
-    <origin xyz="${params['back_camera_xyz']}" rpy="${params['back_camera_rpy']}"/>
-  </joint>
   <gazebo>
     <plugin name="gazebo_ros_control" filename="libgazebo_ros_control.so">

Commit message: WIP: GPS gazebo plugin

File: src/sirius_description/urdf/sirius_2.urdf.xacro (robot description, xacro)
@@ -18,4 +18,5 @@
   <xacro:include filename="materials.urdf.xacro" />
   <xacro:include filename="sirius_2/indicator_light.urdf.xacro" />
+  <xacro:include filename="sirius_2/gnss.urdf.xacro" />
   <xacro:include filename="sirius_2/platform.urdf.xacro" />
   <xacro:include filename="cameras/hp_4310.urdf.xacro" />
@@ -66,4 +67,7 @@
     <xacro:blue_t/>
   </xacro:indicator_light>
+  <xacro:gnss material="light_gray">
+    <xacro:light_gray/>
+  </xacro:gnss>
   <xacro:hp_4310 prefix="front_mast" material="black">
     <xacro:black/>
@@ -117,4 +121,9 @@
     <origin xyz="${params['blue_indicator_light_xyz']}" rpy="0 0 ${pi}"/>
   </joint>
+  <joint name="base_to_gnss" type="fixed">
+    <parent link="base_link"/>
+    <child link="gnss"/>
+    <origin xyz="${params['gnss_xyz']}" rpy="0 0 0"/>
+  </joint>
   <joint name="base_to_front_mast_camera" type="fixed">
     <parent link="main_platform"/>
