Commit message: Resolve "Model urdf Siriusa 2"

File: src/sirius_description/urdf/manipulator.urdf.xacro (robot description, xacro)
@@ -10,9 +10,9 @@
   <xacro:property name="tool_length" value="0.011" />
   <xacro:property name="base_size_x" value="0.2" />
-  <link name="base">
+  <link name="base_link">
     <visual>
       <origin xyz="0 0 0" rpy="0 0 0" />
       <geometry>
-        <mesh filename="package://${package}/meshes/base.stl" scale="0.001 0.001 0.001"/>
+        <mesh filename="package://${package}/meshes/manipulator/base.stl" scale="0.001 0.001 0.001"/>
       </geometry>
       <material name="yellow">
@@ -31,5 +31,5 @@
       <origin xyz="0 0 0" rpy="0 0 0" />
       <geometry>
-        <mesh filename="package://${package}/meshes/cyl.stl" scale="0.001 0.001 0.001"/>
+        <mesh filename="package://${package}/meshes/manipulator/cyl.stl" scale="0.001 0.001 0.001"/>
       </geometry>
       <material name="grey">
@@ -45,5 +45,5 @@
   </link>
   <joint name="base_cyl" type="continuous">
-    <parent link="base"/>
+    <parent link="base_link"/>
     <child link="cylinder"/>
     <origin xyz="0 0 ${base_length}"/>
@@ -54,5 +54,5 @@
       <origin xyz="0 0 0" rpy="0 0 0" />
       <geometry>
-        <mesh filename="package://${package}/meshes/arm1.stl" scale="0.001 0.001 0.001"/>
+        <mesh filename="package://${package}/meshes/manipulator/arm1.stl" scale="0.001 0.001 0.001"/>
       </geometry>
       <material name="green">
@@ -82,5 +82,5 @@
       <origin xyz="0 0 0" rpy="0 0 0" />
       <geometry>
-        <mesh filename="package://${package}/meshes/arm2.stl" scale="0.001 0.001 0.001"/>
+        <mesh filename="package://${package}/meshes/manipulator/arm2.stl" scale="0.001 0.001 0.001"/>
       </geometry>
       <material name="blue">
@@ -110,5 +110,5 @@
       <origin xyz="0 0 0" rpy="0 0 0" />
       <geometry>
-        <mesh filename="package://${package}/meshes/arm3.stl" scale="0.001 0.001 0.001"/>
+        <mesh filename="package://${package}/meshes/manipulator/arm3.stl" scale="0.001 0.001 0.001"/>
       </geometry>
       <material name="red">
@@ -138,5 +138,5 @@
       <origin xyz="0 0 0" rpy="0 0 0" />
       <geometry>
-        <mesh filename="package://${package}/meshes/tool.stl" scale="0.001 0.001 0.001"/>
+        <mesh filename="package://${package}/meshes/manipulator/tool.stl" scale="0.001 0.001 0.001"/>
       </geometry>
       <material name="grey">

Commit message: Fix urdf root link

File: src/sirius_description/urdf/manipulator.urdf.xacro (robot description, xacro)
@@ -11,4 +11,12 @@
   <xacro:property name="tool_length" value="0.011" />
   <xacro:property name="base_size_x" value="0.2" />
+  <link name="root_link">
+  </link>
+  <joint name="root_base" type="fixed">
+    <parent link="root_link"/>
+    <child link="base_link"/>
+    <origin xyz="0 0 0"/>
+    <axis xyz="0 0 0"/>
+  </joint>
   <link name="base_link">
     <visual>

Commit message: Demo version of controllers, materials in gazebo

File: src/sirius_description/urdf/manipulator.urdf.xacro (robot description, xacro)
@@ -3,4 +3,5 @@
   <xacro:property name="package" value="sirius_description" />
   <xacro:property name="inertial" value="${xacro.load_yaml('manipulator_inertial.yaml')}" />
+  <xacro:include filename="materials.urdf.xacro" />
   <xacro:property name="base_length" value="0.006" />
   <xacro:property name="cyl_length" value="0.0655" />
@@ -16,6 +17,4 @@
     <parent link="root_link"/>
     <child link="base_link"/>
-    <origin xyz="0 0 0"/>
-    <axis xyz="0 0 0"/>
   </joint>
   <link name="base_link">
@@ -40,4 +39,9 @@
     </collision>
   </link>
+  <gazebo reference="base_link">
+      <material>
+        Gazebo/Yellow
+      </material>
+  </gazebo>
   <link name="cylinder">
     <visual>
@@ -61,4 +65,9 @@
     </collision>
   </link>
+  <gazebo reference="cylinder">
+      <material>
+        Gazebo/Grey
+      </material>
+  </gazebo>
   <joint name="base_cyl" type="continuous">
     <parent link="base_link"/>
@@ -67,4 +76,14 @@
     <axis xyz="0 0 1"/>
   </joint>
+  <transmission name="trans_base_cyl">
+    <type>transmission_interface/SimpleTransmission</type>
+    <joint name="base_cyl">
+        <hardwareInterface>hardware_interface/EffortJointInterface</hardwareInterface>
+    </joint>
+    <actuator name="motor_base_cyl">
+        <hardwareInterface>hardware_interface/EffortJointInterface</hardwareInterface>
+        <mechanicalReduction>1</mechanicalReduction>
+    </actuator>
+  </transmission>
   <link name="arm1">
     <visual>
@@ -88,4 +107,9 @@
     </collision>
   </link>
+  <gazebo reference="arm1">
+      <material>
+        Gazebo/Green
+      </material>
+  </gazebo>
   <joint name="cyl_arm1" type="revolute">
     <parent link="cylinder"/>
@@ -99,4 +123,14 @@
       velocity="0" />
   </joint>
+  <transmission name="trans_cyl_arm1">
+    <type>transmission_interface/SimpleTransmission</type>
+    <joint name="cyl_arm1">
+        <hardwareInterface>hardware_interface/EffortJointInterface</hardwareInterface>
+    </joint>
+    <actuator name="motor_cyl_arm1">
+        <hardwareInterface>hardware_interface/EffortJointInterface</hardwareInterface>
+        <mechanicalReduction>1</mechanicalReduction>
+    </actuator>
+  </transmission>
   <link name="arm2">
     <visual>
@@ -120,4 +154,9 @@
     </collision>
   </link>
+  <gazebo reference="arm2">
+      <material>
+        Gazebo/Blue
+      </material>
+  </gazebo>
   <joint name="arm1_arm2" type="revolute">
     <parent link="arm1"/>
@@ -131,4 +170,14 @@
       velocity="0" />
   </joint>
+  <transmission name="trans_arm1_arm2">
+    <type>transmission_interface/SimpleTransmission</type>
+    <joint name="arm1_arm2">
+        <hardwareInterface>hardware_interface/EffortJointInterface</hardwareInterface>
+    </joint>
+    <actuator name="motor_arm1_arm2">
+        <hardwareInterface>hardware_interface/EffortJointInterface</hardwareInterface>
+        <mechanicalReduction>1</mechanicalReduction>
+    </actuator>
+  </transmission>
   <link name="arm3">
     <visual>
@@ -152,4 +201,9 @@
     </collision>
   </link>
+  <gazebo reference="arm3">
+      <material>
+        Gazebo/Red
+      </material>
+  </gazebo>
   <joint name="arm2_arm3" type="revolute">
     <parent link="arm2"/>
@@ -163,4 +217,14 @@
       velocity="0" />
   </joint>
+  <transmission name="trans_arm2_arm3">
+    <type>transmission_interface/SimpleTransmission</type>
+    <joint name="arm2_arm3">
+        <hardwareInterface>hardware_interface/EffortJointInterface</hardwareInterface>
+    </joint>
+    <actuator name="motor_arm2_arm3">
+        <hardwareInterface>hardware_interface/EffortJointInterface</hardwareInterface>
+        <mechanicalReduction>1</mechanicalReduction>
+    </actuator>
+  </transmission>
   <link name="tool">
     <visual>
@@ -183,4 +247,9 @@
     </collision>
   </link>
+  <gazebo reference="tool">
+      <material>
+        Gazebo/Grey
+      </material>
+  </gazebo>
   <joint name="arm3_tool" type="continuous">
     <parent link="arm3"/>
@@ -189,4 +258,14 @@
     <axis xyz="0 0 1"/>
   </joint>
+  <transmission name="trans_arm3_tool">
+    <type>transmission_interface/SimpleTransmission</type>
+    <joint name="arm3_tool">
+        <hardwareInterface>hardware_interface/EffortJointInterface</hardwareInterface>
+    </joint>
+    <actuator name="motor_arm3_tool">
+        <hardwareInterface>hardware_interface/EffortJointInterface</hardwareInterface>
+        <mechanicalReduction>1</mechanicalReduction>
+    </actuator>
+  </transmission>
   <link name="fake">
   </link>
@@ -199,5 +278,6 @@
   <gazebo>
     <plugin name="gazebo_ros_control" filename="libgazebo_ros_control.so">
-      <robotNamespace>/</robotNamespace>
+      <robotNamespace>manipulator</robotNamespace>
+      <robotSimType>gazebo_ros_control/DefaultRobotHWSim</robotSimType>
     </plugin>
   </gazebo>

File: src/sirius_description/urdf/materials.urdf.xacro (robot description, xacro)
@@ -20,4 +20,7 @@
   <material name="black">
     <color rgba="0 0 0 1" />
+  </material>
+  <material name="green">
+    <color rgba="0 1 0 1" />
   </material>
   <xacro:macro name="gold">

Commit message: Add service for toggling between cartesian and jointspace modes

File: src/sirius_description/urdf/manipulator.urdf.xacro (robot description, xacro)
@@ -24,6 +24,6 @@
         <mesh filename="package://${package}/meshes/manipulator/base.stl" scale="0.001 0.001 0.001"/>
       </geometry>
-      <material name="yellow">
-        <color rgba=".5 .5 0 1" />
+      <material name="grey">
+        <color rgba=".5 .5 .5 1" />
       </material>
     </visual>
@@ -52,5 +52,4 @@
       </geometry>
       <material name="grey">
-        <color rgba=".5 .5 .5 1" />
       </material>
     </visual>
@@ -93,6 +92,6 @@
         <mesh filename="package://${package}/meshes/manipulator/arm1.stl" scale="0.001 0.001 0.001"/>
       </geometry>
-      <material name="green">
-        <color rgba="0 1 0 1" />
+      <material name="white">
+        <color rgba="1 1 1 1" />
       </material>
     </visual>
@@ -140,6 +139,5 @@
         <mesh filename="package://${package}/meshes/manipulator/arm2.stl" scale="0.001 0.001 0.001"/>
       </geometry>
-      <material name="blue">
-        <color rgba="0 0 1 1" />
+      <material name="grey">
       </material>
     </visual>
@@ -187,6 +185,5 @@
         <mesh filename="package://${package}/meshes/manipulator/arm3.stl" scale="0.001 0.001 0.001"/>
       </geometry>
-      <material name="red">
-        <color rgba="1 0 0 1" />
+      <material name="white">
       </material>
     </visual>

Commit message: wip: Add offsets to urdf

File: src/sirius_description/urdf/manipulator.urdf.xacro (robot description, xacro)
@@ -12,4 +12,7 @@
   <xacro:property name="tool_length" value="0.011" />
   <xacro:property name="base_size_x" value="0.2" />
+  <xacro:property name="arm1_home_angle" value="-0.7853981633974483"/>
+  <xacro:property name="arm2_home_angle" value="2.356194490192345"/>
+  <xacro:property name="arm3_home_angle" value="0.7853981633974483"/>
   <link name="root_link">
   </link>
@@ -115,9 +118,9 @@
     <parent link="cylinder"/>
     <child link="arm1"/>
-    <origin xyz="0 0 ${cyl_length}"/>
+    <origin xyz="0 0 ${cyl_length}" rpy="0 ${arm1_home_angle} 0"/>
     <axis xyz="0 1 0"/>
     <limit
-      lower="-1.45"
-      upper="0.79"
+      lower="${-1.45 - arm1_home_angle}"
+      upper="${1.45 - arm1_home_angle}"
       effort="10"
       velocity="5" />
@@ -161,9 +164,9 @@
     <parent link="arm1"/>
     <child link="arm2"/>
-    <origin xyz="0 0 ${arm1_length}"/>
+    <origin xyz="0 0 ${arm1_length}" rpy="0 ${arm2_home_angle} 0"/>
     <axis xyz="0 1 0"/>
     <limit
-      lower="0.0"
-      upper="2.36"
+      lower="-1.6"
+      upper="0.0"
       effort="100"
       velocity="50" />
@@ -207,9 +210,9 @@
     <parent link="arm2"/>
     <child link="arm3"/>
-    <origin xyz="0 0 ${arm2_length - arm2_lever}"/>
+    <origin xyz="0 0 ${arm2_length - arm2_lever}" rpy="0 ${arm3_home_angle} 0"/>
     <axis xyz="0 1 0"/>
     <limit
-      lower="-1.45"
-      upper="0.79"
+      lower="-1.57"
+      upper="0"
       effort="100"
       velocity="50" />

Commit message: Fix angles in urdf

File: src/sirius_description/urdf/manipulator.urdf.xacro (robot description, xacro)
@@ -14,5 +14,5 @@
   <xacro:property name="arm1_home_angle" value="-0.7853981633974483"/>
   <xacro:property name="arm2_home_angle" value="2.356194490192345"/>
-  <xacro:property name="arm3_home_angle" value="0.7853981633974483"/>
+  <xacro:property name="arm3_home_angle" value="0.5"/>
   <link name="root_link">
   </link>

Commit message: add gripper model

File: src/sirius_description/urdf/manipulator.urdf.xacro (robot description, xacro)
@@ -3,5 +3,5 @@
   <xacro:property name="package" value="sirius_description" />
   <xacro:property name="inertial" value="${xacro.load_yaml('manipulator_inertial.yaml')}" />
-  <xacro:include filename="materials.urdf.xacro" />
+  <!-- <xacro:include filename="materials.urdf.xacro" /> -->
   <xacro:property name="base_length" value="0.006" />
   <xacro:property name="cyl_length" value="0.0655" />
@@ -269,12 +269,10 @@
     </actuator>
   </transmission>
-  <link name="fake">
-  </link>
-  <joint name="tool_fake" type="continuous">
-    <parent link="tool"/>
-    <child link="fake"/>
-    <origin xyz="0 0 ${tool_length}"/>
-    <axis xyz="1 0 0"/>
-  </joint>
+  <joint name="tool_gripper" type="fixed">
+    <parent link="tool" />
+    <child link="gripper" />
+    <origin xyz="0 0 ${tool_length}" />
+  </joint>
+  <xacro:include filename="gripper.urdf.xacro"/>
   <gazebo>
     <plugin name="gazebo_ros_control" filename="libgazebo_ros_control.so">
