Commit message: update and optimize manip description

File: src/sirius_description/urdf/manipulator.urdf.xacro (robot description, xacro)
@@ -2,10 +2,9 @@
 <robot xmlns:xacro="http://www.ros.org/wiki/xacro" name="manipulator">
   <xacro:property name="package" value="sirius_description" />
-  <xacro:property name="inertial" value="${xacro.load_yaml('manipulator_inertial.yaml')}" />
+  <xacro:property name="inertial"
+    value="${xacro.load_yaml('manipulator/manipulator_inertial.yaml')}" />
   <xacro:include filename="materials.urdf.xacro" />
+  <xacro:include filename="manipulator/gripper.urdf.xacro" />
   <xacro:arg name="enable_gripper" default="True" />
-  <xacro:if value="${$(arg enable_gripper)}">
-    <xacro:include filename="gripper.urdf.xacro" />
-  </xacro:if>
   <xacro:property name="base_length" value="0.006" />
   <xacro:property name="cyl_length" value="0.0655" />
@@ -19,6 +18,5 @@
   <xacro:property name="arm2_home_angle" value="2.356194490192345" />
   <xacro:property name="arm3_home_angle" value="0.5" />
-  <link name="root_link">
-  </link>
+  <link name="root_link" />
   <joint name="root_base" type="fixed">
     <parent link="root_link" />
@@ -35,10 +33,5 @@
       </material>
     </visual>
-    <inertial>
-      <mass value="${inertial['base_mass']}" />
-      <inertia ixx="${inertial['base_inertia']['ixx']}" ixy="${inertial['base_inertia']['ixy']}"
-        ixz="${inertial['base_inertia']['ixz']}" iyy="${inertial['base_inertia']['iyy']}"
-        iyz="${inertial['base_inertia']['iyz']}" izz="${inertial['base_inertia']['izz']}" />
-    </inertial>
+    <xacro:inertial inertial="${inertial['base']}"/>
     <collision>
       <origin xyz="0 0 ${base_length / 2}" rpy="0 0 0" />
@@ -50,31 +43,4 @@
   <gazebo reference="base_link">
     <kinematic>true</kinematic>
-    <material>
-      Gazebo/Grey
-    </material>
-  </gazebo>
-  <link name="cylinder">
-    <visual>
-      <origin xyz="0 0 0" rpy="0 0 0" />
-      <geometry>
-        <mesh filename="package://${package}/meshes/manipulator/cyl.stl" scale="0.001 0.001 0.001" />
-      </geometry>
-      <material name="grey">
-      </material>
-    </visual>
-    <inertial>
-      <mass value="${inertial['cyl_mass']}" />
-      <inertia ixx="${inertial['cyl_inertia']['ixx']}" ixy="${inertial['cyl_inertia']['ixy']}"
-        ixz="${inertial['cyl_inertia']['ixz']}" iyy="${inertial['cyl_inertia']['iyy']}"
-        iyz="${inertial['cyl_inertia']['iyz']}" izz="${inertial['cyl_inertia']['izz']}" />
-    </inertial>
-    <collision>
-      <origin xyz="0 0 ${cyl_length/2}" rpy="0 0 0" />
-      <geometry>
-        <cylinder length="${cyl_length}" radius="0.06" />
-      </geometry>
-    </collision>
-  </link>
-  <gazebo reference="cylinder">
     <material>
       Gazebo/Grey
@@ -97,30 +63,24 @@
     </actuator>
   </transmission>
-  <link name="arm1">
-    <visual>
-      <origin xyz="0 0 0" rpy="0 0 0" />
-      <geometry>
-        <mesh filename="package://${package}/meshes/manipulator/arm1.stl" scale="0.001 0.001 0.001" />
-      </geometry>
-      <material name="white">
-        <color rgba="1 1 1 1" />
-      </material>
-    </visual>
-    <inertial>
-      <mass value="${inertial['arm1_mass']}" />
-      <inertia ixx="${inertial['arm1_inertia']['ixx']}" ixy="${inertial['arm1_inertia']['ixy']}"
-        ixz="${inertial['arm1_inertia']['ixz']}" iyy="${inertial['arm1_inertia']['iyy']}"
-        iyz="${inertial['arm1_inertia']['iyz']}" izz="${inertial['arm1_inertia']['izz']}" />
-    </inertial>
-    <collision>
-      <origin xyz="0 0 ${arm1_length/2}" rpy="0 0 0" />
-      <geometry>
-        <box size="0.07 0.07 ${arm1_length}" />
-      </geometry>
-    </collision>
-  </link>
-  <gazebo reference="arm1">
-    <material>
-      Gazebo/White
+  <link name="cylinder">
+    <visual>
+      <origin xyz="0 0 0" rpy="0 0 0" />
+      <geometry>
+        <mesh filename="package://${package}/meshes/manipulator/cyl.stl" scale="0.001 0.001 0.001" />
+      </geometry>
+      <material name="grey">
+      </material>
+    </visual>
+    <xacro:inertial inertial="${inertial['cyl']}"/>
+    <collision>
+      <origin xyz="0 0 ${cyl_length/2}" rpy="0 0 0" />
+      <geometry>
+        <cylinder length="${cyl_length}" radius="0.06" />
+      </geometry>
+    </collision>
+  </link>
+  <gazebo reference="cylinder">
+    <material>
+      Gazebo/Grey
     </material>
   </gazebo>
@@ -146,29 +106,25 @@
     </actuator>
   </transmission>
-  <link name="arm2">
-    <visual>
-      <origin xyz="0 0 0" rpy="0 0 0" />
-      <geometry>
-        <mesh filename="package://${package}/meshes/manipulator/arm2.stl" scale="0.001 0.001 0.001" />
-      </geometry>
-      <material name="grey">
-      </material>
-    </visual>
-    <inertial>
-      <mass value="${inertial['arm2_mass']}" />
-      <inertia ixx="${inertial['arm2_inertia']['ixx']}" ixy="${inertial['arm2_inertia']['ixy']}"
-        ixz="${inertial['arm2_inertia']['ixz']}" iyy="${inertial['arm2_inertia']['iyy']}"
-        iyz="${inertial['arm2_inertia']['iyz']}" izz="${inertial['arm2_inertia']['izz']}" />
-    </inertial>
-    <collision>
-      <origin xyz="0 0 ${arm2_length/2 - arm2_lever}" rpy="0 0 0" />
-      <geometry>
-        <box size="0.06 0.06 ${arm2_length}" />
-      </geometry>
-    </collision>
-  </link>
-  <gazebo reference="arm2">
-    <material>
-      Gazebo/Grey
+  <link name="arm1">
+    <visual>
+      <origin xyz="0 0 0" rpy="0 0 0" />
+      <geometry>
+        <mesh filename="package://${package}/meshes/manipulator/arm1.stl" scale="0.001 0.001 0.001" />
+      </geometry>
+      <material name="white">
+        <color rgba="1 1 1 1" />
+      </material>
+    </visual>
+    <xacro:inertial inertial="${inertial['arm1']}"/>
+    <collision>
+      <origin xyz="0 0 ${arm1_length/2}" rpy="0 0 0" />
+      <geometry>
+        <box size="0.07 0.07 ${arm1_length}" />
+      </geometry>
+    </collision>
+  </link>
+  <gazebo reference="arm1">
+    <material>
+      Gazebo/White
     </material>
   </gazebo>
@@ -194,29 +150,24 @@
     </actuator>
   </transmission>
-  <link name="arm3">
-    <visual>
-      <origin xyz="0 0 0" rpy="0 0 0" />
-      <geometry>
-        <mesh filename="package://${package}/meshes/manipulator/arm3.stl" scale="0.001 0.001 0.001" />
-      </geometry>
-      <material name="white">
-      </material>
-    </visual>
-    <inertial>
-      <mass value="${inertial['arm3_mass']}" />
-      <inertia ixx="${inertial['arm3_inertia']['ixx']}" ixy="${inertial['arm3_inertia']['ixy']}"
-        ixz="${inertial['arm3_inertia']['ixz']}" iyy="${inertial['arm3_inertia']['iyy']}"
-        iyz="${inertial['arm3_inertia']['iyz']}" izz="${inertial['arm3_inertia']['izz']}" />
-    </inertial>
-    <collision>
-      <origin xyz="0 0 ${arm3_length/2}" rpy="0 0 0" />
-      <geometry>
-        <box size="0.06 0.076 ${arm3_length}" />
-      </geometry>
-    </collision>
-  </link>
-  <gazebo reference="arm3">
-    <material>
-      Gazebo/White
+  <link name="arm2">
+    <visual>
+      <origin xyz="0 0 0" rpy="0 0 0" />
+      <geometry>
+        <mesh filename="package://${package}/meshes/manipulator/arm2.stl" scale="0.001 0.001 0.001" />
+      </geometry>
+      <material name="grey">
+      </material>
+    </visual>
+    <xacro:inertial inertial="${inertial['arm2']}"/>
+    <collision>
+      <origin xyz="0 0 ${arm2_length/2 - arm2_lever}" rpy="0 0 0" />
+      <geometry>
+        <box size="0.06 0.06 ${arm2_length}" />
+      </geometry>
+    </collision>
+  </link>
+  <gazebo reference="arm2">
+    <material>
+      Gazebo/Grey
     </material>
   </gazebo>
@@ -242,29 +193,24 @@
     </actuator>
   </transmission>
-  <link name="tool">
-    <visual>
-      <origin xyz="0 0 0" rpy="0 0 0" />
-      <geometry>
-        <mesh filename="package://${package}/meshes/manipulator/tool.stl" scale="0.001 0.001 0.001" />
-      </geometry>
-      <material name="grey">
-      </material>
-    </visual>
-    <inertial>
-      <mass value="${inertial['tool_mass']}" />
-      <inertia ixx="${inertial['tool_inertia']['ixx']}" ixy="${inertial['tool_inertia']['ixy']}"
-        ixz="${inertial['tool_inertia']['ixz']}" iyy="${inertial['tool_inertia']['iyy']}"
-        iyz="${inertial['tool_inertia']['iyz']}" izz="${inertial['tool_inertia']['izz']}" />
-    </inertial>
-    <collision>
-      <origin xyz="0 0 ${tool_length/2}" rpy="0 0 0" />
-      <geometry>
-        <cylinder length="${tool_length}" radius="0.03" />
-      </geometry>
-    </collision>
-  </link>
-  <gazebo reference="tool">
-    <material>
-      Gazebo/Grey
+  <link name="arm3">
+    <visual>
+      <origin xyz="0 0 0" rpy="0 0 0" />
+      <geometry>
+        <mesh filename="package://${package}/meshes/manipulator/arm3.stl" scale="0.001 0.001 0.001" />
+      </geometry>
+      <material name="white">
+      </material>
+    </visual>
+    <xacro:inertial inertial="${inertial['arm3']}"/>
+    <collision>
+      <origin xyz="0 0 ${arm3_length/2}" rpy="0 0 0" />
+      <geometry>
+        <box size="0.06 0.076 ${arm3_length}" />
+      </geometry>
+    </collision>
+  </link>
+  <gazebo reference="arm3">
+    <material>
+      Gazebo/White
     </material>
   </gazebo>
@@ -285,4 +231,26 @@
     </actuator>
   </transmission>
+  <link name="tool">
+    <visual>
+      <origin xyz="0 0 0" rpy="0 0 0" />
+      <geometry>
+        <mesh filename="package://${package}/meshes/manipulator/tool.stl" scale="0.001 0.001 0.001" />
+      </geometry>
+      <material name="grey">
+      </material>
+    </visual>
+    <xacro:inertial inertial="${inertial['tool']}"/>
+    <collision>
+      <origin xyz="0 0 ${tool_length/2}" rpy="0 0 0" />
+      <geometry>
+        <cylinder length="${tool_length}" radius="0.03" />
+      </geometry>
+    </collision>
+  </link>
+  <gazebo reference="tool">
+    <material>
+      Gazebo/Grey
+    </material>
+  </gazebo>
   <xacro:if value="${$(arg enable_gripper)}">
     <joint name="tool_gripper" type="fixed">
@@ -291,5 +259,5 @@
       <origin xyz="0 0 ${tool_length}" />
     </joint>
-    <xacro:gripper package="${package}" inertial="${inertial}" />
+    <xacro:gripper package="${package}" />
   </xacro:if>
   <gazebo>

File: src/sirius_description/urdf/manipulator/gripper.urdf.xacro (robot description, xacro)
@@ -1,8 +1,23 @@
 <?xml version="1.0" encoding="utf-8"?>
 <robot xmlns:xacro="http://www.ros.org/wiki/xacro">
-  <xacro:macro name="gripper" params="package inertial">
+  <xacro:macro name="inertial" params="inertial">
+    <inertial>
+      <mass value="${inertial['mass']}" />
+      <origin
+        xyz="${inertial['mass_center']['x']} ${inertial['mass_center']['y']} ${inertial['mass_center']['z']}"
+        rpy="0.0 0.0 0.0" />
+      <inertia ixx="${inertial['inertia']['ixx']}"
+        ixy="${inertial['inertia']['ixy']}"
+        ixz="${inertial['inertia']['ixz']}"
+        iyy="${inertial['inertia']['iyy']}"
+        iyz="${inertial['inertia']['iyz']}"
+        izz="${inertial['inertia']['izz']}" />
+    </inertial>
+  </xacro:macro>
+  <xacro:macro name="gripper" params="package">
+    <xacro:property name="inertial" value="${xacro.load_yaml('manipulator/gripper_inertial.yaml')}" />
+    <xacro:property name="base_length" value="0.05385" />
+    <xacro:property name="beam_distance" value="0.034" />
     <xacro:property name="beam_length" value="0.04" />
-    <xacro:property name="beam_distance" value="0.034" />
-    <xacro:property name="base_length" value="0.05385" />
     <link name="gripper">
       <visual>
@@ -15,13 +30,5 @@
         </material>
       </visual>
-      <inertial>
-        <mass value="${inertial['gripper_mass']/1000}" />
-        <inertia ixx="${inertial['gripper_inertia']['ixx']/1000}"
-          ixy="${inertial['gripper_inertia']['ixy']/1000}"
-          ixz="${inertial['gripper_inertia']['ixz']/1000}"
-          iyy="${inertial['gripper_inertia']['iyy']/1000}"
-          iyz="${inertial['gripper_inertia']['iyz']/1000}"
-          izz="${inertial['gripper_inertia']['izz']/1000}" />
-      </inertial>
+      <xacro:inertial inertial="${inertial['gripper']}" />
       <collision>
         <origin xyz="0.015 0 0.025" rpy="0 0 0" />
@@ -59,5 +66,5 @@
     <link name="left_beams">
       <visual>
-        <origin xyz="0 ${-beam_distance/2} ${-base_length}" rpy="${pi/2} ${pi/2} ${-pi/2}" />
+        <origin xyz="0 ${-beam_distance/2} ${-base_length}" rpy="${pi} ${pi/2} 0" />
         <geometry>
           <mesh filename="package://${package}/meshes/gripper/left_beams.stl"
@@ -67,8 +74,5 @@
         </material>
       </visual>
-      <inertial>
-        <mass value="0.001" />
-        <inertia ixx="0.0" ixy="0.0" ixz="0.0" iyy="0.0" iyz="0.0" izz="0.0" />
-      </inertial>
+      <xacro:inertial inertial="${inertial['left_beams']}" />
     </link>
     <gazebo reference="left_beams">
@@ -91,5 +95,5 @@
     <link name="right_beams">
       <visual>
-        <origin xyz="0 ${beam_distance/2} ${-base_length}" rpy="${pi/2} ${pi/2} ${-pi/2}" />
+        <origin xyz="0 ${beam_distance/2} ${-base_length}" rpy="${pi} ${pi/2} 0" />
         <geometry>
           <mesh filename="package://${package}/meshes/gripper/right_beams.stl"
@@ -99,8 +103,5 @@
         </material>
       </visual>
-      <inertial>
-        <mass value="0.001" />
-        <inertia ixx="0.0" ixy="0.0" ixz="0.0" iyy="0.0" iyz="0.0" izz="0.0" />
-      </inertial>
+      <xacro:inertial inertial="${inertial['right_beams']}" />
     </link>
     <gazebo reference="right_beams">
@@ -124,5 +125,5 @@
       <visual>
         <origin xyz="0 ${-beam_distance/2} ${-base_length-beam_length}"
-          rpy="${pi/2} ${pi/2} ${-pi/2}" />
+          rpy="${pi} ${pi/2} 0" />
         <geometry>
           <mesh filename="package://${package}/meshes/gripper/left_claw.stl"
@@ -132,8 +133,5 @@
         </material>
       </visual>
-      <inertial>
-        <mass value="0.001" />
-        <inertia ixx="0.0" ixy="0.0" ixz="0.0" iyy="0.0" iyz="0.0" izz="0.0" />
-      </inertial>
+      <xacro:inertial inertial="${inertial['left_claw']}" />
       <collision>
         <origin xyz="-0.005 0.003 0.058" rpy="0 0 0" />
@@ -163,5 +161,5 @@
       <visual>
         <origin xyz="0 ${beam_distance/2} ${-base_length-beam_length}"
-          rpy="${pi/2} ${pi/2} ${-pi/2}" />
+          rpy="${pi} ${pi/2} 0" />
         <geometry>
           <mesh filename="package://${package}/meshes/gripper/right_claw.stl"
@@ -171,8 +169,5 @@
         </material>
       </visual>
-      <inertial>
-        <mass value="0.001" />
-        <inertia ixx="0.0" ixy="0.0" ixz="0.0" iyy="0.0" iyz="0.0" izz="0.0" />
-      </inertial>
+      <xacro:inertial inertial="${inertial['right_claw']}" />
       <collision>
         <origin xyz="-0.005 -0.003 0.058" rpy="0 0 0" />
