Commit message: Change manip model to macro and add to sirius urdf

File: src/sirius_description/urdf/manipulator.urdf.xacro (robot description, xacro)
@@ -1,31 +1,16 @@
-<?xml version="1.0" encoding="utf-8"?>
-<robot xmlns:xacro="http://www.ros.org/wiki/xacro" name="manipulator">
-  <xacro:property name="package" value="sirius_description" />
-  <xacro:property name="inertial" value="${xacro.load_yaml('manipulator_inertial.yaml')}" />
-  <xacro:include filename="materials.urdf.xacro" />
-  <xacro:property name="base_length" value="0.006" />
-  <xacro:property name="cyl_length" value="0.0655" />
-  <xacro:property name="arm1_length" value="0.43498" />
-  <xacro:property name="arm2_length" value="0.5236" />
-  <xacro:property name="arm2_lever" value="0.0586" />
-  <xacro:property name="arm3_length" value="0.129" />
-  <xacro:property name="tool_length" value="0.011" />
-  <xacro:property name="base_size_x" value="0.2" />
-  <xacro:property name="arm1_home_angle" value="-0.7853981633974483"/>
-  <xacro:property name="arm2_home_angle" value="2.356194490192345"/>
-  <xacro:property name="arm3_home_angle" value="0.5"/>
-  <link name="root_link">
-  </link>
-  <joint name="root_base" type="fixed">
-    <parent link="root_link"/>
-    <child link="base_link"/>
-  </joint>
-  <link name="base_link">
-    <visual>
-      <origin xyz="0 0 0" rpy="0 0 0" />
+<robot xmlns:xacro="http://wiki.ros.org/xacro">
+<xacro:macro name="manipulator" params="prefix:='' package:=^">
+  <!-- Parse parameters -->
+  <xacro:property name="_prefix" value="${prefix + '_' if prefix else ''}"/>
+   <!-- Load model parameters -->
+  <xacro:property name="params" value="${xacro.load_yaml('manipulator.yaml')}" />
+  <!-- Load inertial parameters -->
+  <xacro:property name="inertial" value="${xacro.load_yaml('sirius_2/manipulator_inertial.yaml')}" />
+  <link name="${_prefix}base">
+    <visual>
       <geometry>
         <mesh filename="package://${package}/meshes/manipulator/base.stl" scale="0.001 0.001 0.001"/>
       </geometry>
-      <material name="grey">
+      <material name="${_prefix}grey">
         <color rgba=".5 .5 .5 1" />
       </material>
@@ -36,17 +21,16 @@
     </inertial>
     <collision>
-      <origin xyz="0 0 ${base_length / 2}" rpy="0 0 0" />
-      <geometry>
-        <box size="0.192 0.337 ${base_length}" />
-      </geometry>
-    </collision>
-  </link>
-  <gazebo reference="base_link">
-      <kinematic> true </kinematic>
-      <material>
-        Gazebo/Grey
-      </material>
-  </gazebo>
-  <link name="cylinder">
+      <origin xyz="0 0 ${params['base_length'] / 2}" rpy="0 0 0" />
+      <geometry>
+        <box size="0.192 0.337 ${params['base_length']}" />
+      </geometry>
+    </collision>
+  </link>
+  <gazebo reference="${_prefix}base">
+      <material>
+        Gazebo/Grey
+      </material>
+  </gazebo>
+  <link name="${_prefix}cylinder">
     <visual>
       <origin xyz="0 0 0" rpy="0 0 0" />
@@ -54,5 +38,5 @@
         <mesh filename="package://${package}/meshes/manipulator/cyl.stl" scale="0.001 0.001 0.001"/>
       </geometry>
-      <material name="grey">
+      <material name="${_prefix}grey">
       </material>
     </visual>
@@ -62,32 +46,33 @@
     </inertial>
     <collision>
-      <origin xyz="0 0 ${cyl_length/2}" rpy="0 0 0" />
-      <geometry>
-        <cylinder length="${cyl_length}" radius="0.06" />
-      </geometry>
-    </collision>
-  </link>
-  <gazebo reference="cylinder">
-      <material>
-        Gazebo/Grey
-      </material>
-  </gazebo>
-  <joint name="base_cyl" type="continuous">
-    <parent link="base_link"/>
-    <child link="cylinder"/>
-    <origin xyz="0 0 ${base_length}"/>
+      <origin xyz="0 0 ${params['cyl_length']/2}" rpy="0 0 0" />
+      <geometry>
+        <cylinder length="${params['cyl_length']}" radius="0.06" />
+      </geometry>
+    </collision>
+  </link>
+  <gazebo reference="${_prefix}cylinder">
+      <material>
+        Gazebo/Grey
+      </material>
+  </gazebo>
+  <joint name="${_prefix}base_cyl" type="continuous">
+    <parent link="${_prefix}base"/>
+    <child link="${_prefix}cylinder"/>
+    <origin xyz="0 0 ${params['base_length']}"/>
     <axis xyz="0 0 1"/>
-  </joint>
-  <transmission name="trans_base_cyl">
-    <type>transmission_interface/SimpleTransmission</type>
-    <joint name="base_cyl">
-        <hardwareInterface>hardware_interface/EffortJointInterface</hardwareInterface>
-    </joint>
-    <actuator name="motor_base_cyl">
-        <hardwareInterface>hardware_interface/EffortJointInterface</hardwareInterface>
+    <limit effort="100" velocity="5" />
+  </joint>
+  <transmission name="${_prefix}trans_base_cyl">
+    <type>transmission_interface/SimpleTransmission</type>
+    <joint name="${_prefix}base_cyl">
+        <hardwareInterface>hardware_interface/VelocityJointInterface</hardwareInterface>
+    </joint>
+    <actuator name="${_prefix}motor_base_cyl">
+        <hardwareInterface>hardware_interface/VelocityJointInterface</hardwareInterface>
         <mechanicalReduction>150</mechanicalReduction>
     </actuator>
   </transmission>
-  <link name="arm1">
+  <link name="${_prefix}arm1">
     <visual>
       <origin xyz="0 0 0" rpy="0 0 0" />
@@ -95,5 +80,5 @@
         <mesh filename="package://${package}/meshes/manipulator/arm1.stl" scale="0.001 0.001 0.001"/>
       </geometry>
-      <material name="white">
+      <material name="${_prefix}white">
         <color rgba="1 1 1 1" />
       </material>
@@ -104,37 +89,37 @@
     </inertial>
     <collision>
-      <origin xyz="0 0 ${arm1_length/2}" rpy="0 0 0" />
-      <geometry>
-        <box size="0.07 0.07 ${arm1_length}" />
-      </geometry>
-    </collision>
-  </link>
-  <gazebo reference="arm1">
+      <origin xyz="0 0 ${params['arm1_length']/2}" rpy="0 0 0" />
+      <geometry>
+        <box size="0.07 0.07 ${params['arm1_length']}" />
+      </geometry>
+    </collision>
+  </link>
+  <gazebo reference="${_prefix}arm1">
       <material>
         Gazebo/White
       </material>
   </gazebo>
-  <joint name="cyl_arm1" type="revolute">
-    <parent link="cylinder"/>
-    <child link="arm1"/>
-    <origin xyz="0 0 ${cyl_length}" rpy="0 ${arm1_home_angle} 0"/>
+  <joint name="${_prefix}cyl_arm1" type="revolute">
+    <parent link="${_prefix}cylinder"/>
+    <child link="${_prefix}arm1"/>
+    <origin xyz="0 0 ${params['cyl_length']}" rpy="0 ${params['arm1_home_angle']} 0"/>
     <axis xyz="0 1 0"/>
     <limit
-      lower="${-1.45 - arm1_home_angle}"
-      upper="${1.45 - arm1_home_angle}"
+      lower="${-1.45 - params['arm1_home_angle']}"
+      upper="${1.45 - params['arm1_home_angle']}"
       effort="10"
       velocity="5" />
   </joint>
-  <transmission name="trans_cyl_arm1">
-    <type>transmission_interface/SimpleTransmission</type>
-    <joint name="cyl_arm1">
-        <hardwareInterface>hardware_interface/EffortJointInterface</hardwareInterface>
-    </joint>
-    <actuator name="motor_cyl_arm1">
-        <hardwareInterface>hardware_interface/EffortJointInterface</hardwareInterface>
+  <transmission name="${_prefix}trans_cyl_arm1">
+    <type>transmission_interface/SimpleTransmission</type>
+    <joint name="${_prefix}cyl_arm1">
+        <hardwareInterface>hardware_interface/VelocityJointInterface</hardwareInterface>
+    </joint>
+    <actuator name="${_prefix}motor_cyl_arm1">
+        <hardwareInterface>hardware_interface/VelocityJointInterface</hardwareInterface>
         <mechanicalReduction>120</mechanicalReduction>
     </actuator>
   </transmission>
-  <link name="arm2">
+  <link name="${_prefix}arm2">
     <visual>
       <origin xyz="0 0 0" rpy="0 0 0" />
@@ -142,5 +127,5 @@
         <mesh filename="package://${package}/meshes/manipulator/arm2.stl" scale="0.001 0.001 0.001"/>
       </geometry>
-      <material name="grey">
+      <material name="${_prefix}grey">
       </material>
     </visual>
@@ -150,19 +135,19 @@
     </inertial>
     <collision>
-      <origin xyz="0 0 ${arm2_length/2 - arm2_lever}" rpy="0 0 0" />
-      <geometry>
-        <box size="0.06 0.06 ${arm2_length}" />
-      </geometry>
-    </collision>
-  </link>
-  <gazebo reference="arm2">
-      <material>
-        Gazebo/Grey
-      </material>
-  </gazebo>
-  <joint name="arm1_arm2" type="revolute">
-    <parent link="arm1"/>
-    <child link="arm2"/>
-    <origin xyz="0 0 ${arm1_length}" rpy="0 ${arm2_home_angle} 0"/>
+      <origin xyz="0 0 ${params['arm2_length']/2 - params['arm2_lever']}" rpy="0 0 0" />
+      <geometry>
+        <box size="0.06 0.06 ${params['arm2_length']}" />
+      </geometry>
+    </collision>
+  </link>
+  <gazebo reference="${_prefix}arm2">
+      <material>
+        Gazebo/Grey
+      </material>
+  </gazebo>
+  <joint name="${_prefix}arm1_arm2" type="revolute">
+    <parent link="${_prefix}arm1"/>
+    <child link="${_prefix}arm2"/>
+    <origin xyz="0 0 ${params['arm1_length']}" rpy="0 ${params['arm2_home_angle']} 0"/>
     <axis xyz="0 1 0"/>
     <limit
@@ -172,15 +157,15 @@
       velocity="50" />
   </joint>
-  <transmission name="trans_arm1_arm2">
-    <type>transmission_interface/SimpleTransmission</type>
-    <joint name="arm1_arm2">
-        <hardwareInterface>hardware_interface/EffortJointInterface</hardwareInterface>
-    </joint>
-    <actuator name="motor_arm1_arm2">
-        <hardwareInterface>hardware_interface/EffortJointInterface</hardwareInterface>
+  <transmission name="${_prefix}trans_arm1_arm2">
+    <type>transmission_interface/SimpleTransmission</type>
+    <joint name="${_prefix}arm1_arm2">
+        <hardwareInterface>hardware_interface/VelocityJointInterface</hardwareInterface>
+    </joint>
+    <actuator name="${_prefix}motor_arm1_arm2">
+        <hardwareInterface>hardware_interface/VelocityJointInterface</hardwareInterface>
         <mechanicalReduction>100</mechanicalReduction>
     </actuator>
   </transmission>
-  <link name="arm3">
+  <link name="${_prefix}arm3">
     <visual>
       <origin xyz="0 0 0" rpy="0 0 0" />
@@ -188,5 +173,5 @@
         <mesh filename="package://${package}/meshes/manipulator/arm3.stl" scale="0.001 0.001 0.001"/>
       </geometry>
-      <material name="white">
+      <material name="${_prefix}white">
       </material>
     </visual>
@@ -196,19 +181,19 @@
     </inertial>
     <collision>
-      <origin xyz="0 0 ${arm3_length/2}" rpy="0 0 0" />
-      <geometry>
-        <box size="0.06 0.076 ${arm3_length}" />
-      </geometry>
-    </collision>
-  </link>
-  <gazebo reference="arm3">
+      <origin xyz="0 0 ${params['arm3_length']/2}" rpy="0 0 0" />
+      <geometry>
+        <box size="0.06 0.076 ${params['arm3_length']}" />
+      </geometry>
+    </collision>
+  </link>
+  <gazebo reference="${_prefix}arm3">
       <material>
         Gazebo/White
       </material>
   </gazebo>
-  <joint name="arm2_arm3" type="revolute">
-    <parent link="arm2"/>
-    <child link="arm3"/>
-    <origin xyz="0 0 ${arm2_length - arm2_lever}" rpy="0 ${arm3_home_angle} 0"/>
+  <joint name="${_prefix}arm2_arm3" type="revolute">
+    <parent link="${_prefix}arm2"/>
+    <child link="${_prefix}arm3"/>
+    <origin xyz="0 0 ${params['arm2_length'] - params['arm2_lever']}" rpy="0 ${params['arm3_home_angle']} 0"/>
     <axis xyz="0 1 0"/>
     <limit
@@ -218,15 +203,15 @@
       velocity="50" />
   </joint>
-  <transmission name="trans_arm2_arm3">
-    <type>transmission_interface/SimpleTransmission</type>
-    <joint name="arm2_arm3">
-        <hardwareInterface>hardware_interface/EffortJointInterface</hardwareInterface>
-    </joint>
-    <actuator name="motor_arm2_arm3">
-        <hardwareInterface>hardware_interface/EffortJointInterface</hardwareInterface>
+  <transmission name="${_prefix}trans_arm2_arm3">
+    <type>transmission_interface/SimpleTransmission</type>
+    <joint name="${_prefix}arm2_arm3">
+        <hardwareInterface>hardware_interface/VelocityJointInterface</hardwareInterface>
+    </joint>
+    <actuator name="${_prefix}motor_arm2_arm3">
+        <hardwareInterface>hardware_interface/VelocityJointInterface</hardwareInterface>
         <mechanicalReduction>1</mechanicalReduction>
     </actuator>
   </transmission>
-  <link name="tool">
+  <link name="${_prefix}tool">
     <visual>
       <origin xyz="0 0 0" rpy="0 0 0" />
@@ -234,5 +219,5 @@
         <mesh filename="package://${package}/meshes/manipulator/tool.stl" scale="0.001 0.001 0.001"/>
       </geometry>
-      <material name="grey">
+      <material name="${_prefix}grey">
       </material>
     </visual>
@@ -242,37 +227,38 @@
     </inertial>
     <collision>
-      <origin xyz="0 0 ${tool_length/2}" rpy="0 0 0" />
-      <geometry>
-        <cylinder length="${tool_length}" radius="0.03" />
-      </geometry>
-    </collision>
-  </link>
-  <gazebo reference="tool">
-      <material>
-        Gazebo/Grey
-      </material>
-  </gazebo>
-  <joint name="arm3_tool" type="continuous">
-    <parent link="arm3"/>
-    <child link="tool"/>
-    <origin xyz="0 0 ${arm3_length}"/>
+      <origin xyz="0 0 ${params['tool_length']/2}" rpy="0 0 0" />
+      <geometry>
+        <cylinder length="${params['tool_length']}" radius="0.03" />
+      </geometry>
+    </collision>
+  </link>
+  <gazebo reference="${_prefix}tool">
+      <material>
+        Gazebo/Grey
+      </material>
+  </gazebo>
+  <joint name="${_prefix}arm3_tool" type="continuous">
+    <parent link="${_prefix}arm3"/>
+    <child link="${_prefix}tool"/>
+    <origin xyz="0 0 ${params['arm3_length']}"/>
     <axis xyz="0 0 1"/>
-  </joint>
-  <transmission name="trans_arm3_tool">
-    <type>transmission_interface/SimpleTransmission</type>
-    <joint name="arm3_tool">
-        <hardwareInterface>hardware_interface/EffortJointInterface</hardwareInterface>
-    </joint>
-    <actuator name="motor_arm3_tool">
-        <hardwareInterface>hardware_interface/EffortJointInterface</hardwareInterface>
+    <limit effort="20" velocity="5" />
+  </joint>
+  <transmission name="${_prefix}trans_arm3_tool">
+    <type>transmission_interface/SimpleTransmission</type>
+    <joint name="${_prefix}arm3_tool">
+        <hardwareInterface>hardware_interface/VelocityJointInterface</hardwareInterface>
+    </joint>
+    <actuator name="${_prefix}motor_arm3_tool">
+        <hardwareInterface>hardware_interface/VelocityJointInterface</hardwareInterface>
         <mechanicalReduction>1</mechanicalReduction>
     </actuator>
   </transmission>
-  <link name="fake">
-  </link>
-  <joint name="tool_fake" type="continuous">
-    <parent link="tool"/>
-    <child link="fake"/>
-    <origin xyz="0 0 ${tool_length}"/>
+  <link name="${_prefix}fake">
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
File: src/sirius_description/urdf/sirius_2.urdf.xacro (robot description, xacro)
@@ -7,4 +7,5 @@
   <xacro:arg name="elevation" default="0.0"/>
   <xacro:arg name="imu_frequency" default="200.0"/>
+  <xacro:arg name="manipulator" default="true"/>
   <xacro:arg name="joint_prefix" default=""/>
   <xacro:arg name="link_prefix" default=""/>
@@ -20,4 +21,5 @@
   <xacro:property name="elevation" value="$(arg elevation)" />
   <xacro:property name="imu_frequency" value="$(arg imu_frequency)" />
+  <xacro:property name="manipulator" value="$(arg manipulator)" />
   <xacro:property name="stereo_fps" value="$(arg stereo_fps)" />
   <xacro:property name="year" value="$(arg year)" />
@@ -37,4 +39,7 @@
   <xacro:include filename="sirius_2/indicator_light.urdf.xacro" />
   <xacro:include filename="sirius_2/platform.urdf.xacro" />
+  <xacro:if value="${manipulator}">
+    <xacro:include filename="manipulator.urdf.xacro" />
+  </xacro:if>
   <!-- Load sensors and cameras xacro -->
   <xacro:include filename="cameras/hp_4310.urdf.xacro" />
@@ -86,4 +91,7 @@
   <xacro:drive_system prefix="right_front"  flip_x="true"/>
   <xacro:indicator_light material="gray" />
+  <xacro:if value="${manipulator}">
+    <xacro:manipulator prefix="manipulator"/>
+  </xacro:if>
   <!-- Define sensors and cameras links -->
   <xacro:hp_4310 prefix="back_mast" material="black" />
@@ -115,4 +123,11 @@
                child="indicator_light"
                xyz="${params['indicator_light_xyz']}"/>
+  <xacro:if value="${manipulator}">
+    <xacro:joint name="base_to_manipulator"
+                 parent="platform"
+                 child="manipulator_base"
+                 xyz="${params['manipulator_xyz']}"
+                 rpy="${params['manipulator_rpy']}"/>
+  </xacro:if>
   <!-- Define sensors and cameras joints -->
   <xacro:joint name="base_to_front_mast_camera"
