Commit message: open_vins partial config

File: src/sirius_description/urdf/cameras/zed2i.urdf.xacro (robot description, xacro)
@@ -1,4 +1,5 @@
 <?xml version="1.0"?>
 <robot xmlns:xacro="http://ros.org/wiki/xacro">
+<!-- https://support.stereolabs.com/hc/en-us/articles/360007395634-What-is-the-camera-focal-length-and-field-of-view- -->
   <xacro:property name="baseline" value="0.12"/>
   <xacro:property name="optical_offset_x" value="-0.01" />
@@ -46,6 +47,5 @@
     </joint>
     <joint name="${prefix}_imu_frame_joint" type="fixed">
-      <!-- IMU frame offset copied from an actual ZED2 camera -->
-      <origin xyz="-0.002 -0.023 -0.002" rpy="0.0014025 -0.0000012 -0.0016915"/>
+      <origin xyz="-0.002 -0.023 -0.002" rpy="0 0 0"/>
       <parent link="${prefix}_left_camera_frame"/>
       <child link="${prefix}_imu_frame"/>
@@ -59,5 +59,5 @@
         <visualize>false</visualize>
         <camera name="/${prefix}_camera/left_raw">
-          <horizontal_fov>${110 * pi/180}</horizontal_fov>
+          <horizontal_fov>${104 * pi/180}</horizontal_fov>
           <image>
             <width>1280</width>
@@ -75,10 +75,9 @@
           </noise>
           <distortion>
-            <!-- Values copied from an actual ZED2 camera -->
-            <k1>-0.043693598</k1>
-            <k2>0.0146164996</k2>
-            <p1>-0.006573319</p1>
-            <p2>-0.000216900</p2>
-            <k3>0.000084328</k3>
+            <!-- Radial-tangential model -->
+            <k1>0</k1> <!-- k1 in kalibr-->
+            <k2>0</k2> <!-- k2 in kalibr-->
+            <p1>0</p1> <!-- r1 in kalibr-->
+            <p2>0</p2> <!-- r2 in kalibr-->
             <center>0.5 0.5</center>
           </distortion>
@@ -89,12 +88,11 @@
           <cameraInfoTopicName>camera_info</cameraInfoTopicName>
           <frameName>${prefix}_left_camera_optical_frame</frameName>
-          <distortionK1>-0.043693598</distortionK1>
-          <distortionK2>0.0146164996</distortionK2>
-          <distortionT1>-0.006573319</distortionT1>
-          <distortionT2>-0.000216900</distortionT2>
-          <distortionK3>0.000084328</distortionK3>
-          <CxPrime>648.5</CxPrime>
-          <Cx>648.5</Cx>
-          <Cy>366.8340148925781</Cy>
+          <distortionK1>0</distortionK1>
+          <distortionK2>0</distortionK2>
+          <distortionT1>0</distortionT1>
+          <distortionT2>0</distortionT2>
+          <CxPrime>640</CxPrime>
+          <Cx>640</Cx>
+          <Cy>360/Cy>
           <hackBaseline>0.0</hackBaseline>
         </plugin>
@@ -106,5 +104,5 @@
         <visualize>false</visualize>
         <camera name="/${prefix}_camera/depth">
-          <horizontal_fov>${110 * pi/180}</horizontal_fov>
+          <horizontal_fov>${104 * pi/180}</horizontal_fov>
           <image>
             <width>1280</width>
@@ -133,7 +131,7 @@
           <frameName>${prefix}_left_camera_optical_frame</frameName>
           <baseline>0.12</baseline>
-          <CxPrime>658.8206787109375</CxPrime>
-          <Cx>658.8206787109375</Cx>
-          <Cy>372.25787353515625</Cy>
+          <CxPrime>640</CxPrime>
+          <Cx>640</Cx>
+          <Cy>360/Cy>
           <hackBaseline>0.0</hackBaseline>
         </plugin>
@@ -148,5 +146,5 @@
         <visualize>false</visualize>
         <camera name="/${prefix}_camera/right_raw">
-          <horizontal_fov>${110 * pi/180}</horizontal_fov>
+          <horizontal_fov>${104 * pi/180}</horizontal_fov>
           <image>
             <width>1280</width>
@@ -164,9 +162,9 @@
           </noise>
           <distortion>
-            <k1>-0.040993299</k1>
-            <k2>0.009593590</k2>
-            <p1>-0.004429849</p1>
-            <p2>0.000192024</p2>
-            <k3>-0.000320880</k3>
+            <!-- Radial-tangential model -->
+            <k1>0</k1> <!-- k1 in kalibr-->
+            <k2>0</k2> <!-- k2 in kalibr-->
+            <p1>0</p1> <!-- r1 in kalibr-->
+            <p2>0</p2> <!-- r2 in kalibr-->
             <center>0.5 0.5</center>
           </distortion>
@@ -177,13 +175,12 @@
           <cameraInfoTopicName>camera_info</cameraInfoTopicName>
           <frameName>${prefix}_right_camera_optical_frame</frameName>
-          <distortionK1>-0.040993299</distortionK1>
-          <distortionK2>0.009593590</distortionK2>
-          <distortionT1>-0.004429849</distortionT1>
-          <distortionT2>0.000192024</distortionT2>
-          <distortionK3>-0.000320880</distortionK3>
-          <CxPrime>659.3049926757812</CxPrime>
-          <Cx>659.3049926757812</Cx>
-          <Cy>371.39849853515625</Cy>
-          <hackBaseline>0.12</hackBaseline>
+          <distortionK1>0</distortionK1>
+          <distortionK2>0</distortionK2>
+          <distortionT1>0</distortionT1>
+          <distortionT2>0</distortionT2>
+          <CxPrime>640</CxPrime>
+          <Cx>640</Cx>
+          <Cy>360/Cy>
+          <hackBaseline>0.0</hackBaseline>
         </plugin>
       </sensor>
@@ -194,5 +191,5 @@
         <visualize>false</visualize>
         <camera name="/${prefix}_camera/right">
-          <horizontal_fov>${110 * pi/180}</horizontal_fov>
+          <horizontal_fov>${104 * pi/180}</horizontal_fov>
           <image>
             <width>1280</width>
@@ -215,8 +212,8 @@
           <cameraInfoTopicName>camera_info</cameraInfoTopicName>
           <frameName>${prefix}_right_camera_optical_frame</frameName>
-          <CxPrime>658.8206787109375</CxPrime>
-          <Cx>658.8206787109375</Cx>
-          <Cy>372.25787353515625</Cy>
-          <hackBaseline>0.12</hackBaseline>
+          <CxPrime>640</CxPrime>
+          <Cx>640</Cx>
+          <Cy>360/Cy>
+          <hackBaseline>0</hackBaseline>
         </plugin>
       </sensor>
