Commit message: Resolve "Automatyczna aktualizacja ska_robotics.gitlab.io"

File: src/sirius_description/urdf/cameras/hp_4310.urdf.xacro (robot description, xacro)
@@ -1,4 +1,4 @@
 <robot xmlns:xacro="http://wiki.ros.org/xacro">
-<xacro:macro name="hp_4310" params="prefix material *gazebo_material package:=^ cameras:=^ cameras_inertial:=^">
+<xacro:macro name="hp_4310" params="prefix:=hp_4310 material *gazebo_material package:=^ cameras:=^ cameras_inertial:=^">
   <link name="${prefix}_camera">
     <visual>

File: src/sirius_description/urdf/materials.urdf.xacro (robot description, xacro)
@@ -14,4 +14,7 @@
   <material name="gray">
     <color rgba=".796 .824 .937 1" />
+  </material>
+  <material name="light_gray">
+        <color rgba="0.25 0.25 0.25 1"/>
   </material>
   <material name="black">
@@ -58,4 +61,12 @@
     </material>
   </xacro:macro>
+  <xacro:macro name="light_gray">
+    <material>
+      <ambient>0.25 0.25 0.25 1</ambient>
+      <diffuse>0.25 0.25 0.25 1</diffuse>
+      <specular>0.5 0.5 0.5 1</specular>
+      <emissive>0.0 0.0 0.0 0.0</emissive>
+    </material>
+  </xacro:macro>
   <xacro:macro name="black">
     <material>

File: src/sirius_description/urdf/sirius_2.urdf.xacro (robot description, xacro)
@@ -11,4 +11,9 @@
   <xacro:include filename="sirius_2/platform.urdf.xacro" />
   <xacro:include filename="cameras/hp_4310.urdf.xacro" />
+  <xacro:include filename="cameras/zed2i.urdf.xacro" />
+  <xacro:include filename="cameras/oak-d-w.urdf.xacro" />
+  <xacro:property name="link_prefix" value=""/>
+  <xacro:property name="robot_ns" value=""/>
+  <xacro:property name="joint_prefix" value=""/>
   <xacro:macro name="drive_system" params="reflect:=false prefix:='' params:=^ direction:=1">
     <xacro:include filename="sirius_2/suspension.urdf.xacro" />
@@ -53,10 +58,12 @@
     <xacro:blue_t/>
   </xacro:indicator_light>
-  <xacro:hp_4310 prefix="left_side" material="black">
+  <xacro:hp_4310 prefix="front_mast" material="black">
     <xacro:black/>
   </xacro:hp_4310>
-  <xacro:hp_4310 prefix="right_side" material="black">
+  <xacro:hp_4310 prefix="back_mast" material="black">
     <xacro:black/>
   </xacro:hp_4310>
+  <xacro:zed2i prefix="front"/>
+  <xacro:oak-d-w prefix="back"/>
   <xacro:drive_system prefix="right_front" />
   <xacro:drive_system reflect="true" prefix="right_back" direction="-1"/>
@@ -70,5 +77,5 @@
     <parent link="base_link"/>
     <child link="main_platform"/>
-    <origin xyz="0 0 ${params['wheel_radius'] + params['suspension_height'] - params['suspension_z']}" rpy="0 0 0"/>
+    <origin xyz="0 0 ${params['wheel_radius'] + params['suspension_height'] - params['suspension_z']}" rpy="0 0 ${pi}"/>
     <axis xyz="0 0 1"/>
   </joint>
@@ -103,13 +110,23 @@
     <origin xyz="${params['blue_indicator_light_xyz']}" rpy="0 0 ${pi}"/>
   </joint>
-  <joint name="base_to_left_side_camera" type="fixed">
+  <joint name="base_to_front_mast_camera" type="fixed">
     <parent link="main_platform"/>
-    <child link="left_side_camera"/>
-    <origin xyz="${params['left_side_camera_xyz']}" rpy="${params['left_side_camera_rpy']}"/>
+    <child link="front_mast_camera"/>
+    <origin xyz="${params['front_mast_camera_xyz']}" rpy="${params['front_mast_camera_rpy']}"/>
   </joint>
-  <joint name="base_to_right_side_camera" type="fixed">
+  <joint name="base_to_back_mast_camera" type="fixed">
     <parent link="main_platform"/>
-    <child link="right_side_camera"/>
-    <origin xyz="${params['right_side_camera_xyz']}" rpy="${params['right_side_camera_rpy']}"/>
+    <child link="back_mast_camera"/>
+    <origin xyz="${params['back_mast_camera_xyz']}" rpy="${params['back_mast_camera_rpy']}"/>
+  </joint>
+  <joint name="base_to_front_camera" type="fixed">
+    <parent link="main_platform"/>
+    <child link="front_camera_center"/>
+    <origin xyz="${params['front_camera_xyz']}" rpy="${params['front_camera_rpy']}"/>
+  </joint>
+  <joint name="base_to_back_camera" type="fixed">
+    <parent link="main_platform"/>
+    <child link="back_camera_center"/>
+    <origin xyz="${params['back_camera_xyz']}" rpy="${params['back_camera_rpy']}"/>
   </joint>
   <gazebo>

Commit message: simplify material parameters

File: src/sirius_description/urdf/cameras/hp_4310.urdf.xacro (robot description, xacro)
@@ -1,4 +1,4 @@
 <robot xmlns:xacro="http://wiki.ros.org/xacro">
-<xacro:macro name="hp_4310" params="prefix:=hp_4310 material *gazebo_material package:=^ cameras:=^ cameras_inertial:=^">
+<xacro:macro name="hp_4310" params="prefix:=hp_4310 material package:=^ cameras:=^ cameras_inertial:=^">
   <link name="${prefix}_camera">
     <visual>
@@ -22,5 +22,5 @@
   <gazebo reference="${prefix}_camera">
       <visual>
-        <xacro:insert_block name="gazebo_material" />
+        <xacro:element xacro:name="xacro:${material}" />
       </visual>
       <sensor type="camera" name="${prefix}_camera">

File: src/sirius_description/urdf/sirius_2.urdf.xacro (robot description, xacro)
@@ -57,11 +57,6 @@
     <xacro:include filename="sirius_2/suspension.urdf.xacro" />
     <xacro:include filename="sirius_2/wheel.urdf.xacro" />
-    <xacro:suspension prefix="${prefix}" material="dark_bronze" flip="${flip_y}">
-      <xacro:dark_bronze/>
-    </xacro:suspension>
-    <xacro:wheel prefix="${prefix}" material="dark_gray" material_rim="white" flip="${flip_x}">
-      <xacro:dark_gray/>
-      <xacro:white/>
-    </xacro:wheel>
+    <xacro:suspension prefix="${prefix}" material="dark_bronze" flip="${flip_y}" />
+    <xacro:wheel prefix="${prefix}" material="dark_gray" material_rim="white" flip="${flip_x}" />
     <xacro:joint  name="${prefix}_wheel_joint"
                   type="continuous"
@@ -85,21 +80,15 @@
   <!-- Define subcomponents links -->
   <link name="base_link" />
-  <xacro:platform material="white">
-    <xacro:white/>
-  </xacro:platform>
+  <xacro:platform material="white" />
   <xacro:drive_system prefix="left_back" flip_y="true" />
   <xacro:drive_system prefix="left_front" />
   <xacro:drive_system prefix="right_back" flip_x="true" flip_y="true"/>
   <xacro:drive_system prefix="right_front"  flip_x="true"/>
-  <xacro:indicator_light material="gray"><xacro:gray/></xacro:indicator_light>
+  <xacro:indicator_light material="gray" />
   <!-- Define sensors and cameras links -->
-  <xacro:hp_4310 prefix="back_mast" material="black">
-    <xacro:black/>
-  </xacro:hp_4310>
-  <xacro:hp_4310 prefix="front_mast" material="black">
-    <xacro:black/>
-  </xacro:hp_4310>
+  <xacro:hp_4310 prefix="back_mast" material="black" />
+  <xacro:hp_4310 prefix="front_mast" material="black" />
   <xacro:oak-d-w prefix="front"/>
-  <xacro:gnss material="gray"><xacro:gray/></xacro:gnss>
+  <xacro:gnss material="gray" />
   <!-- Define subcomponents joints -->
   <xacro:joint name="base_link_to_platform"

File: src/sirius_description/urdf/sirius_2/gnss.urdf.xacro (robot description, xacro)
@@ -3,5 +3,5 @@
      https://www.sparkfun.com/products/21801 -->
 <robot xmlns:xacro="http://wiki.ros.org/xacro">
-<xacro:macro name="gnss" params="material *gazebo_material package:=^ collisions:=^ inertial:=^ datum:=^ elevation:=^">
+<xacro:macro name="gnss" params="material package:=^ collisions:=^ inertial:=^ datum:=^ elevation:=^">
   <link name="gnss">
     <visual>
@@ -73,4 +73,9 @@
     </sensor>
   </gazebo>
+  <gazebo reference="gnss">
+      <visual>
+        <xacro:element xacro:name="xacro:${material}" />
+      </visual>
+  </gazebo>
 </xacro:macro>
 </robot>

File: src/sirius_description/urdf/sirius_2/indicator_light.urdf.xacro (robot description, xacro)
@@ -1,5 +1,5 @@
 <?xml version="1.0" encoding="utf-8"?>
 <robot xmlns:xacro="http://wiki.ros.org/xacro">
-<xacro:macro name="indicator_light" params="material prefix:='' *gazebo_material package:=^ collisions:=^ inertial:=^">
+<xacro:macro name="indicator_light" params="material prefix:='' package:=^ collisions:=^ inertial:=^">
   <link name="${prefix + '_' if prefix else prefix}indicator_light">
     <visual>
@@ -23,5 +23,5 @@
   <gazebo reference="${prefix + '_' if prefix else prefix}indicator_light">
       <visual>
-        <xacro:insert_block name="gazebo_material" />
+        <xacro:element xacro:name="xacro:${material}" />
       </visual>
   </gazebo>

File: src/sirius_description/urdf/sirius_2/platform.urdf.xacro (robot description, xacro)
@@ -1,4 +1,4 @@
 <robot xmlns:xacro="http://wiki.ros.org/xacro">
-<xacro:macro name="platform" params="material prefix:='' *gazebo_material  package:=^ collisions:=^ params:=^ inertial:=^">
+<xacro:macro name="platform" params="material prefix:=''  package:=^ collisions:=^ params:=^ inertial:=^">
     <link name="${prefix + '_' if prefix else prefix}platform">
       <visual>
@@ -65,5 +65,5 @@
     <gazebo reference="${prefix + '_' if prefix else prefix}platform">
       <visual>
-        <xacro:insert_block name="gazebo_material" />
+        <xacro:element xacro:name="xacro:${material}" />
       </visual>
     </gazebo>

File: src/sirius_description/urdf/sirius_2/suspension.urdf.xacro (robot description, xacro)
@@ -1,4 +1,4 @@
 <robot xmlns:xacro="http://wiki.ros.org/xacro">
-<xacro:macro name="suspension" params="prefix material *gazebo_material flip:=false params:=^ package:=^ collisions:=^ inertial:=^">
+<xacro:macro name="suspension" params="prefix material flip:=false params:=^ package:=^ collisions:=^ inertial:=^">
     <link name="${prefix}_suspension">
       <visual>
@@ -22,5 +22,5 @@
     <gazebo reference="${prefix}_suspension">
       <visual>
-        <xacro:insert_block name="gazebo_material" />
+        <xacro:element xacro:name="xacro:${material}" />
       </visual>
     </gazebo>

File: src/sirius_description/urdf/sirius_2/wheel.urdf.xacro (robot description, xacro)
@@ -1,4 +1,4 @@
 <robot xmlns:xacro="http://wiki.ros.org/xacro">
-<xacro:macro name="wheel" params="prefix material material_rim *gazebo_material **gazebo_material_rim flip:=false package:=^ params:=^ inertial:=^">
+<xacro:macro name="wheel" params="prefix material material_rim flip:=false package:=^ params:=^ inertial:=^">
     <link name="${prefix}_wheel">
       <visual>
@@ -34,5 +34,5 @@
       </collision>
     </link>
-    <joint name="${prefix}_wheel_to_rim" type="fixed">
+    <joint name="${prefix}_wheel_to_rim_joint" type="fixed">
       <parent link="${prefix}_wheel"/>
       <child link="${prefix}_wheel_rim"/>
@@ -41,10 +41,10 @@
     <gazebo reference="${prefix}_wheel">
       <visual>
-        <xacro:insert_block name="gazebo_material" />
+        <xacro:element xacro:name="xacro:${material}" />
       </visual>
     </gazebo>
     <gazebo reference="${prefix}_wheel_rim">
       <visual>
-        <xacro:insert_block name="gazebo_material_rim" />
+        <xacro:element xacro:name="xacro:${material_rim}" />
       </visual>
     </gazebo>
