Commit message: Load calibration data in camera urdf

File: src/sirius_description/urdf/cameras/oak-d-w.urdf.xacro (robot description, xacro)
@@ -1,7 +1,7 @@
 <?xml version="1.0"?>
 <robot xmlns:xacro="http://ros.org/wiki/xacro">
-  <xacro:property name="baseline" value="0.075"/>
   <xacro:property name="optical_offset_x" value="-0.01" />
-  <xacro:macro name="oak-d-w" params="prefix:=oak-d-w package:=^ cameras:=^ cameras_inertial:=^">
+  <xacro:macro name="oak-d-w" params="prefix:=oak-d-w package:=^ cameras:=^ cameras_inertial:=^ stereo_fps:=^|30 imu_frequency:=^|200 calibration:=^|${xacro.load_yaml('$(find sirius_description)/config/oak_d_w/kalibr_imucam_chain.yaml')}">
+    <xacro:property name="baseline" value="${sqrt(calibration.cam1.T_cn_cnm1[0][3]**2 + calibration.cam1.T_cn_cnm1[1][3]**2 + calibration.cam1.T_cn_cnm1[2][3]**2)}"/>
     <link name="${prefix}_camera_center">
       <visual>
@@ -54,14 +54,13 @@
     <!-- Left/Depth camera -->
     <gazebo reference="${prefix}_left_camera_frame">
-      <!-- Raw images (with lens distortion) -->
-      <sensor type="camera" name="${prefix}_left_camera_image_raw">
+       <sensor type="depth" name="${prefix}_camera_depth">
+        <!-- Rectified images, Depth images, Point Clouds -->
         <always_on>true</always_on>
-        <update_rate>15.0</update_rate>
+        <update_rate>${stereo_fps}</update_rate>
         <visualize>false</visualize>
-        <camera name="/${prefix}_camera/left_raw">
-          <horizontal_fov>${127 * pi/180}</horizontal_fov>
+        <camera name="/${prefix}_camera/depth">
           <image>
-            <width>1280</width>
-            <height>800</height>
+            <width>${calibration.cam0.resolution[0]}</width>
+            <height>${calibration.cam0.resolution[1]}</height>
             <format>L8</format>
           </image>
@@ -75,51 +74,14 @@
             <stddev>0.007</stddev>
           </noise>
-          <distortion>
-            <!-- Values copied from ZED2 camera -->
-            <k1>-0.043693598</k1>
-            <k2>0.0146164996</k2>
-            <p1>-0.006573319</p1>
-            <p2>-0.000216900</p2>
-            <k3>0.000084328</k3>
-            <center>0.5 0.5</center>
-          </distortion>
-        </camera>
-        <plugin name="camera_controller" filename="libgazebo_ros_camera.so">
-          <cameraName>/${prefix}_camera/left_raw</cameraName>
-          <imageTopicName>image_raw_gray</imageTopicName>
-          <cameraInfoTopicName>camera_info</cameraInfoTopicName>
-          <frameName>${prefix}_left_camera_optical_frame</frameName>
-          <distortionK1>-0.043693598</distortionK1>
-          <distortionK2>0.0146164996</distortionK2>
-          <distortionT1>-0.006573319</distortionT1>
-          <distortionT2>-0.000216900</distortionT2>
-          <distortionK3>0.000084328</distortionK3>
-          <CxPrime>648.5</CxPrime>
-          <Cx>648.5</Cx>
-          <Cy>366.8340148925781</Cy>
-          <hackBaseline>0.0</hackBaseline>
-        </plugin>
-      </sensor>
-      <sensor type="depth" name="${prefix}_camera_depth">
-        <!-- Rectified images, Depth images, Point Clouds -->
-        <always_on>true</always_on>
-        <update_rate>15.0</update_rate>
-        <visualize>false</visualize>
-        <camera name="/${prefix}_camera/depth">
-          <horizontal_fov>${127 * pi/180}</horizontal_fov>
-          <image>
-            <width>1280</width>
-            <height>800</height>
-            <format>L8</format>
-          </image>
-          <clip>
-            <near>0.02</near>
-            <far>300</far>
-          </clip>
-          <noise>
-            <type>gaussian</type>
-            <mean>0.0</mean>
-            <stddev>0.007</stddev>
-          </noise>
+          <lens>
+            <intrinsics>
+            <fx>${calibration.cam0.intrinsics[0]}</fx>
+            <fy>${calibration.cam0.intrinsics[1]}</fy>
+            <cx>${calibration.cam0.intrinsics[2]}</cx>
+            <cy>${calibration.cam0.intrinsics[3]}</cy>
+            <s>0</s>
+            </intrinsics>
+            <scale_to_hfov>false</scale_to_hfov>
+          </lens>
         </camera>
         <plugin name="camera_controller" filename="libgazebo_ros_openni_kinect.so">
@@ -134,7 +96,7 @@
           <frameName>${prefix}_left_camera_optical_frame</frameName>
           <baseline>${baseline}</baseline>
-          <CxPrime>658.8206787109375</CxPrime>
-          <Cx>658.8206787109375</Cx>
-          <Cy>372.25787353515625</Cy>
+          <CxPrime>${calibration.cam0.intrinsics[2]}</CxPrime>
+          <Cx>${calibration.cam0.intrinsics[2]}</Cx>
+          <Cy>${calibration.cam0.intrinsics[3]}</Cy>
           <hackBaseline>0.0</hackBaseline>
         </plugin>
@@ -143,14 +105,13 @@
     <!-- Right camera -->
     <gazebo reference="${prefix}_right_camera_frame">
-      <!-- Raw images (with lens distortion) -->
-      <sensor type="camera" name="${prefix}_left_camera_raw">
+      <sensor type="camera" name="${prefix}_right_camera_rect">
+        <!-- Rectified images -->
         <always_on>true</always_on>
-        <update_rate>15.0</update_rate>
+        <update_rate>${stereo_fps}</update_rate>
         <visualize>false</visualize>
-        <camera name="/${prefix}_camera/right_raw">
-          <horizontal_fov>${127 * pi/180}</horizontal_fov>
+        <camera name="/${prefix}_camera/right">
           <image>
-            <width>1280</width>
-            <height>800</height>
+            <width>${calibration.cam1.resolution[0]}</width>
+            <height>${calibration.cam1.resolution[1]}</height>
             <format>L8</format>
           </image>
@@ -164,50 +125,14 @@
             <stddev>0.007</stddev>
           </noise>
-          <distortion>
-            <k1>-0.040993299</k1>
-            <k2>0.009593590</k2>
-            <p1>-0.004429849</p1>
-            <p2>0.000192024</p2>
-            <k3>-0.000320880</k3>
-            <center>0.5 0.5</center>
-          </distortion>
-        </camera>
-        <plugin name="camera_controller" filename="libgazebo_ros_camera.so">
-          <cameraName>/${prefix}_camera/right_raw</cameraName>
-          <imageTopicName>image_raw_gray</imageTopicName>
-          <cameraInfoTopicName>camera_info</cameraInfoTopicName>
-          <frameName>${prefix}_right_camera_optical_frame</frameName>
-          <distortionK1>-0.040993299</distortionK1>
-          <distortionK2>0.009593590</distortionK2>
-          <distortionT1>-0.004429849</distortionT1>
-          <distortionT2>0.000192024</distortionT2>
-          <distortionK3>-0.000320880</distortionK3>
-          <CxPrime>659.3049926757812</CxPrime>
-          <Cx>659.3049926757812</Cx>
-          <Cy>371.39849853515625</Cy>
-          <hackBaseline>${baseline}</hackBaseline>
-        </plugin>
-      </sensor>
-      <sensor type="camera" name="${prefix}_right_camera_rect">
-        <!-- Rectified images -->
-        <always_on>true</always_on>
-        <update_rate>15.0</update_rate>
-        <visualize>false</visualize>
-        <camera name="/${prefix}_camera/right">
-          <horizontal_fov>${127 * pi/180}</horizontal_fov>
-          <image>
-            <width>1280</width>
-            <height>800</height>
-            <format>L8</format>
-          </image>
-          <clip>
-            <near>0.02</near>
-            <far>300</far>
-          </clip>
-          <noise>
-            <type>gaussian</type>
-            <mean>0.0</mean>
-            <stddev>0.007</stddev>
-          </noise>
+          <lens>
+            <intrinsics>
+            <fx>${calibration.cam1.intrinsics[0]}</fx>
+            <fy>${calibration.cam1.intrinsics[1]}</fy>
+            <cx>${calibration.cam1.intrinsics[2]}</cx>
+            <cy>${calibration.cam1.intrinsics[3]}</cy>
+            <s>0</s>
+            </intrinsics>
+            <scale_to_hfov>false</scale_to_hfov>
+          </lens>
         </camera>
         <plugin name="camera_controller" filename="libgazebo_ros_camera.so">
@@ -216,7 +141,7 @@
           <cameraInfoTopicName>camera_info</cameraInfoTopicName>
           <frameName>${prefix}_right_camera_optical_frame</frameName>
-          <CxPrime>658.8206787109375</CxPrime>
-          <Cx>658.8206787109375</Cx>
-          <Cy>372.25787353515625</Cy>
+          <CxPrime>${calibration.cam1.intrinsics[2]}</CxPrime>
+          <Cx>${calibration.cam1.intrinsics[2]}</Cx>
+          <Cy>${calibration.cam1.intrinsics[3]}</Cy>
           <hackBaseline>${baseline}</hackBaseline>
         </plugin>
@@ -226,9 +151,9 @@
     <gazebo reference="${prefix}_imu_frame">
       <sensor type="imu" name="imu_sensor">
-        <update_rate>100</update_rate>
+        <update_rate>${imu_frequency}</update_rate>
         <plugin filename="libgazebo_ros_imu_sensor.so" name="imu_plugin">
           <topicName>/${prefix}_camera/imu/data</topicName>
           <frameName>${prefix}_imu_frame</frameName>
-          <updateRateHZ>100.0</updateRateHZ>
+          <updateRateHZ>${imu_frequency}</updateRateHZ>
           <gaussianNoise>0.01</gaussianNoise>
           <initialOrientationAsReference>false</initialOrientationAsReference>

File: src/sirius_description/urdf/sirius_2.urdf.xacro (robot description, xacro)
@@ -3,4 +3,13 @@
   <xacro:property name="package" value="sirius_description" />
   <xacro:property name="params" value="${xacro.load_yaml('sirius_2.yaml')}" />
+  <xacro:arg name="calibration_path" default=""/>
+  <xacro:property name="calibration_path" value="$(arg calibration_path)" />
+  <xacro:if value="${calibration_path != ''}">
+    <xacro:property name="calibration" value="${xacro.load_yaml(calibration_path)}" />
+  </xacro:if>
+  <xacro:arg name="stereo_fps" default="30"/>
+  <xacro:property name="stereo_fps" value="$(arg stereo_fps)" />
+  <xacro:arg name="imu_frequency" default="200.0"/>
+  <xacro:property name="imu_frequency" value="$(arg imu_frequency)" />
   <xacro:property name="collisions" value="${xacro.load_yaml('sirius_2/sirius_2_collisions.yaml')}" />
   <xacro:property name="inertial" value="${xacro.load_yaml('sirius_2/sirius_2_inertial.yaml')}" />

Commit message: sirius_cameras package, working simulation

File: src/sirius_description/urdf/cameras/oak-d-w.urdf.xacro (robot description, xacro)
@@ -2,5 +2,5 @@
 <robot xmlns:xacro="http://ros.org/wiki/xacro">
   <xacro:property name="optical_offset_x" value="-0.01" />
-  <xacro:macro name="oak-d-w" params="prefix:=oak-d-w package:=^ cameras:=^ cameras_inertial:=^ stereo_fps:=^|30 imu_frequency:=^|200 calibration:=^|${xacro.load_yaml('$(find sirius_description)/config/oak_d_w/kalibr_imucam_chain.yaml')}">
+  <xacro:macro name="oak-d-w" params="prefix:=oak-d-w package:=^ cameras:=^ cameras_inertial:=^ stereo_fps:=^|30 imu_frequency:=^|200 calibration:=^|${xacro.load_yaml('$(find sirius_cameras)/config/oak_d_w/kalibr_imucam_chain.yaml')}">
     <xacro:property name="baseline" value="${sqrt(calibration.cam1.T_cn_cnm1[0][3]**2 + calibration.cam1.T_cn_cnm1[1][3]**2 + calibration.cam1.T_cn_cnm1[2][3]**2)}"/>
     <link name="${prefix}_camera_center">
@@ -21,4 +21,5 @@
       </inertial>
     </link>
+    <link name="${prefix}_rgb_camera_optical_frame"/>
     <link name="${prefix}_left_camera_frame" />
     <link name="${prefix}_left_camera_optical_frame"/>
@@ -26,4 +27,9 @@
     <link name="${prefix}_right_camera_optical_frame"/>
     <link name="${prefix}_imu_frame"/>
+    <joint name="${prefix}_rgb_camera_optical_joint" type="fixed">
+      <origin xyz="${optical_offset_x} 0 0" rpy="-${pi/2} 0.0 -${pi/2}"/>
+      <parent link="${prefix}_camera_center"/>
+      <child link="${prefix}_rgb_camera_optical_frame"/>
+    </joint>
     <joint name="${prefix}_left_camera_joint" type="fixed">
       <parent link="${prefix}_camera_center"/>
@@ -48,16 +54,16 @@
     <joint name="${prefix}_imu_frame_joint" type="fixed">
       <!-- IMU frame offset copied from ZED2 camera -->
-      <origin xyz="-0.002 -0.023 -0.002" rpy="0.0014025 -0.0000012 -0.0016915"/>
+      <origin xyz="${calibration.cam0.T_imu_cam[0][3]} ${calibration.cam0.T_imu_cam[1][3]} ${calibration.cam0.T_imu_cam[2][3]}" rpy="${atan2(calibration.cam0.T_imu_cam[2][1],calibration.cam0.T_imu_cam[2][2])} ${atan2(-calibration.cam0.T_imu_cam[2][0],sqrt(calibration.cam0.T_imu_cam[2][1]**2 + calibration.cam0.T_imu_cam[2][2]**2))} ${atan2(calibration.cam0.T_imu_cam[1][0],calibration.cam0.T_imu_cam[0][0])}"/>
       <parent link="${prefix}_left_camera_frame"/>
       <child link="${prefix}_imu_frame"/>
     </joint>
     <!-- Left/Depth camera -->
-    <gazebo reference="${prefix}_left_camera_frame">
-       <sensor type="depth" name="${prefix}_camera_depth">
-        <!-- Rectified images, Depth images, Point Clouds -->
+    <gazebo reference="${prefix}_camera_center">
+      <sensor type="multicamera" name="${prefix}_stereo_camera">
         <always_on>true</always_on>
         <update_rate>${stereo_fps}</update_rate>
         <visualize>false</visualize>
-        <camera name="/${prefix}_camera/depth">
+        <camera name="/${prefix}_camera/left">
+          <pose>0 ${baseline/2} 0 0 0 0</pose>
           <image>
             <width>${calibration.cam0.resolution[0]}</width>
@@ -85,33 +91,9 @@
           </lens>
         </camera>
-        <plugin name="camera_controller" filename="libgazebo_ros_openni_kinect.so">
-          <cameraName>/${prefix}_camera</cameraName>
-          <imageTopicName>left/image_rect_gray</imageTopicName>
-          <cameraInfoTopicName>left/camera_info</cameraInfoTopicName>
-          <depthImageTopicName>depth/depth_registered</depthImageTopicName>
-          <depthImageInfoTopicName>depth/camera_info</depthImageInfoTopicName>
-          <pointCloudTopicName>point_cloud/cloud_registered</pointCloudTopicName>
-          <pointCloudCutoff>0.35</pointCloudCutoff>
-          <pointCloudCutoffMax>35.0</pointCloudCutoffMax>
-          <frameName>${prefix}_left_camera_optical_frame</frameName>
-          <baseline>${baseline}</baseline>
-          <CxPrime>${calibration.cam0.intrinsics[2]}</CxPrime>
-          <Cx>${calibration.cam0.intrinsics[2]}</Cx>
-          <Cy>${calibration.cam0.intrinsics[3]}</Cy>
-          <hackBaseline>0.0</hackBaseline>
-        </plugin>
-      </sensor>
-    </gazebo>
-    <!-- Right camera -->
-    <gazebo reference="${prefix}_right_camera_frame">
-      <sensor type="camera" name="${prefix}_right_camera_rect">
-        <!-- Rectified images -->
-        <always_on>true</always_on>
-        <update_rate>${stereo_fps}</update_rate>
-        <visualize>false</visualize>
         <camera name="/${prefix}_camera/right">
+          <pose>0 -${baseline/2} 0 0 0 0</pose>
           <image>
-            <width>${calibration.cam1.resolution[0]}</width>
-            <height>${calibration.cam1.resolution[1]}</height>
+            <width>${calibration.cam0.resolution[0]}</width>
+            <height>${calibration.cam0.resolution[1]}</height>
             <format>L8</format>
           </image>
@@ -127,8 +109,8 @@
           <lens>
             <intrinsics>
-            <fx>${calibration.cam1.intrinsics[0]}</fx>
-            <fy>${calibration.cam1.intrinsics[1]}</fy>
-            <cx>${calibration.cam1.intrinsics[2]}</cx>
-            <cy>${calibration.cam1.intrinsics[3]}</cy>
+            <fx>${calibration.cam0.intrinsics[0]}</fx>
+            <fy>${calibration.cam0.intrinsics[1]}</fy>
+            <cx>${calibration.cam0.intrinsics[2]}</cx>
+            <cy>${calibration.cam0.intrinsics[3]}</cy>
             <s>0</s>
             </intrinsics>
@@ -136,12 +118,12 @@
           </lens>
         </camera>
-        <plugin name="camera_controller" filename="libgazebo_ros_camera.so">
-          <cameraName>/${prefix}_camera/right</cameraName>
+        <plugin name="stereo_camera_controller" filename="libgazebo_ros_multicamera.so">
+          <alwaysOn>true</alwaysOn>
+          <updateRate>${stereo_fps}</updateRate>
+          <cameraName>/${prefix}_camera</cameraName>
           <imageTopicName>image_rect_gray</imageTopicName>
           <cameraInfoTopicName>camera_info</cameraInfoTopicName>
-          <frameName>${prefix}_right_camera_optical_frame</frameName>
-          <CxPrime>${calibration.cam1.intrinsics[2]}</CxPrime>
-          <Cx>${calibration.cam1.intrinsics[2]}</Cx>
-          <Cy>${calibration.cam1.intrinsics[3]}</Cy>
+          <frameName>${prefix}_left_camera_optical_frame</frameName>
+          <rightFrameName>${prefix}_right_camera_optical_frame</rightFrameName>
           <hackBaseline>${baseline}</hackBaseline>
         </plugin>
@@ -156,5 +138,5 @@
           <frameName>${prefix}_imu_frame</frameName>
           <updateRateHZ>${imu_frequency}</updateRateHZ>
-          <gaussianNoise>0.01</gaussianNoise>
+          <gaussianNoise>0.0</gaussianNoise>
           <initialOrientationAsReference>false</initialOrientationAsReference>
           <xyzOffset>0 0.0 0.0</xyzOffset>
