Commit message: 12 magnetometr i odometria wizualna w symulacji (#10)
* add gazebo_ros_magnetometer_sensor as submodule

* Add magnetometer plugin to zed and luxonis cameras

* add gaussian noise to magnetometers

* Add package for visual odometry

* open_vins partial config

* remove open_vins

* remove open_vins from submodules

* add morb_slam_ros

* Fix typos in zed urdf

* remove zed camera

* Change oak-d-w camera to (pseudo) grayscale

* Add oak_d_w calibration

* Match topic names with simulation

* Remove yaml version so xacro and ros can load file

* Add morb_slam configs for real camera and sim

* Load calibration data in camera urdf

* add viewer parameters to morb_slam_gazebo

* Add launch for morb_slam

* Real imu noise values

* sirius_cameras package, working simulation

* remove visualizer settings; update morb_slam_ros

* change oak_d_w camera namespace

* change tf from map to odom

* Remove unused commented code in oak node

File: src/sirius_description/urdf/cameras/oak-d-w.urdf.xacro (robot description, xacro)
@@ -1,7 +1,7 @@
 <?xml version="1.0"?>
 <robot xmlns:xacro="http://ros.org/wiki/xacro">
-  <xacro:property name="baseline" value="0.075"/>
   <xacro:property name="optical_offset_x" value="-0.01" />
-  <xacro:macro name="oak-d-w" params="prefix:=oak-d-w package:=^ cameras:=^ cameras_inertial:=^">
+  <xacro:macro name="oak-d-w" params="prefix:=oak-d-w package:=^ cameras:=^ cameras_inertial:=^ stereo_fps:=^|30 imu_frequency:=^|200 calibration:=^|${xacro.load_yaml('$(find sirius_cameras)/config/oak_d_w/kalibr_imucam_chain.yaml')}">
+    <xacro:property name="baseline" value="${sqrt(calibration.cam1.T_cn_cnm1[0][3]**2 + calibration.cam1.T_cn_cnm1[1][3]**2 + calibration.cam1.T_cn_cnm1[2][3]**2)}"/>
     <link name="${prefix}_camera_center">
       <visual>
@@ -21,4 +21,5 @@
       </inertial>
     </link>
+    <link name="${prefix}_rgb_camera_optical_frame"/>
     <link name="${prefix}_left_camera_frame" />
     <link name="${prefix}_left_camera_optical_frame"/>
@@ -26,4 +27,9 @@
     <link name="${prefix}_right_camera_optical_frame"/>
     <link name="${prefix}_imu_frame"/>
+    <joint name="${prefix}_rgb_camera_optical_joint" type="fixed">
+      <origin xyz="${optical_offset_x} 0 0" rpy="-${pi/2} 0.0 -${pi/2}"/>
+      <parent link="${prefix}_camera_center"/>
+      <child link="${prefix}_rgb_camera_optical_frame"/>
+    </joint>
     <joint name="${prefix}_left_camera_joint" type="fixed">
       <parent link="${prefix}_camera_center"/>
@@ -47,22 +53,21 @@
     </joint>
     <joint name="${prefix}_imu_frame_joint" type="fixed">
-      <!-- IMU frame offset copied from an actual ZED2 camera -->
-      <origin xyz="-0.002 -0.023 -0.002" rpy="0.0014025 -0.0000012 -0.0016915"/>
+      <!-- IMU frame offset copied from ZED2 camera -->
+      <origin xyz="${calibration.cam0.T_imu_cam[0][3]} ${calibration.cam0.T_imu_cam[1][3]} ${calibration.cam0.T_imu_cam[2][3]}" rpy="${atan2(calibration.cam0.T_imu_cam[2][1],calibration.cam0.T_imu_cam[2][2])} ${atan2(-calibration.cam0.T_imu_cam[2][0],sqrt(calibration.cam0.T_imu_cam[2][1]**2 + calibration.cam0.T_imu_cam[2][2]**2))} ${atan2(calibration.cam0.T_imu_cam[1][0],calibration.cam0.T_imu_cam[0][0])}"/>
       <parent link="${prefix}_left_camera_frame"/>
       <child link="${prefix}_imu_frame"/>
     </joint>
     <!-- Left/Depth camera -->
-    <gazebo reference="${prefix}_left_camera_frame">
-      <!-- Raw images (with lens distortion) -->
-      <sensor type="camera" name="${prefix}_left_camera_image_raw">
+    <gazebo reference="${prefix}_camera_center">
+      <sensor type="multicamera" name="${prefix}_stereo_camera">
         <always_on>true</always_on>
-        <update_rate>15.0</update_rate>
+        <update_rate>${stereo_fps}</update_rate>
         <visualize>false</visualize>
-        <camera name="/${prefix}_camera/left_raw">
-          <horizontal_fov>${127 * pi/180}</horizontal_fov>
+        <camera name="/${prefix}_camera/left">
+          <pose>0 ${baseline/2} 0 0 0 0</pose>
           <image>
-            <width>1280</width>
-            <height>800</height>
-            <format>R8G8B8</format>
+            <width>${calibration.cam0.resolution[0]}</width>
+            <height>${calibration.cam0.resolution[1]}</height>
+            <format>L8</format>
           </image>
           <clip>
@@ -75,41 +80,21 @@
             <stddev>0.007</stddev>
           </noise>
-          <distortion>
-            <!-- Values copied from an actual ZED2 camera -->
-            <k1>-0.043693598</k1>
-            <k2>0.0146164996</k2>
-            <p1>-0.006573319</p1>
-            <p2>-0.000216900</p2>
-            <k3>0.000084328</k3>
-            <center>0.5 0.5</center>
-          </distortion>
+          <lens>
+            <intrinsics>
+            <fx>${calibration.cam0.intrinsics[0]}</fx>
+            <fy>${calibration.cam0.intrinsics[1]}</fy>
+            <cx>${calibration.cam0.intrinsics[2]}</cx>
+            <cy>${calibration.cam0.intrinsics[3]}</cy>
+            <s>0</s>
+            </intrinsics>
+            <scale_to_hfov>false</scale_to_hfov>
+          </lens>
         </camera>
-        <plugin name="camera_controller" filename="libgazebo_ros_camera.so">
-          <cameraName>/${prefix}_camera/left_raw</cameraName>
-          <imageTopicName>image_raw_color</imageTopicName>
-          <cameraInfoTopicName>camera_info</cameraInfoTopicName>
-          <frameName>${prefix}_left_camera_optical_frame</frameName>
-          <distortionK1>-0.043693598</distortionK1>
-          <distortionK2>0.0146164996</distortionK2>
-          <distortionT1>-0.006573319</distortionT1>
-          <distortionT2>-0.000216900</distortionT2>
-          <distortionK3>0.000084328</distortionK3>
-          <CxPrime>648.5</CxPrime>
-          <Cx>648.5</Cx>
-          <Cy>366.8340148925781</Cy>
-          <hackBaseline>0.0</hackBaseline>
-        </plugin>
-      </sensor>
-      <sensor type="depth" name="${prefix}_camera_depth">
-        <!-- Rectified images, Depth images, Point Clouds -->
-        <always_on>true</always_on>
-        <update_rate>15.0</update_rate>
-        <visualize>false</visualize>
-        <camera name="/${prefix}_camera/depth">
-          <horizontal_fov>${127 * pi/180}</horizontal_fov>
+        <camera name="/${prefix}_camera/right">
+          <pose>0 -${baseline/2} 0 0 0 0</pose>
           <image>
-            <width>1280</width>
-            <height>800</height>
-            <format>R8G8B8</format>
+            <width>${calibration.cam0.resolution[0]}</width>
+            <height>${calibration.cam0.resolution[1]}</height>
+            <format>L8</format>
           </image>
           <clip>
@@ -122,101 +107,23 @@
             <stddev>0.007</stddev>
           </noise>
+          <lens>
+            <intrinsics>
+            <fx>${calibration.cam0.intrinsics[0]}</fx>
+            <fy>${calibration.cam0.intrinsics[1]}</fy>
+            <cx>${calibration.cam0.intrinsics[2]}</cx>
+            <cy>${calibration.cam0.intrinsics[3]}</cy>
+            <s>0</s>
+            </intrinsics>
+            <scale_to_hfov>false</scale_to_hfov>
+          </lens>
         </camera>
-        <plugin name="camera_controller" filename="libgazebo_ros_openni_kinect.so">
+        <plugin name="stereo_camera_controller" filename="libgazebo_ros_multicamera.so">
+          <alwaysOn>true</alwaysOn>
+          <updateRate>${stereo_fps}</updateRate>
           <cameraName>/${prefix}_camera</cameraName>
-          <imageTopicName>left_rect/image_raw_color</imageTopicName>
-          <cameraInfoTopicName>left_rect/camera_info</cameraInfoTopicName>
-          <depthImageTopicName>depth/depth_registered</depthImageTopicName>
-          <depthImageInfoTopicName>depth/camera_info</depthImageInfoTopicName>
-          <pointCloudTopicName>point_cloud/cloud_registered</pointCloudTopicName>
-          <pointCloudCutoff>0.35</pointCloudCutoff>
-          <pointCloudCutoffMax>35.0</pointCloudCutoffMax>
+          <imageTopicName>image_rect_gray</imageTopicName>
+          <cameraInfoTopicName>camera_info</cameraInfoTopicName>
           <frameName>${prefix}_left_camera_optical_frame</frameName>
-          <baseline>${baseline}</baseline>
-          <CxPrime>658.8206787109375</CxPrime>
-          <Cx>658.8206787109375</Cx>
-          <Cy>372.25787353515625</Cy>
-          <hackBaseline>0.0</hackBaseline>
-        </plugin>
-      </sensor>
-    </gazebo>
-    <!-- Right camera -->
-    <gazebo reference="${prefix}_right_camera_frame">
-      <!-- Raw images (with lens distortion) -->
-      <sensor type="camera" name="${prefix}_left_camera_raw">
-        <always_on>true</always_on>
-        <update_rate>15.0</update_rate>
-        <visualize>false</visualize>
-        <camera name="/${prefix}_camera/right_raw">
-          <horizontal_fov>${127 * pi/180}</horizontal_fov>
-          <image>
-            <width>1280</width>
-            <height>800</height>
-            <format>R8G8B8</format>
-          </image>
-          <clip>
-            <near>0.02</near>
-            <far>300</far>
-          </clip>
-          <noise>
-            <type>gaussian</type>
-            <mean>0.0</mean>
-            <stddev>0.007</stddev>
-          </noise>
-          <distortion>
-            <k1>-0.040993299</k1>
-            <k2>0.009593590</k2>
-            <p1>-0.004429849</p1>
-            <p2>0.000192024</p2>
-            <k3>-0.000320880</k3>
-            <center>0.5 0.5</center>
-          </distortion>
-        </camera>
-        <plugin name="camera_controller" filename="libgazebo_ros_camera.so">
-          <cameraName>/${prefix}_camera/right_raw</cameraName>
-          <imageTopicName>image_raw_color</imageTopicName>
-          <cameraInfoTopicName>camera_info</cameraInfoTopicName>
-          <frameName>${prefix}_right_camera_optical_frame</frameName>
-          <distortionK1>-0.040993299</distortionK1>
-          <distortionK2>0.009593590</distortionK2>
-          <distortionT1>-0.004429849</distortionT1>
-          <distortionT2>0.000192024</distortionT2>
-          <distortionK3>-0.000320880</distortionK3>
-          <CxPrime>659.3049926757812</CxPrime>
-          <Cx>659.3049926757812</Cx>
-          <Cy>371.39849853515625</Cy>
-          <hackBaseline>${baseline}</hackBaseline>
-        </plugin>
-      </sensor>
-      <sensor type="camera" name="${prefix}_right_camera_rect">
-        <!-- Rectified images -->
-        <always_on>true</always_on>
-        <update_rate>15.0</update_rate>
-        <visualize>false</visualize>
-        <camera name="/${prefix}_camera/right">
-          <horizontal_fov>${127 * pi/180}</horizontal_fov>
-          <image>
-            <width>1280</width>
-            <height>800</height>
-            <format>R8G8B8</format>
-          </image>
-          <clip>
-            <near>0.02</near>
-            <far>300</far>
-          </clip>
-          <noise>
-            <type>gaussian</type>
-            <mean>0.0</mean>
-            <stddev>0.007</stddev>
-          </noise>
-        </camera>
-        <plugin name="camera_controller" filename="libgazebo_ros_camera.so">
-          <cameraName>/${prefix}_camera/right</cameraName>
-          <imageTopicName>image_rect_color</imageTopicName>
-          <cameraInfoTopicName>camera_info</cameraInfoTopicName>
-          <frameName>${prefix}_right_camera_optical_frame</frameName>
-          <CxPrime>658.8206787109375</CxPrime>
-          <Cx>658.8206787109375</Cx>
-          <Cy>372.25787353515625</Cy>
+          <rightFrameName>${prefix}_right_camera_optical_frame</rightFrameName>
           <hackBaseline>${baseline}</hackBaseline>
         </plugin>
@@ -225,11 +132,11 @@
     <!-- IMU -->
     <gazebo reference="${prefix}_imu_frame">
-      <sensor type="imu" name="zed2_imu_sensor">
-        <update_rate>100</update_rate>
+      <sensor type="imu" name="imu_sensor">
+        <update_rate>${imu_frequency}</update_rate>
         <plugin filename="libgazebo_ros_imu_sensor.so" name="imu_plugin">
           <topicName>/${prefix}_camera/imu/data</topicName>
           <frameName>${prefix}_imu_frame</frameName>
-          <updateRateHZ>100.0</updateRateHZ>
-          <gaussianNoise>0.01</gaussianNoise>
+          <updateRateHZ>${imu_frequency}</updateRateHZ>
+          <gaussianNoise>0.0</gaussianNoise>
           <initialOrientationAsReference>false</initialOrientationAsReference>
           <xyzOffset>0 0.0 0.0</xyzOffset>
@@ -238,4 +145,36 @@
       </sensor>
     </gazebo>
+    <!-- MAGNETOMETER -->
+    <gazebo reference="${prefix}_imu_frame">
+      <sensor type="magnetometer" name="magnetometer_sensor">
+        <always_on>true</always_on>
+        <update_rate>50</update_rate>
+        <magnetometer>
+          <x>
+            <noise type="gaussian">
+              <mean>0.0</mean>
+              <stddev>5e-7</stddev>
+            </noise>
+          </x>
+          <y>
+            <noise type="gaussian">
+              <mean>0.0</mean>
+              <stddev>5e-7</stddev>
+            </noise>
+          </y>
+          <z>
+            <noise type="gaussian">
+              <mean>0.0</mean>
+              <stddev>5e-7</stddev>
+            </noise>
+          </z>
+        </magnetometer>
+        <plugin filename="libgazebo_ros_magnetometer_sensor.so" name="magnetometer_plugin">
+          <topicName>/${prefix}_camera/imu/mag</topicName>
+          <frameName>${prefix}_imu_frame</frameName>
+          <updateRateHZ>50.0</updateRateHZ>
+        </plugin>
+      </sensor>
+    </gazebo>
   </xacro:macro>
 </robot>

File: src/sirius_description/urdf/cameras/zed2i.urdf.xacro (robot description, xacro)
@@ -1,4 +1,5 @@
 <?xml version="1.0"?>
 <robot xmlns:xacro="http://ros.org/wiki/xacro">
+<!-- https://support.stereolabs.com/hc/en-us/articles/360007395634-What-is-the-camera-focal-length-and-field-of-view- -->
   <xacro:property name="baseline" value="0.12"/>
   <xacro:property name="optical_offset_x" value="-0.01" />
@@ -46,6 +47,5 @@
     </joint>
     <joint name="${prefix}_imu_frame_joint" type="fixed">
-      <!-- IMU frame offset copied from an actual ZED2 camera -->
-      <origin xyz="-0.002 -0.023 -0.002" rpy="0.0014025 -0.0000012 -0.0016915"/>
+      <origin xyz="-0.002 -0.023 -0.002" rpy="0 0 0"/>
       <parent link="${prefix}_left_camera_frame"/>
       <child link="${prefix}_imu_frame"/>
@@ -59,5 +59,5 @@
         <visualize>false</visualize>
         <camera name="/${prefix}_camera/left_raw">
-          <horizontal_fov>${110 * pi/180}</horizontal_fov>
+          <horizontal_fov>${104 * pi/180}</horizontal_fov>
           <image>
             <width>1280</width>
@@ -75,10 +75,9 @@
           </noise>
           <distortion>
-            <!-- Values copied from an actual ZED2 camera -->
-            <k1>-0.043693598</k1>
-            <k2>0.0146164996</k2>
-            <p1>-0.006573319</p1>
-            <p2>-0.000216900</p2>
-            <k3>0.000084328</k3>
+            <!-- Radial-tangential model -->
+            <k1>0</k1> <!-- k1 in kalibr-->
+            <k2>0</k2> <!-- k2 in kalibr-->
+            <p1>0</p1> <!-- r1 in kalibr-->
+            <p2>0</p2> <!-- r2 in kalibr-->
             <center>0.5 0.5</center>
           </distortion>
@@ -89,12 +88,11 @@
           <cameraInfoTopicName>camera_info</cameraInfoTopicName>
           <frameName>${prefix}_left_camera_optical_frame</frameName>
-          <distortionK1>-0.043693598</distortionK1>
-          <distortionK2>0.0146164996</distortionK2>
-          <distortionT1>-0.006573319</distortionT1>
-          <distortionT2>-0.000216900</distortionT2>
-          <distortionK3>0.000084328</distortionK3>
-          <CxPrime>648.5</CxPrime>
-          <Cx>648.5</Cx>
-          <Cy>366.8340148925781</Cy>
+          <distortionK1>0</distortionK1>
+          <distortionK2>0</distortionK2>
+          <distortionT1>0</distortionT1>
+          <distortionT2>0</distortionT2>
+          <CxPrime>640</CxPrime>
+          <Cx>640</Cx>
+          <Cy>360</Cy>
           <hackBaseline>0.0</hackBaseline>
         </plugin>
@@ -106,5 +104,5 @@
         <visualize>false</visualize>
         <camera name="/${prefix}_camera/depth">
-          <horizontal_fov>${110 * pi/180}</horizontal_fov>
+          <horizontal_fov>${104 * pi/180}</horizontal_fov>
           <image>
             <width>1280</width>
@@ -133,7 +131,7 @@
           <frameName>${prefix}_left_camera_optical_frame</frameName>
           <baseline>0.12</baseline>
-          <CxPrime>658.8206787109375</CxPrime>
-          <Cx>658.8206787109375</Cx>
-          <Cy>372.25787353515625</Cy>
+          <CxPrime>640</CxPrime>
+          <Cx>640</Cx>
+          <Cy>360</Cy>
           <hackBaseline>0.0</hackBaseline>
         </plugin>
@@ -148,5 +146,5 @@
         <visualize>false</visualize>
         <camera name="/${prefix}_camera/right_raw">
-          <horizontal_fov>${110 * pi/180}</horizontal_fov>
+          <horizontal_fov>${104 * pi/180}</horizontal_fov>
           <image>
             <width>1280</width>
@@ -164,9 +162,9 @@
           </noise>
           <distortion>
-            <k1>-0.040993299</k1>
-            <k2>0.009593590</k2>
-            <p1>-0.004429849</p1>
-            <p2>0.000192024</p2>
-            <k3>-0.000320880</k3>
+            <!-- Radial-tangential model -->
+            <k1>0</k1> <!-- k1 in kalibr-->
+            <k2>0</k2> <!-- k2 in kalibr-->
+            <p1>0</p1> <!-- r1 in kalibr-->
+            <p2>0</p2> <!-- r2 in kalibr-->
             <center>0.5 0.5</center>
           </distortion>
@@ -177,13 +175,12 @@
           <cameraInfoTopicName>camera_info</cameraInfoTopicName>
           <frameName>${prefix}_right_camera_optical_frame</frameName>
-          <distortionK1>-0.040993299</distortionK1>
-          <distortionK2>0.009593590</distortionK2>
-          <distortionT1>-0.004429849</distortionT1>
-          <distortionT2>0.000192024</distortionT2>
-          <distortionK3>-0.000320880</distortionK3>
-          <CxPrime>659.3049926757812</CxPrime>
-          <Cx>659.3049926757812</Cx>
-          <Cy>371.39849853515625</Cy>
-          <hackBaseline>0.12</hackBaseline>
+          <distortionK1>0</distortionK1>
+          <distortionK2>0</distortionK2>
+          <distortionT1>0</distortionT1>
+          <distortionT2>0</distortionT2>
+          <CxPrime>640</CxPrime>
+          <Cx>640</Cx>
+          <Cy>360</Cy>
+          <hackBaseline>0.0</hackBaseline>
         </plugin>
       </sensor>
@@ -194,5 +191,5 @@
         <visualize>false</visualize>
         <camera name="/${prefix}_camera/right">
-          <horizontal_fov>${110 * pi/180}</horizontal_fov>
+          <horizontal_fov>${104 * pi/180}</horizontal_fov>
           <image>
             <width>1280</width>
@@ -215,8 +212,8 @@
           <cameraInfoTopicName>camera_info</cameraInfoTopicName>
           <frameName>${prefix}_right_camera_optical_frame</frameName>
-          <CxPrime>658.8206787109375</CxPrime>
-          <Cx>658.8206787109375</Cx>
-          <Cy>372.25787353515625</Cy>
-          <hackBaseline>0.12</hackBaseline>
+          <CxPrime>640</CxPrime>
+          <Cx>640</Cx>
+          <Cy>360</Cy>
+          <hackBaseline>0</hackBaseline>
         </plugin>
       </sensor>
@@ -224,5 +221,5 @@
     <!-- IMU -->
     <gazebo reference="${prefix}_imu_frame">
-      <sensor type="imu" name="zed2_imu_sensor">
+      <sensor type="imu" name="imu_sensor">
         <update_rate>100</update_rate>
         <plugin filename="libgazebo_ros_imu_sensor.so" name="imu_plugin">
@@ -237,4 +234,36 @@
       </sensor>
     </gazebo>
+    <!-- MAGNETOMETER -->
+    <gazebo reference="${prefix}_imu_frame">
+      <sensor type="magnetometer" name="magnetometer_sensor">
+        <always_on>true</always_on>
+        <update_rate>50</update_rate>
+        <magnetometer>
+          <x>
+            <noise type="gaussian">
+              <mean>0.0</mean>
+              <stddev>5e-7</stddev>
+            </noise>
+          </x>
+          <y>
+            <noise type="gaussian">
+              <mean>0.0</mean>
+              <stddev>5e-7</stddev>
+            </noise>
+          </y>
+          <z>
+            <noise type="gaussian">
+              <mean>0.0</mean>
+              <stddev>5e-7</stddev>
+            </noise>
+          </z>
+        </magnetometer>
+        <plugin filename="libgazebo_ros_magnetometer_sensor.so" name="magnetometer_plugin">
+          <topicName>/${prefix}_camera/imu/mag</topicName>
+          <frameName>${prefix}_imu_frame</frameName>
+          <updateRateHZ>50.0</updateRateHZ>
+        </plugin>
+      </sensor>
+    </gazebo>
   </xacro:macro>
 </robot>

File: src/sirius_description/urdf/sirius_2.urdf.xacro (robot description, xacro)
@@ -3,4 +3,13 @@
   <xacro:property name="package" value="sirius_description" />
   <xacro:property name="params" value="${xacro.load_yaml('sirius_2.yaml')}" />
+  <xacro:arg name="calibration_path" default=""/>
+  <xacro:property name="calibration_path" value="$(arg calibration_path)" />
+  <xacro:if value="${calibration_path != ''}">
+    <xacro:property name="calibration" value="${xacro.load_yaml(calibration_path)}" />
+  </xacro:if>
+  <xacro:arg name="stereo_fps" default="30"/>
+  <xacro:property name="stereo_fps" value="$(arg stereo_fps)" />
+  <xacro:arg name="imu_frequency" default="200.0"/>
+  <xacro:property name="imu_frequency" value="$(arg imu_frequency)" />
   <xacro:property name="collisions" value="${xacro.load_yaml('sirius_2/sirius_2_collisions.yaml')}" />
   <xacro:property name="inertial" value="${xacro.load_yaml('sirius_2/sirius_2_inertial.yaml')}" />
@@ -11,5 +20,4 @@
   <xacro:include filename="sirius_2/platform.urdf.xacro" />
   <xacro:include filename="cameras/hp_4310.urdf.xacro" />
-  <xacro:include filename="cameras/zed2i.urdf.xacro" />
   <xacro:include filename="cameras/oak-d-w.urdf.xacro" />
   <xacro:property name="link_prefix" value=""/>
@@ -64,6 +72,5 @@
     <xacro:black/>
   </xacro:hp_4310>
-  <xacro:zed2i prefix="front"/>
-  <xacro:oak-d-w prefix="back"/>
+  <xacro:oak-d-w prefix="front"/>
   <xacro:drive_system prefix="right_front" />
   <xacro:drive_system reflect="true" prefix="right_back" direction="-1"/>
@@ -125,9 +132,4 @@
     <origin xyz="${params['front_camera_xyz']}" rpy="${params['front_camera_rpy']}"/>
   </joint>
-  <joint name="base_to_back_camera" type="fixed">
-    <parent link="main_platform"/>
-    <child link="back_camera_center"/>
-    <origin xyz="${params['back_camera_xyz']}" rpy="${params['back_camera_rpy']}"/>
-  </joint>
   <gazebo>
     <plugin name="gazebo_ros_control" filename="libgazebo_ros_control.so">
