Commit message: Fix camera and imu orientation in imu

File: src/sirius_description/urdf/cameras/oak-d-w.urdf.xacro (robot description, xacro)
@@ -26,5 +26,5 @@
     <link name="${prefix}_right_camera_frame" />
     <link name="${prefix}_right_camera_optical_frame"/>
-    <link name="${prefix}_imu_frame"/>
+    <link name="${prefix}_camera_imu_frame"/>
     <joint name="${prefix}_rgb_camera_optical_joint" type="fixed">
       <origin xyz="${optical_offset_x} 0 0" rpy="-${pi/2} 0.0 -${pi/2}"/>
@@ -38,6 +38,6 @@
     </joint>
     <joint name="${prefix}_left_camera_optical_joint" type="fixed">
-      <origin xyz="${optical_offset_x} 0 0" rpy="-${pi/2} 0.0 -${pi/2}"/>
-      <parent link="${prefix}_left_camera_frame"/>
+      <origin xyz="${calibration.cam1.T_cn_cnm1[0][3]} ${calibration.cam1.T_cn_cnm1[1][3]} ${calibration.cam1.T_cn_cnm1[2][3]}" rpy="${atan2(calibration.cam1.T_cn_cnm1[2][1],calibration.cam1.T_cn_cnm1[2][2])} ${atan2(-calibration.cam1.T_cn_cnm1[2][0],sqrt(calibration.cam1.T_cn_cnm1[2][1]**2 + calibration.cam1.T_cn_cnm1[2][2]**2))} ${atan2(calibration.cam1.T_cn_cnm1[1][0],calibration.cam1.T_cn_cnm1[0][0])}"/>
+      <parent link="${prefix}_right_camera_optical_frame"/>
       <child link="${prefix}_left_camera_optical_frame"/>
     </joint>
@@ -52,9 +52,9 @@
       <child link="${prefix}_right_camera_optical_frame"/>
     </joint>
-    <joint name="${prefix}_imu_frame_joint" type="fixed">
+    <joint name="${prefix}_camera_imu_frame_joint" type="fixed">
       <!-- IMU frame offset copied from ZED2 camera -->
-      <origin xyz="${calibration.cam0.T_imu_cam[0][3]} ${calibration.cam0.T_imu_cam[1][3]} ${calibration.cam0.T_imu_cam[2][3]}" rpy="${atan2(calibration.cam0.T_imu_cam[2][1],calibration.cam0.T_imu_cam[2][2])} ${atan2(-calibration.cam0.T_imu_cam[2][0],sqrt(calibration.cam0.T_imu_cam[2][1]**2 + calibration.cam0.T_imu_cam[2][2]**2))} ${atan2(calibration.cam0.T_imu_cam[1][0],calibration.cam0.T_imu_cam[0][0])}"/>
-      <parent link="${prefix}_left_camera_frame"/>
-      <child link="${prefix}_imu_frame"/>
+      <origin xyz="${calibration.cam0.T_cam_imu[0][3]} ${calibration.cam0.T_cam_imu[1][3]} ${calibration.cam0.T_cam_imu[2][3]}" rpy="${atan2(calibration.cam0.T_cam_imu[2][1],calibration.cam0.T_cam_imu[2][2])} ${atan2(-calibration.cam0.T_cam_imu[2][0],sqrt(calibration.cam0.T_cam_imu[2][1]**2 + calibration.cam0.T_cam_imu[2][2]**2))} ${atan2(calibration.cam0.T_cam_imu[1][0],calibration.cam0.T_cam_imu[0][0])}"/>
+      <parent link="${prefix}_left_camera_optical_frame"/>
+      <child link="${prefix}_camera_imu_frame"/>
     </joint>
     <!-- Left/Depth camera -->
@@ -131,10 +131,10 @@
     </gazebo>
     <!-- IMU -->
-    <gazebo reference="${prefix}_imu_frame">
+    <gazebo reference="${prefix}_camera_imu_frame">
       <sensor type="imu" name="imu_sensor">
         <update_rate>${imu_frequency}</update_rate>
         <plugin filename="libgazebo_ros_imu_sensor.so" name="imu_plugin">
           <topicName>/${prefix}_camera/imu/data</topicName>
-          <frameName>${prefix}_imu_frame</frameName>
+          <frameName>${prefix}_camera_imu_frame</frameName>
           <updateRateHZ>${imu_frequency}</updateRateHZ>
           <gaussianNoise>0.0</gaussianNoise>
@@ -146,5 +146,5 @@
     </gazebo>
     <!-- MAGNETOMETER -->
-    <gazebo reference="${prefix}_imu_frame">
+    <gazebo reference="${prefix}_camera_imu_frame">
       <sensor type="magnetometer" name="magnetometer_sensor">
         <always_on>true</always_on>
@@ -172,5 +172,5 @@
         <plugin filename="libgazebo_ros_magnetometer_sensor.so" name="magnetometer_plugin">
           <topicName>/${prefix}_camera/imu/mag</topicName>
-          <frameName>${prefix}_imu_frame</frameName>
+          <frameName>${prefix}_camera_imu_frame</frameName>
           <updateRateHZ>50.0</updateRateHZ>
         </plugin>

Commit message: Add and set datum parameters to localization and simulation

File: src/sirius_description/urdf/cameras/oak-d-w.urdf.xacro (robot description, xacro)
@@ -2,5 +2,5 @@
 <robot xmlns:xacro="http://ros.org/wiki/xacro">
   <xacro:property name="optical_offset_x" value="-0.01" />
-  <xacro:macro name="oak-d-w" params="prefix:=oak-d-w package:=^ cameras:=^ cameras_inertial:=^ stereo_fps:=^|30 imu_frequency:=^|200 calibration:=^|${xacro.load_yaml('$(find sirius_cameras)/config/oak_d_w/kalibr_imucam_chain.yaml')}">
+  <xacro:macro name="oak-d-w" params="prefix:=oak-d-w package:=^ cameras:=^ cameras_inertial:=^ stereo_fps:=^|30 imu_frequency:=^|200 datum:=^ elevation:=^ year:=^ calibration:=^|${xacro.load_yaml('$(find sirius_cameras)/config/oak_d_w/kalibr_imucam_chain.yaml')}">
     <xacro:property name="baseline" value="${sqrt(calibration.cam1.T_cn_cnm1[0][3]**2 + calibration.cam1.T_cn_cnm1[1][3]**2 + calibration.cam1.T_cn_cnm1[2][3]**2)}"/>
     <link name="${prefix}_camera_center">
@@ -189,5 +189,5 @@
           <initialOrientationAsReference>false</initialOrientationAsReference>
           <xyzOffset>0 0.0 0.0</xyzOffset>
-          <rpyOffset>0.0 0.0 0.0</rpyOffset>
+          <rpyOffset>0 0 ${datum[2] * pi/180}</rpyOffset>
         </plugin>
       </sensor>
@@ -222,4 +222,11 @@
           <frameName>${prefix}_camera_imu_frame</frameName>
           <updateRateHZ>50.0</updateRateHZ>
+          <sphericalCoordinates>
+            <latitudeDeg>${datum[0]}</latitudeDeg>
+            <longitudeDeg>${datum[1]}</longitudeDeg>
+            <headingDeg>${datum[2]}</headingDeg>
+            <elevation>${elevation}</elevation>
+            <year>${year}</year>
+          </sphericalCoordinates>
         </plugin>
       </sensor>

File: src/sirius_description/urdf/sirius_2.urdf.xacro (robot description, xacro)
@@ -12,4 +12,10 @@
   <xacro:arg name="imu_frequency" default="200.0"/>
   <xacro:property name="imu_frequency" value="$(arg imu_frequency)" />
+  <xacro:arg name="datum" default="[50.878151, 20.642273, -35.59]"/>
+  <xacro:property name="datum" value="${$(arg datum)}" />
+  <xacro:arg name="elevation" default="0.0"/>
+  <xacro:property name="elevation" value="$(arg elevation)" />
+  <xacro:arg name="year" default=""/>
+  <xacro:property name="year" value="$(arg year)" />
   <xacro:property name="collisions" value="${xacro.load_yaml('sirius_2/sirius_2_collisions.yaml')}" />
   <xacro:property name="inertial" value="${xacro.load_yaml('sirius_2/sirius_2_inertial.yaml')}" />
@@ -151,4 +157,6 @@
       <topicName>ground_truth</topicName>
       <frameName>map</frameName>
+      <!-- <rpyOffset>0 0 ${-35.59 * pi/180}</rpyOffset> -->
+      <rpyOffset>0 0 ${datum[2] * pi/180}</rpyOffset>
     </plugin>
   </gazebo>

File: src/sirius_description/urdf/sirius_2/gnss.urdf.xacro (robot description, xacro)
@@ -3,5 +3,5 @@
      https://www.sparkfun.com/products/21801 -->
 <robot xmlns:xacro="http://wiki.ros.org/xacro">
-<xacro:macro name="gnss" params="material *gazebo_material package:=^ collisions:=^ inertial:=^">
+<xacro:macro name="gnss" params="material *gazebo_material package:=^ collisions:=^ inertial:=^ datum:=^ elevation:=^">
   <link name="gnss">
     <visual>
@@ -62,10 +62,10 @@
         <frameName>gnss</frameName>
         <updateRateHZ>20.0</updateRateHZ>
-        <spherical_coordinates>
-          <latitude_deg>50.87816930685754</latitude_deg>
-          <longitude_deg>20.64235537910024</longitude_deg>
-          <elevation>268</elevation>
-          <heading_deg>-45</heading_deg>
-        </spherical_coordinates>
+        <sphericalCoordinates>
+            <latitudeDeg>${datum[0]}</latitudeDeg>
+            <longitudeDeg>${datum[1]}</longitudeDeg>
+            <headingDeg>${datum[2]}</headingDeg>
+            <elevation>${elevation}</elevation>
+        </sphericalCoordinates>
       </plugin>
     </sensor>
