Commit message: Sensor fusion (#14)
* add gazebo_ros_magnetometer_sensor as submodule

* Add magnetometer plugin to zed and luxonis cameras

* add gaussian noise to magnetometers

* Add package for visual odometry

* open_vins partial config

* remove open_vins

* remove open_vins from submodules

* add morb_slam_ros

* Fix typos in zed urdf

* remove zed camera

* Change oak-d-w camera to (pseudo) grayscale

* Add oak_d_w calibration

* Match topic names with simulation

* Remove yaml version so xacro and ros can load file

* Add morb_slam configs for real camera and sim

* Load calibration data in camera urdf

* add viewer parameters to morb_slam_gazebo

* Add launch for morb_slam

* Real imu noise values

* sirius_cameras package, working simulation

* remove visualizer settings; update morb_slam_ros

* change oak_d_w camera namespace

* change tf from map to odom

* WIP: Fuse odom

* Oak-d pubilsh rotation vector and magnetometer

* Oak-d add rotation and magnetic covariance in launch

* Fix doubly defined parameters in gazebo launch

* Fuse wheel and imu (odom frame)

* add imu covariances

* Add gnss launch

* Set sensor fusion parameters in each sensor launch

* Fuse vz from wheel odometry

* add depthai-ros newer release as subpackage

* Change depthai branch to noetic

* Fix camera and imu orientation in imu

* publish robot tf

* hard iron calibration

* madgwick_filter

* Update magnetometer calibration

* add imu_filter_madgwick as dependency

* add depth camera to gazebo

* set use_sim_time param when starting gazego

* remove commented code (old imu)

* add navsat_transform_node

* add localization meta launch

* launch gnss in sirius_description package

* WIP: map sensor fusion

* WIP: map sensor fusion

* WIP: launch map sensof fusion in meta launch

* don't remove gravity vectror in madgwick

* Transform imu msg to base link frame

* WIP: GPS gazebo plugin

* Refactor package

* Optional spherical_coordinates parameter

* move gazebo gps plugin to src

* add ground turth gazebo

* Node for random traversal

* Calculating sensors noise variance from bag

* remove transform test

* Sort functions classes and variables

* Fork magnetometer plugin

* Refactor: raw pointers to smart, simplify warnings

* Refactor: raw pointers to smart, simplify warnings

* Add brief descriptions

* Simplify warning

* Rename parameters

* Don't convert gps lat, long and heading to rad

* Update gazebo ros magnetometer plugin

* use magnetometer in madgwick and reset mag bias

* Add and set datum parameters to localization and simulation

* Update marsyard map from 2020 to 2022

* Do convert gps lat long heading to rad

* Fix marsyard heading (rotate 180deg)

* Fix navsat_transform datum param

* add arg for datum in gnss launch

* Don't transform ground_truth for odometry twist if child_frame_id is empty

* add transform timeout for navsat_transform

* Rotate gps heading by 180deg (gazebo bug workaround)

* Modify p3d gazebo plugin to add map frame rpy offset

* Combine ekf config

* fix erc heading in launch files comments

* navsat_transform zero_altitude

* positionCovariance param in gazebo gps plugin for navsatfix msg

* imu and mag covariances

* fix gps heading again

* fix noiseVariance not handling lack of ground truth for early stamps

* Update frequency and process noise for map and odom ekf

* fix gnss pose in urdf

* Spawn robot at z=0 and update gazebo rviz

* Change rover velocity limits

* tweak ekf covariances

* Add camera focalLength for ros msg publisher

* Change 2d camera in depth plugin to color

* Change camera topic from depth plugin to rgb

* Add update rate to ros depth gazebo plugin

File: src/sirius_description/urdf/cameras/oak-d-w.urdf.xacro (robot description, xacro)
@@ -2,5 +2,5 @@
 <robot xmlns:xacro="http://ros.org/wiki/xacro">
   <xacro:property name="optical_offset_x" value="-0.01" />
-  <xacro:macro name="oak-d-w" params="prefix:=oak-d-w package:=^ cameras:=^ cameras_inertial:=^ stereo_fps:=^|30 imu_frequency:=^|200 calibration:=^|${xacro.load_yaml('$(find sirius_cameras)/config/oak_d_w/kalibr_imucam_chain.yaml')}">
+  <xacro:macro name="oak-d-w" params="prefix:=oak-d-w package:=^ cameras:=^ cameras_inertial:=^ stereo_fps:=^|30 imu_frequency:=^|200 datum:=^ elevation:=^ year:=^ calibration:=^|${xacro.load_yaml('$(find sirius_cameras)/config/oak_d_w/kalibr_imucam_chain.yaml')}">
     <xacro:property name="baseline" value="${sqrt(calibration.cam1.T_cn_cnm1[0][3]**2 + calibration.cam1.T_cn_cnm1[1][3]**2 + calibration.cam1.T_cn_cnm1[2][3]**2)}"/>
     <link name="${prefix}_camera_center">
@@ -26,5 +26,5 @@
     <link name="${prefix}_right_camera_frame" />
     <link name="${prefix}_right_camera_optical_frame"/>
-    <link name="${prefix}_imu_frame"/>
+    <link name="${prefix}_camera_imu_frame"/>
     <joint name="${prefix}_rgb_camera_optical_joint" type="fixed">
       <origin xyz="${optical_offset_x} 0 0" rpy="-${pi/2} 0.0 -${pi/2}"/>
@@ -38,6 +38,6 @@
     </joint>
     <joint name="${prefix}_left_camera_optical_joint" type="fixed">
-      <origin xyz="${optical_offset_x} 0 0" rpy="-${pi/2} 0.0 -${pi/2}"/>
-      <parent link="${prefix}_left_camera_frame"/>
+      <origin xyz="${calibration.cam1.T_cn_cnm1[0][3]} ${calibration.cam1.T_cn_cnm1[1][3]} ${calibration.cam1.T_cn_cnm1[2][3]}" rpy="${atan2(calibration.cam1.T_cn_cnm1[2][1],calibration.cam1.T_cn_cnm1[2][2])} ${atan2(-calibration.cam1.T_cn_cnm1[2][0],sqrt(calibration.cam1.T_cn_cnm1[2][1]**2 + calibration.cam1.T_cn_cnm1[2][2]**2))} ${atan2(calibration.cam1.T_cn_cnm1[1][0],calibration.cam1.T_cn_cnm1[0][0])}"/>
+      <parent link="${prefix}_right_camera_optical_frame"/>
       <child link="${prefix}_left_camera_optical_frame"/>
     </joint>
@@ -52,9 +52,9 @@
       <child link="${prefix}_right_camera_optical_frame"/>
     </joint>
-    <joint name="${prefix}_imu_frame_joint" type="fixed">
+    <joint name="${prefix}_camera_imu_frame_joint" type="fixed">
       <!-- IMU frame offset copied from ZED2 camera -->
-      <origin xyz="${calibration.cam0.T_imu_cam[0][3]} ${calibration.cam0.T_imu_cam[1][3]} ${calibration.cam0.T_imu_cam[2][3]}" rpy="${atan2(calibration.cam0.T_imu_cam[2][1],calibration.cam0.T_imu_cam[2][2])} ${atan2(-calibration.cam0.T_imu_cam[2][0],sqrt(calibration.cam0.T_imu_cam[2][1]**2 + calibration.cam0.T_imu_cam[2][2]**2))} ${atan2(calibration.cam0.T_imu_cam[1][0],calibration.cam0.T_imu_cam[0][0])}"/>
-      <parent link="${prefix}_left_camera_frame"/>
-      <child link="${prefix}_imu_frame"/>
+      <origin xyz="${calibration.cam0.T_cam_imu[0][3]} ${calibration.cam0.T_cam_imu[1][3]} ${calibration.cam0.T_cam_imu[2][3]}" rpy="${atan2(calibration.cam0.T_cam_imu[2][1],calibration.cam0.T_cam_imu[2][2])} ${atan2(-calibration.cam0.T_cam_imu[2][0],sqrt(calibration.cam0.T_cam_imu[2][1]**2 + calibration.cam0.T_cam_imu[2][2]**2))} ${atan2(calibration.cam0.T_cam_imu[1][0],calibration.cam0.T_cam_imu[0][0])}"/>
+      <parent link="${prefix}_left_camera_optical_frame"/>
+      <child link="${prefix}_camera_imu_frame"/>
     </joint>
     <!-- Left/Depth camera -->
@@ -82,6 +82,6 @@
           <lens>
             <intrinsics>
-            <fx>${calibration.cam0.intrinsics[0]}</fx>
-            <fy>${calibration.cam0.intrinsics[1]}</fy>
+            <fx>${(calibration.cam0.intrinsics[0] + calibration.cam0.intrinsics[1])/2}</fx>
+            <fy>${(calibration.cam0.intrinsics[0] + calibration.cam0.intrinsics[1])/2}</fy>
             <cx>${calibration.cam0.intrinsics[2]}</cx>
             <cy>${calibration.cam0.intrinsics[3]}</cy>
@@ -109,6 +109,6 @@
           <lens>
             <intrinsics>
-            <fx>${calibration.cam0.intrinsics[0]}</fx>
-            <fy>${calibration.cam0.intrinsics[1]}</fy>
+            <fx>${(calibration.cam0.intrinsics[0] + calibration.cam0.intrinsics[1])/2}</fx>
+            <fy>${(calibration.cam0.intrinsics[0] + calibration.cam0.intrinsics[1])/2}</fy>
             <cx>${calibration.cam0.intrinsics[2]}</cx>
             <cy>${calibration.cam0.intrinsics[3]}</cy>
@@ -127,24 +127,113 @@
           <rightFrameName>${prefix}_right_camera_optical_frame</rightFrameName>
           <hackBaseline>${baseline}</hackBaseline>
+          <focalLength>${(calibration.cam0.intrinsics[0] + calibration.cam0.intrinsics[1])/2}</focalLength>
+          <Cx>${calibration.cam0.intrinsics[2]}</Cx>
+          <Cy>${calibration.cam0.intrinsics[3]}</Cy>
+        </plugin>
+      </sensor>
+       <sensor type="depth" name="${prefix}_camera_depth">
+        <!-- Rectified images, Depth images, Point Clouds -->
+        <always_on>true</always_on>
+        <update_rate>${stereo_fps}</update_rate>
+        <visualize>false</visualize>
+        <camera name="/${prefix}_camera/depth">
+          <image>
+            <width>${calibration.cam0.resolution[0]}</width>
+            <height>${calibration.cam0.resolution[1]}</height>
+            <format>R8G8B8</format>
+          </image>
+          <clip>
+            <near>0.02</near>
+            <far>300</far>
+          </clip>
+          <noise>
+            <type>gaussian</type>
+            <mean>0.0</mean>
+            <stddev>0.007</stddev>
+          </noise>
+          <lens>
+            <intrinsics>
+            <fx>${(calibration.cam0.intrinsics[0] + calibration.cam0.intrinsics[1])/2}</fx>
+            <fy>${(calibration.cam0.intrinsics[0] + calibration.cam0.intrinsics[1])/2}</fy>
+            <cx>${calibration.cam0.intrinsics[2]}</cx>
+            <cy>${calibration.cam0.intrinsics[3]}</cy>
+            <s>0</s>
+            </intrinsics>
+            <scale_to_hfov>false</scale_to_hfov>
+          </lens>
+        </camera>
+        <plugin name="camera_controller" filename="libgazebo_ros_openni_kinect.so">
+          <alwaysOn>true</alwaysOn>
+          <updateRate>${stereo_fps}</updateRate>
+          <cameraName>/${prefix}_camera</cameraName>
+          <imageTopicName>rgb/image_raw_rgb</imageTopicName>
+          <cameraInfoTopicName>rgb/camera_info</cameraInfoTopicName>
+          <depthImageTopicName>depth/depth_registered</depthImageTopicName>
+          <depthImageInfoTopicName>depth/camera_info</depthImageInfoTopicName>
+          <pointCloudTopicName>point_cloud/cloud_registered</pointCloudTopicName>
+          <pointCloudCutoff>0.35</pointCloudCutoff>
+          <pointCloudCutoffMax>35.0</pointCloudCutoffMax>
+          <frameName>${prefix}_left_camera_optical_frame</frameName>
+          <baseline>${baseline}</baseline>
+          <focalLength>${(calibration.cam0.intrinsics[0] + calibration.cam0.intrinsics[1])/2}</focalLength>
+          <Cx>${calibration.cam0.intrinsics[2]}</Cx>
+          <Cy>${calibration.cam0.intrinsics[3]}</Cy>
+          <hackBaseline>0.0</hackBaseline>
         </plugin>
       </sensor>
     </gazebo>
     <!-- IMU -->
-    <gazebo reference="${prefix}_imu_frame">
+    <gazebo reference="${prefix}_camera_imu_frame">
       <sensor type="imu" name="imu_sensor">
+        <always_on>true</always_on>
         <update_rate>${imu_frequency}</update_rate>
+        <imu>
+          <angular_velocity>
+            <x>
+              <noise type="gaussian">
+                <stddev>0.0541052</stddev>
+              </noise>
+            </x>
+            <y>
+              <noise type="gaussian">
+                <stddev>0.0541052</stddev>
+              </noise>
+            </y>
+            <z>
+              <noise type="gaussian">
+                <stddev>0.0541052</stddev>
+              </noise>
+            </z>
+          </angular_velocity>
+          <linear_acceleration>
+            <x>
+              <noise type="gaussian">
+                <stddev>0.35</stddev>
+              </noise>
+            </x>
+            <y>
+              <noise type="gaussian">
+                <stddev>0.35</stddev>
+              </noise>
+            </y>
+            <z>
+              <noise type="gaussian">
+                <stddev>0.35</stddev>
+              </noise>
+            </z>
+          </linear_acceleration>
+        </imu>
         <plugin filename="libgazebo_ros_imu_sensor.so" name="imu_plugin">
           <topicName>/${prefix}_camera/imu/data</topicName>
-          <frameName>${prefix}_imu_frame</frameName>
+          <frameName>${prefix}_camera_imu_frame</frameName>
           <updateRateHZ>${imu_frequency}</updateRateHZ>
-          <gaussianNoise>0.0</gaussianNoise>
           <initialOrientationAsReference>false</initialOrientationAsReference>
           <xyzOffset>0 0.0 0.0</xyzOffset>
-          <rpyOffset>0.0 0.0 0.0</rpyOffset>
+          <rpyOffset>0 0 ${datum[2] * pi/180}</rpyOffset>
         </plugin>
       </sensor>
     </gazebo>
     <!-- MAGNETOMETER -->
-    <gazebo reference="${prefix}_imu_frame">
+    <gazebo reference="${prefix}_camera_imu_frame">
       <sensor type="magnetometer" name="magnetometer_sensor">
         <always_on>true</always_on>
@@ -153,18 +242,15 @@
           <x>
             <noise type="gaussian">
-              <mean>0.0</mean>
-              <stddev>5e-7</stddev>
+              <stddev>1.4e-6</stddev>
             </noise>
           </x>
           <y>
             <noise type="gaussian">
-              <mean>0.0</mean>
-              <stddev>5e-7</stddev>
+              <stddev>1.4e-6</stddev>
             </noise>
           </y>
           <z>
             <noise type="gaussian">
-              <mean>0.0</mean>
-              <stddev>5e-7</stddev>
+              <stddev>1.4e-6</stddev>
             </noise>
           </z>
@@ -172,6 +258,13 @@
         <plugin filename="libgazebo_ros_magnetometer_sensor.so" name="magnetometer_plugin">
           <topicName>/${prefix}_camera/imu/mag</topicName>
-          <frameName>${prefix}_imu_frame</frameName>
+          <frameName>${prefix}_camera_imu_frame</frameName>
           <updateRateHZ>50.0</updateRateHZ>
+          <sphericalCoordinates>
+            <latitudeDeg>${datum[0]}</latitudeDeg>
+            <longitudeDeg>${datum[1]}</longitudeDeg>
+            <headingDeg>${datum[2]}</headingDeg>
+            <elevation>${elevation}</elevation>
+            <year>${year}</year>
+          </sphericalCoordinates>
         </plugin>
       </sensor>

File: src/sirius_description/urdf/sirius_2.urdf.xacro (robot description, xacro)
@@ -12,4 +12,10 @@
   <xacro:arg name="imu_frequency" default="200.0"/>
   <xacro:property name="imu_frequency" value="$(arg imu_frequency)" />
+  <xacro:arg name="datum" default="[50.878151, 20.642273, 144.41]"/>
+  <xacro:property name="datum" value="${$(arg datum)}" />
+  <xacro:arg name="elevation" default="0.0"/>
+  <xacro:property name="elevation" value="$(arg elevation)" />
+  <xacro:arg name="year" default=""/>
+  <xacro:property name="year" value="$(arg year)" />
   <xacro:property name="collisions" value="${xacro.load_yaml('sirius_2/sirius_2_collisions.yaml')}" />
   <xacro:property name="inertial" value="${xacro.load_yaml('sirius_2/sirius_2_inertial.yaml')}" />
@@ -18,4 +24,5 @@
   <xacro:include filename="materials.urdf.xacro" />
   <xacro:include filename="sirius_2/indicator_light.urdf.xacro" />
+  <xacro:include filename="sirius_2/gnss.urdf.xacro" />
   <xacro:include filename="sirius_2/platform.urdf.xacro" />
   <xacro:include filename="cameras/hp_4310.urdf.xacro" />
@@ -66,4 +73,7 @@
     <xacro:blue_t/>
   </xacro:indicator_light>
+  <xacro:gnss material="light_gray">
+    <xacro:light_gray/>
+  </xacro:gnss>
   <xacro:hp_4310 prefix="front_mast" material="black">
     <xacro:black/>
@@ -117,4 +127,9 @@
     <origin xyz="${params['blue_indicator_light_xyz']}" rpy="0 0 ${pi}"/>
   </joint>
+  <joint name="base_to_gnss" type="fixed">
+    <parent link="base_link"/>
+    <child link="gnss"/>
+    <origin xyz="${params['gnss_xyz']}" rpy="0 0 0"/>
+  </joint>
   <joint name="base_to_front_mast_camera" type="fixed">
     <parent link="main_platform"/>
@@ -136,4 +151,12 @@
       <robotNamespace>/</robotNamespace>
     </plugin>
+    <plugin name="p3d_plugin" filename="libsirius_gazebo_ros_p3d.so">
+      <alwaysOn>true</alwaysOn>
+      <updateRate>100.0</updateRate>
+      <bodyName>base_link</bodyName>
+      <topicName>ground_truth</topicName>
+      <frameName>map</frameName>
+      <frameRpyOffset>0 0 ${datum[2] * pi/180}</frameRpyOffset>
+    </plugin>
   </gazebo>
 </robot>
