Commit message: Update platform model

File: src/sirius_description/urdf/cameras/oak-d-w.urdf.xacro (robot description, xacro)
@@ -6,8 +6,11 @@
     <link name="${prefix}_camera_center">
       <visual>
+      <material name="oak-d-w-material">
+            <color rgba="0.35 0.35 0.35 1"/>
+      </material>
         <geometry>
           <mesh filename="package://${package}/meshes/cameras/OAK-D-W.stl"/>
         </geometry>
-        <origin xyz="${cameras['oak-d-w_thickness']/2} 0 0" rpy="-${pi/2} ${pi} -${pi/2}"/>
+        <origin xyz="${-cameras['oak-d-w_thickness']/2} 0 0" rpy="-${pi/2} ${pi} ${pi/2}"/>
       </visual>
       <collision>
@@ -270,4 +273,14 @@
       </sensor>
     </gazebo>
+    <gazebo reference="${prefix}_camera_center">
+        <visual>
+          <material>
+            <ambient>0.25 0.25 0.25 1</ambient>
+            <diffuse>0.25 0.25 0.25 1</diffuse>
+            <specular>0 0 0 1</specular>
+            <emissive>0.0 0.0 0.0 0.0</emissive>
+          </material>
+        </visual>
+    </gazebo>
   </xacro:macro>
 </robot>

File: src/sirius_description/urdf/materials.urdf.xacro (robot description, xacro)
@@ -1,27 +1,36 @@
 <robot xmlns:xacro="http://wiki.ros.org/xacro">
-  <material name="yellow_t">
-    <color rgba=".75 .75 0 0.5" />
-  </material>
-  <material name="blue_t">
-    <color rgba="0 0 1 0.5" />
-  </material>
-  <material name="bronze">
-    <color rgba=".839 .471 .369 1" />
-  </material>
-  <material name="gold">
-    <color rgba=".910 .443 .031 1" />
-  </material>
-  <material name="gray">
-    <color rgba=".796 .824 .937 1" />
-  </material>
-  <material name="light_gray">
-        <color rgba="0.25 0.25 0.25 1"/>
-  </material>
-  <material name="black">
-    <color rgba="0 0 0 1" />
-  </material>
-  <material name="green">
-    <color rgba="0 1 0 1" />
-  </material>
+  <!-- URDF colors -->
+  <material name="black">       <color rgba="0 0 0 1" /></material>
+  <material name="dark_bronze"> <color rgba=".36 .29 .22 1" /></material>
+  <material name="dark_gray">   <color rgba="0.35 0.35 0.35 1"/></material>
+  <material name="gold">        <color rgba=".910 .443 .031 1" /></material>
+  <material name="gray">        <color rgba=".796 .824 .937 1" /></material>
+  <material name="green">       <color rgba="0 1 0 1" /></material>
+  <material name="white">       <color rgba="1 1 1 1" /></material>
+  <!-- Gazebo colors -->
+  <xacro:macro name="black">
+    <material>
+      <ambient>0 0 0 1</ambient>
+      <diffuse>0 0 0 1</diffuse>
+      <specular>0 0 0 1</specular>
+      <emissive>0.0 0.0 0.0 0.0</emissive>
+    </material>
+  </xacro:macro>
+  <xacro:macro name="dark_bronze">
+    <material>
+      <ambient>.36 .29 .22 1</ambient>
+      <diffuse>.36 .29 .22 1</diffuse>
+      <specular>1 1 1 1</specular>
+      <emissive>0.0 0.0 0.0 0.0</emissive>
+    </material>
+  </xacro:macro>
+  <xacro:macro name="dark_gray">
+    <material>
+      <ambient>0.25 0.25 0.25 1</ambient>
+      <diffuse>0.25 0.25 0.25 1</diffuse>
+      <specular>0 0 0 1</specular>
+      <emissive>0.0 0.0 0.0 0.0</emissive>
+    </material>
+  </xacro:macro>
   <xacro:macro name="gold">
     <material>
@@ -40,43 +49,19 @@
     </material>
   </xacro:macro>
-  <xacro:macro name="bronze">
+  <xacro:macro name="green">
     <material>
-      <ambient>.9 .5 .4 1</ambient>
-      <diffuse>.9 .5 .4 1</diffuse>
-      <specular>1 1 1 1</specular>
-      <emissive>0.0 0.0 0.0 0.0</emissive>
-    </material>
-  </xacro:macro>
-  <xacro:macro name="yellow_t">
-    <material>
-      <ambient>1 1 0 0.5</ambient>
-      <diffuse>1 1 0 0.5</diffuse>
-      <specular>1 1 1 0.5</specular>
-      <emissive>0.0 0.0 0.0 0.0</emissive>
-    </material>
-  </xacro:macro>
-  <xacro:macro name="blue_t">
-    <material>
-      <ambient>0 0 1 0.5</ambient>
-      <diffuse>0 0 1 0.5</diffuse>
-      <specular>0 0 1 0.5</specular>
-      <emissive>0.0 0.0 0.0 0.0</emissive>
-    </material>
-  </xacro:macro>
-  <xacro:macro name="light_gray">
-    <material>
-      <ambient>0.25 0.25 0.25 1</ambient>
-      <diffuse>0.25 0.25 0.25 1</diffuse>
-      <specular>0.5 0.5 0.5 1</specular>
-      <emissive>0.0 0.0 0.0 0.0</emissive>
-    </material>
-  </xacro:macro>
-  <xacro:macro name="black">
-    <material>
-      <ambient>0 0 0 1</ambient>
-      <diffuse>0 0 0 1</diffuse>
+      <ambient>0 1 0 1</ambient>
+      <diffuse>0 1 0 1</diffuse>
       <specular>0 0 0 1</specular>
       <emissive>0.0 0.0 0.0 0.0</emissive>
     </material>
   </xacro:macro>
+  <xacro:macro name="white">
+    <material>
+      <ambient>0.8 0.8 0.8 1</ambient>
+      <diffuse>0.8 0.8 0.8 1</diffuse>
+      <specular>0.1 0.1 0.1 1</specular>
+      <emissive>0.0 0.0 0.0 0.0</emissive>
+    </material>
+  </xacro:macro>
 </robot>

File: src/sirius_description/urdf/sirius_2.urdf.xacro (robot description, xacro)
@@ -2,59 +2,75 @@
 <robot xmlns:xacro="http://www.ros.org/wiki/xacro" name="sirius_2">
   <xacro:property name="package" value="sirius_description" />
-  <xacro:property name="params" value="${xacro.load_yaml('sirius_2.yaml')}" />
+  <!-- User arguments -->
   <xacro:arg name="calibration_path" default=""/>
+  <xacro:arg name="datum" default="[50.878151, 20.642273, 144.41]"/>
+  <xacro:arg name="elevation" default="0.0"/>
+  <xacro:arg name="imu_frequency" default="200.0"/>
+  <xacro:arg name="joint_prefix" default=""/>
+  <xacro:arg name="link_prefix" default=""/>
+  <xacro:arg name="robot_ns" default=""/>
+  <xacro:arg name="stereo_fps" default="30"/>
+  <xacro:arg name="year" default=""/>
+  <!-- Parse arguments -->
   <xacro:property name="calibration_path" value="$(arg calibration_path)" />
   <xacro:if value="${calibration_path != ''}">
     <xacro:property name="calibration" value="${xacro.load_yaml(calibration_path)}" />
   </xacro:if>
-  <xacro:arg name="stereo_fps" default="30"/>
+  <xacro:property name="datum" value="${$(arg datum)}" />
+  <xacro:property name="elevation" value="$(arg elevation)" />
+  <xacro:property name="imu_frequency" value="$(arg imu_frequency)" />
   <xacro:property name="stereo_fps" value="$(arg stereo_fps)" />
-  <xacro:arg name="imu_frequency" default="200.0"/>
-  <xacro:property name="imu_frequency" value="$(arg imu_frequency)" />
-  <xacro:arg name="datum" default="[50.878151, 20.642273, 144.41]"/>
-  <xacro:property name="datum" value="${$(arg datum)}" />
-  <xacro:arg name="elevation" default="0.0"/>
-  <xacro:property name="elevation" value="$(arg elevation)" />
-  <xacro:arg name="year" default=""/>
   <xacro:property name="year" value="$(arg year)" />
+  <xacro:property name="link_prefix" value="$(arg link_prefix)" />
+  <xacro:property name="robot_ns" value="$(arg robot_ns)" />
+  <xacro:property name="joint_prefix" value="$(arg joint_prefix)" />
+  <!-- Load model parameters -->
+  <xacro:property name="params" value="${xacro.load_yaml('sirius_2.yaml')}" />
+  <xacro:property name="cameras" value="${xacro.load_yaml('cameras/cameras.yaml')}" />
   <xacro:property name="collisions" value="${xacro.load_yaml('sirius_2/sirius_2_collisions.yaml')}" />
+  <!-- Load inertial parameters -->
   <xacro:property name="inertial" value="${xacro.load_yaml('sirius_2/sirius_2_inertial.yaml')}" />
-  <xacro:property name="cameras" value="${xacro.load_yaml('cameras/cameras.yaml')}" />
   <xacro:property name="cameras_inertial" value="${xacro.load_yaml('cameras/cameras_inertial.yaml')}" />
+  <!-- Load materials -->
   <xacro:include filename="materials.urdf.xacro" />
+  <!-- Load subcomponents xacro -->
   <xacro:include filename="sirius_2/indicator_light.urdf.xacro" />
-  <xacro:include filename="sirius_2/gnss.urdf.xacro" />
   <xacro:include filename="sirius_2/platform.urdf.xacro" />
+  <!-- Load sensors and cameras xacro -->
   <xacro:include filename="cameras/hp_4310.urdf.xacro" />
   <xacro:include filename="cameras/oak-d-w.urdf.xacro" />
-  <xacro:property name="link_prefix" value=""/>
-  <xacro:property name="robot_ns" value=""/>
-  <xacro:property name="joint_prefix" value=""/>
-  <xacro:macro name="drive_system" params="reflect:=false prefix:='' params:=^ direction:=1">
+  <xacro:include filename="sirius_2/gnss.urdf.xacro" />
+  <!-- Macro to simplify joint definition -->
+  <xacro:macro name="joint" params="name:='' type:='fixed' parent:='base_link' child:='' xyz:='0 0 0' rpy:='0 0 0' axis:='0 0 1' limit_effort:='0.0' limit_velocity:='0.0'">
+    <joint name="${name}" type="${type}">
+      <parent link="${parent}"/>
+      <child link="${child}"/>
+      <origin xyz="${xyz}" rpy="${rpy}"/>
+      <axis xyz="${axis}"/>
+      <xacro:if value="${type != 'fixed'}">
+        <limit effort="${limit_effort}" velocity="${limit_velocity}"/>
+      </xacro:if>
+    </joint>
+  </xacro:macro>
+  <!-- Macro to combine suspension and wheel -->
+  <xacro:macro name="drive_system" params="flip_x:=false flip_y:=false prefix:='' params:=^">
     <xacro:include filename="sirius_2/suspension.urdf.xacro" />
     <xacro:include filename="sirius_2/wheel.urdf.xacro" />
-    <xacro:include filename="sirius_2/drive_train.urdf.xacro" />
-    <xacro:suspension prefix="${prefix}" material="bronze">
-      <xacro:bronze/>
+    <xacro:suspension prefix="${prefix}" material="dark_bronze" flip="${flip_y}">
+      <xacro:dark_bronze/>
     </xacro:suspension>
-    <xacro:drive_train prefix="${prefix}" material="gray">
-      <xacro:gray/>
-    </xacro:drive_train>
-    <xacro:wheel prefix="${prefix}" material="gold">
-      <xacro:gold/>
+    <xacro:wheel prefix="${prefix}" material="dark_gray" material_rim="white" flip="${flip_x}">
+      <xacro:dark_gray/>
+      <xacro:white/>
     </xacro:wheel>
-    <joint name="${prefix}_suspension_to_${prefix}_drive_train" type="fixed">
-      <parent link="${prefix}_suspension"/>
-      <child link="${prefix}_drive_train"/>
-      <origin xyz="${params['suspension_separation_x']/2 - params['wheel_base']/2} ${-reflect*params['suspension_thickness']} ${-params['suspension_height']}" rpy="0 0 ${reflect*pi}"/>
-      <axis xyz="0 0 1"/>
-    </joint>
-    <joint name="${prefix}_wheel_joint" type="continuous">
-      <parent link="${prefix}_drive_train"/>
-      <child link="${prefix}_wheel"/>
-      <origin xyz="0 ${params['track']/2 - params['suspension_thickness']/2 - params['suspension_separation_y']/2} 0"/>
-      <axis xyz="0 ${-(1-2*reflect) * direction} 0"/>
-      <limit effort="18.0" velocity="8.0"/>
-    </joint>
+    <xacro:joint  name="${prefix}_wheel_joint"
+                  type="continuous"
+                  parent="${prefix}_suspension"
+                  child="${prefix}_wheel"
+                  xyz="${(1 - 2 * flip_y)  * (params['wheel_base'] - params['suspension_separation_x'])/2 } ${(1 - 2 * flip_x)  * (params['track'] - params['suspension_separation_y'])/2} ${-params['suspension_height']}"
+                  rpy="0 0 0"
+                  axis="0 1 0"
+                  limit_effort="18.0"
+                  limit_velocity="8.0" />
     <transmission name="${prefix}_wheel_transmission">
       <type>transmission_interface/SimpleTransmission</type>
@@ -67,88 +83,71 @@
     </transmission>
   </xacro:macro>
-  <xacro:indicator_light prefix="yellow" material="yellow_t">
-    <xacro:yellow_t/>
-  </xacro:indicator_light>
-  <xacro:indicator_light prefix="blue" material="blue_t">
-    <xacro:blue_t/>
-  </xacro:indicator_light>
-  <xacro:gnss material="light_gray">
-    <xacro:light_gray/>
-  </xacro:gnss>
+  <!-- Define subcomponents links -->
+  <link name="base_link" />
+  <xacro:platform material="white">
+    <xacro:white/>
+  </xacro:platform>
+  <xacro:drive_system prefix="left_back" flip_y="true" />
+  <xacro:drive_system prefix="left_front" />
+  <xacro:drive_system prefix="right_back" flip_x="true" flip_y="true"/>
+  <xacro:drive_system prefix="right_front"  flip_x="true"/>
+  <xacro:indicator_light material="gray"><xacro:gray/></xacro:indicator_light>
+  <!-- Define sensors and cameras links -->
+  <xacro:hp_4310 prefix="back_mast" material="black">
+    <xacro:black/>
+  </xacro:hp_4310>
   <xacro:hp_4310 prefix="front_mast" material="black">
     <xacro:black/>
   </xacro:hp_4310>
-  <xacro:hp_4310 prefix="back_mast" material="black">
-    <xacro:black/>
-  </xacro:hp_4310>
   <xacro:oak-d-w prefix="front"/>
-  <xacro:drive_system prefix="right_front" />
-  <xacro:drive_system reflect="true" prefix="right_back" direction="-1"/>
-  <xacro:drive_system reflect="true" prefix="left_front" />
-  <xacro:drive_system prefix="left_back" direction="-1"/>
-  <link name="base_link" />
-  <xacro:platform prefix="main" material="gray">
-    <xacro:gray/>
-  </xacro:platform>
-  <joint name="base_link_to_main_platform" type="fixed">
-    <parent link="base_link"/>
-    <child link="main_platform"/>
-    <origin xyz="0 0 ${params['wheel_radius'] + params['suspension_height'] - params['suspension_z']}" rpy="0 0 ${pi}"/>
-    <axis xyz="0 0 1"/>
-  </joint>
-  <joint name="base_right_front_suspension" type="fixed">
-    <parent link="main_platform"/>
-    <child link="right_front_suspension"/>
-    <origin xyz="${-params['suspension_separation_x']/2} ${params['suspension_separation_y']/2 + params['suspension_thickness']/2} ${params['suspension_z']}" rpy="0 0 0"/>
-  </joint>
-  <joint name="base_right_back_suspension" type="fixed">
-    <parent link="main_platform"/>
-    <child link="right_back_suspension"/>
-    <origin xyz="${params['suspension_separation_x']/2} ${params['suspension_separation_y']/2 - params['suspension_thickness']/2} ${params['suspension_z']}" rpy="0 0 ${pi}"/>
-  </joint>
-  <joint name="base_left_front_suspension" type="fixed">
-    <parent link="main_platform"/>
-    <child link="left_front_suspension"/>
-    <origin xyz="${-params['suspension_separation_x']/2} ${-params['suspension_separation_y']/2 + params['suspension_thickness']/2} ${params['suspension_z']}"/>
-  </joint>
-  <joint name="base_left_back_suspension" type="fixed">
-    <parent link="main_platform"/>
-    <child link="left_back_suspension"/>
-    <origin xyz="${params['suspension_separation_x']/2} ${-params['suspension_separation_y']/2 - params['suspension_thickness']/2} ${params['suspension_z']}" rpy="0 0 ${pi}"/>
-  </joint>
-  <joint name="base_to_yellow_indicator_light" type="fixed">
-    <parent link="main_platform"/>
-    <child link="yellow_indicator_light"/>
-    <origin xyz="${params['yellow_indicator_light_xyz']}" rpy="0 0 ${pi}"/>
-  </joint>
-  <joint name="base_to_blue_indicator_light" type="fixed">
-    <parent link="main_platform"/>
-    <child link="blue_indicator_light"/>
-    <origin xyz="${params['blue_indicator_light_xyz']}" rpy="0 0 ${pi}"/>
-  </joint>
-  <joint name="base_to_gnss" type="fixed">
-    <parent link="base_link"/>
-    <child link="gnss"/>
-    <origin xyz="${params['gnss_xyz']}" rpy="0 0 0"/>
-  </joint>
-  <joint name="base_to_front_mast_camera" type="fixed">
-    <parent link="main_platform"/>
-    <child link="front_mast_camera"/>
-    <origin xyz="${params['front_mast_camera_xyz']}" rpy="${params['front_mast_camera_rpy']}"/>
-  </joint>
-  <joint name="base_to_back_mast_camera" type="fixed">
-    <parent link="main_platform"/>
-    <child link="back_mast_camera"/>
-    <origin xyz="${params['back_mast_camera_xyz']}" rpy="${params['back_mast_camera_rpy']}"/>
-  </joint>
-  <joint name="base_to_front_camera" type="fixed">
-    <parent link="main_platform"/>
-    <child link="front_camera_center"/>
-    <origin xyz="${params['front_camera_xyz']}" rpy="${params['front_camera_rpy']}"/>
-  </joint>
+  <xacro:gnss material="gray"><xacro:gray/></xacro:gnss>
+  <!-- Define subcomponents joints -->
+  <xacro:joint name="base_link_to_platform"
+               child="platform"
+               xyz="0 0 ${params['wheel_radius'] + params['suspension_height'] - params['suspension_z']}" />
+  <xacro:joint name="base_to_left_back_suspension"
+               parent="platform"
+               child="left_back_suspension"
+               xyz="${-params['suspension_separation_x']/2} ${params['suspension_separation_y']/2} ${params['suspension_z']}" />
+  <xacro:joint name="base_to_left_front_suspension"
+               parent="platform"
+               child="left_front_suspension"
+               xyz="${params['suspension_separation_x']/2} ${params['suspension_separation_y']/2} ${params['suspension_z']}" />
+  <xacro:joint name="base_to_right_back_suspension"
+               parent="platform"
+               child="right_back_suspension"
+               xyz="${-params['suspension_separation_x']/2} ${-params['suspension_separation_y']/2} ${params['suspension_z']}" />
+  <xacro:joint name="base_to_right_front_suspension"
+               parent="platform"
+               child="right_front_suspension"
+               xyz="${params['suspension_separation_x']/2} ${-params['suspension_separation_y']/2} ${params['suspension_z']}" />
+  <xacro:joint name="base_to_indicator_light"
+               parent="platform"
+               child="indicator_light"
+               xyz="${params['indicator_light_xyz']}"/>
+  <!-- Define sensors and cameras joints -->
+  <xacro:joint name="base_to_front_mast_camera"
+               parent="platform"
+               child="front_mast_camera"
+               xyz="${params['front_mast_camera_xyz']}"
+               rpy="${params['front_mast_camera_rpy']}"/>
+  <xacro:joint name="base_to_back_mast_camera"
+               parent="platform"
+               child="back_mast_camera"
+               xyz="${params['back_mast_camera_xyz']}"
+               rpy="${params['back_mast_camera_rpy']}"/>
+  <xacro:joint name="base_to_front_camera"
+               parent="platform"
+               child="front_camera_center"
+               xyz="${params['front_camera_xyz']}"
+               rpy="${params['front_camera_rpy']}"/>
+  <xacro:joint name="base_to_gnss" child="gnss" xyz="${params['gnss_xyz']}" />
+  <!-- Gazebo plugins -->
   <gazebo>
+    <!-- hardware interfaces for wheels -->
     <plugin name="gazebo_ros_control" filename="libgazebo_ros_control.so">
       <robotNamespace>/</robotNamespace>
     </plugin>
+    <!-- Ground truth pose for base_link -->
     <plugin name="p3d_plugin" filename="libsirius_gazebo_ros_p3d.so">
       <alwaysOn>true</alwaysOn>

File: src/sirius_description/urdf/sirius_2/indicator_light.urdf.xacro (robot description, xacro)
@@ -1,6 +1,6 @@
 <?xml version="1.0" encoding="utf-8"?>
 <robot xmlns:xacro="http://wiki.ros.org/xacro">
-<xacro:macro name="indicator_light" params="prefix material *gazebo_material package:=^ collisions:=^ inertial:=^">
-  <link name="${prefix}_indicator_light">
+<xacro:macro name="indicator_light" params="material prefix:='' *gazebo_material package:=^ collisions:=^ inertial:=^">
+  <link name="${prefix + '_' if prefix else prefix}indicator_light">
     <visual>
       <material name="${material}">
@@ -21,5 +21,5 @@
     </collision>
   </link>
-  <gazebo reference="${prefix}_indicator_light">
+  <gazebo reference="${prefix + '_' if prefix else prefix}indicator_light">
       <visual>
         <xacro:insert_block name="gazebo_material" />
