Commit message: Update platform model

File: src/sirius_description/urdf/sirius_2/platform.urdf.xacro (robot description, xacro)
@@ -1,5 +1,5 @@
 <robot xmlns:xacro="http://wiki.ros.org/xacro">
-<xacro:macro name="platform" params="prefix material *gazebo_material package:=^ collisions:=^ params:=^ inertial:=^">
-    <link name="${prefix}_platform">
+<xacro:macro name="platform" params="material prefix:='' *gazebo_material  package:=^ collisions:=^ params:=^ inertial:=^">
+    <link name="${prefix + '_' if prefix else prefix}platform">
       <visual>
         <material name="${material}"/>
@@ -9,4 +9,5 @@
       </visual>
       <inertial>
+        <origin xyz="0 0 0" rpy="0 0 ${pi}"/>
         <mass value="${inertial['platform_mass']}"/>
         <inertia ixx="${inertial['platform_inertia']['ixx']}" ixy="${inertial['platform_inertia']['ixy']}" ixz="${inertial['platform_inertia']['ixz']}" iyy="${inertial['platform_inertia']['iyy']}" iyz="${inertial['platform_inertia']['iyz']}" izz="${inertial['platform_inertia']['izz']}"/>
@@ -14,5 +15,5 @@
       <collision>
         <geometry>
-          <box size="${collisions['platform_box_length']} ${params['suspension_separation_y'] - params['suspension_thickness']*1.5} ${collisions['platform_height']}"/>
+          <box size="${collisions['platform_box_length']} ${params['suspension_separation_y'] - collisions['suspension_thickness']*1.5} ${collisions['platform_height']}"/>
         </geometry>
         <origin xyz="${collisions['platform_box_x']} 0 ${collisions['platform_height']/2}" />
@@ -20,23 +21,24 @@
       <collision>
         <geometry>
-          <box size="${collisions['platform_height'] + collisions['platform_profile_size']*1.25} ${params['suspension_separation_y'] - params['suspension_thickness']*1.5} ${collisions['platform_profile_size']}"/>
+          <box size="${collisions['platform_height']/tan(collisions['platform_angle'] * pi / 180) - collisions['platform_profile_size']} ${params['suspension_separation_y'] - collisions['suspension_thickness']*1.5} ${collisions['platform_profile_size']}"/>
         </geometry>
-        <origin xyz="-${collisions['platform_height'] + collisions['platform_box_x'] - collisions['platform_box_length']/2} 0 ${collisions['platform_height'] - collisions['platform_profile_size']/2}" />
+        <origin xyz="${collisions['platform_height']/(tan(collisions['platform_angle'] * pi / 180)*2) - collisions['platform_profile_size']/2 + collisions['platform_box_x'] + collisions['platform_box_length']/2} 0 ${collisions['platform_height'] - collisions['platform_profile_size']/2}" />
       </collision>
       <collision>
         <geometry>
-          <box size="${collisions['platform_height']*1.5 - collisions['platform_profile_size']} ${collisions['platform_profile_size']} ${collisions['platform_profile_size']}"/>
+          <box size="${collisions['platform_height']/cos(collisions['platform_angle'] * pi / 180) - collisions['platform_profile_size']/2} ${collisions['platform_profile_size']} ${collisions['platform_profile_size']}"/>
         </geometry>
-        <origin xyz="-${collisions['platform_height'] + collisions['platform_box_x'] - collisions['platform_box_length']/2} ${params['suspension_separation_x']/2 + collisions['platform_profile_size']*0.8} ${collisions['platform_height']/2}" rpy="0 ${collisions['platform_angle']} 0"/>
+        <origin xyz="${collisions['platform_box_x'] + collisions['platform_box_length']/2 + collisions['platform_height']/(tan(collisions['platform_angle'] * pi / 180) * 2) - collisions['platform_profile_size']/2} ${params['suspension_separation_y']/2 - collisions['platform_profile_size']*1.8} ${collisions['platform_height']/2 + collisions['platform_profile_size']/6}" rpy="0 ${-collisions['platform_angle'] * pi / 180} 0"/>
       </collision>
       <collision>
         <geometry>
-          <box size="${collisions['platform_height']*1.5 - collisions['platform_profile_size']} ${collisions['platform_profile_size']} ${collisions['platform_profile_size']}"/>
+          <box size="${collisions['platform_height']/cos(collisions['platform_angle'] * pi / 180) - collisions['platform_profile_size']/2} ${collisions['platform_profile_size']} ${collisions['platform_profile_size']}"/>
         </geometry>
-        <origin xyz="-${collisions['platform_height'] + collisions['platform_box_x'] - collisions['platform_box_length']/2} ${-params['suspension_separation_x']/2 - collisions['platform_profile_size']*0.8} ${collisions['platform_height']/2}" rpy="0 ${collisions['platform_angle']} 0"/>
+        <origin xyz="${collisions['platform_box_x'] + collisions['platform_box_length']/2 + collisions['platform_height']/(tan(collisions['platform_angle'] * pi / 180) * 2) - collisions['platform_profile_size']/2} ${-params['suspension_separation_y']/2 + collisions['platform_profile_size']*1.8} ${collisions['platform_height']/2 + collisions['platform_profile_size']/6}" rpy="0 ${-collisions['platform_angle'] * pi / 180} 0"/>
       </collision>
       <collision>
         <geometry>
-          <cylinder length="${collisions['platform_mast_height']}" radius="${collisions['platform_mast_radius']}"/>
+        <!-- ${collisions['platform_mast_radius']} -->
+          <box size="${collisions['platform_profile_size']} ${collisions['platform_profile_size']} ${collisions['platform_mast_height']}"/>
         </geometry>
         <origin xyz="${collisions['platform_mast_x']} ${collisions['platform_mast_y']} ${collisions['platform_mast_height']/2}" />
@@ -44,5 +46,5 @@
       <collision>
         <geometry>
-          <cylinder length="${collisions['platform_mast_height']}" radius="${collisions['platform_mast_radius']}"/>
+          <box size="${collisions['platform_profile_size']} ${collisions['platform_profile_size']} ${collisions['platform_mast_height']}"/>
         </geometry>
         <origin xyz="${collisions['platform_mast_x']} ${-collisions['platform_mast_y']} ${collisions['platform_mast_height']/2}" />
@@ -50,7 +52,7 @@
       <collision>
         <geometry>
-          <box size="0.028 ${collisions['platform_mast_y']*2} ${collisions['platform_mast_routers_height']}"/>
+          <box size="${collisions['platform_profile_size']} ${collisions['platform_mast_y']*2} ${collisions['platform_profile_size']}"/>
         </geometry>
-        <origin xyz="${collisions['platform_mast_x'] + collisions['platform_mast_radius']*2} 0 ${collisions['platform_mast_height'] - collisions['platform_mast_routers_height']/2}" />
+        <origin xyz="${collisions['platform_mast_x']} 0 ${collisions['platform_mast_height'] - collisions['platform_profile_size']*2.55}" />
       </collision>
       <collision>
@@ -60,12 +62,6 @@
         <origin xyz="${collisions['platform_mast_5g_xyz']}" />
       </collision>
-      <collision>
-        <geometry>
-          <cylinder length="${collisions['platform_mast_2g_length']}" radius="${collisions['platform_mast_2g_radius']}"/>
-        </geometry>
-        <origin xyz="${collisions['platform_mast_2g_xyz']}" />
-      </collision>
     </link>
-    <gazebo reference="${prefix}_platform">
+    <gazebo reference="${prefix + '_' if prefix else prefix}platform">
       <visual>
         <xacro:insert_block name="gazebo_material" />

File: src/sirius_description/urdf/sirius_2/suspension.urdf.xacro (robot description, xacro)
@@ -1,4 +1,4 @@
 <robot xmlns:xacro="http://wiki.ros.org/xacro">
-<xacro:macro name="suspension" params="prefix material *gazebo_material params:=^ package:=^ collisions:=^ inertial:=^">
+<xacro:macro name="suspension" params="prefix material *gazebo_material flip:=false params:=^ package:=^ collisions:=^ inertial:=^">
     <link name="${prefix}_suspension">
       <visual>
@@ -7,4 +7,5 @@
           <mesh filename="package://${package}/meshes/sirius_2/suspension.stl" scale="0.001 0.001 0.001"/>
         </geometry>
+        <origin xyz="0 0 0" rpy="0 0 ${pi if flip else 0}" />
       </visual>
       <inertial>
@@ -14,7 +15,7 @@
       <collision>
         <geometry>
-          <box size="${collisions['suspension_width']} ${params['suspension_thickness']} ${collisions['suspension_length']}"/>
+          <box size="${collisions['suspension_width']} ${collisions['suspension_thickness']} ${collisions['suspension_length']}"/>
         </geometry>
-        <origin xyz="${-params['wheel_base']/4 + params['suspension_separation_x']/4 - collisions['suspension_x_shift']} ${-params['suspension_thickness']/2} ${-params['suspension_height']/2}" rpy="0 ${collisions['suspension_angle']} 0" />
+        <origin xyz="${(1 - 2 * flip) * (params['wheel_base']/4 - params['suspension_separation_x']/4 + collisions['suspension_x_shift'])} 0 ${-params['suspension_height']/2}" rpy="0 ${collisions['suspension_angle'] * pi / 180} ${pi if flip else 0}" />
       </collision>
     </link>

File: src/sirius_description/urdf/sirius_2/wheel.urdf.xacro (robot description, xacro)
@@ -1,4 +1,4 @@
 <robot xmlns:xacro="http://wiki.ros.org/xacro">
-<xacro:macro name="wheel" params="prefix material *gazebo_material package:=^ params:=^ inertial:=^">
+<xacro:macro name="wheel" params="prefix material material_rim *gazebo_material **gazebo_material_rim flip:=false package:=^ params:=^ inertial:=^">
     <link name="${prefix}_wheel">
       <visual>
@@ -7,4 +7,5 @@
           <mesh filename="package://${package}/meshes/sirius_2/wheel.stl" scale="0.001 0.001 0.001"/>
         </geometry>
+        <origin xyz="0 0 0" />
       </visual>
       <inertial>
@@ -19,4 +20,23 @@
       </collision>
     </link>
+    <link name="${prefix}_wheel_rim">
+      <visual>
+        <material name="${material_rim}" />
+        <geometry>
+          <mesh filename="package://${package}/meshes/sirius_2/rim.stl" scale="0.001 0.001 0.001"/>
+        </geometry>
+      </visual>
+      <collision>
+        <geometry>
+          <cylinder length="${params['rim_width']}" radius="${params['wheel_radius'] * 0.8}"/>
+        </geometry>
+        <origin xyz="0 0 0" rpy="${pi/2} 0 0" />
+      </collision>
+    </link>
+    <joint name="${prefix}_wheel_to_rim" type="fixed">
+      <parent link="${prefix}_wheel"/>
+      <child link="${prefix}_wheel_rim"/>
+      <origin xyz="0 ${ (1 - 2*flip) * (params['wheel_width'] + params['rim_width'])/2} 0" />
+    </joint>
     <gazebo reference="${prefix}_wheel">
       <visual>
@@ -24,4 +44,9 @@
       </visual>
     </gazebo>
+    <gazebo reference="${prefix}_wheel_rim">
+      <visual>
+        <xacro:insert_block name="gazebo_material_rim" />
+      </visual>
+    </gazebo>
 </xacro:macro>
 </robot>

Commit message: Move properties to local scope

File: src/sirius_description/urdf/cameras/oak-d-w.urdf.xacro (robot description, xacro)
@@ -1,6 +1,6 @@
 <?xml version="1.0"?>
 <robot xmlns:xacro="http://ros.org/wiki/xacro">
-  <xacro:property name="optical_offset_x" value="-0.01" />
   <xacro:macro name="oak-d-w" params="prefix:=oak-d-w package:=^ cameras:=^ cameras_inertial:=^ stereo_fps:=^|30 imu_frequency:=^|200 datum:=^ elevation:=^ year:=^ calibration:=^|${xacro.load_yaml('$(find sirius_cameras)/config/oak_d_w/kalibr_imucam_chain.yaml')}">
+    <xacro:property name="optical_offset_x" value="-0.01" />
     <xacro:property name="baseline" value="${sqrt(calibration.cam1.T_cn_cnm1[0][3]**2 + calibration.cam1.T_cn_cnm1[1][3]**2 + calibration.cam1.T_cn_cnm1[2][3]**2)}"/>
     <link name="${prefix}_camera_center">

Commit message: Fix camera point cloud FoV

File: src/sirius_description/urdf/cameras/oak-d-w.urdf.xacro (robot description, xacro)
@@ -2,9 +2,9 @@
 <robot xmlns:xacro="http://ros.org/wiki/xacro">
   <xacro:macro name="oak-d-w" params="prefix:=oak-d-w package:=^ cameras:=^ cameras_inertial:=^ stereo_fps:=^|30 imu_frequency:=^|200 datum:=^ elevation:=^ year:=^ calibration:=^|${xacro.load_yaml('$(find sirius_cameras)/config/oak_d_w/kalibr_imucam_chain.yaml')}">
-    <xacro:property name="optical_offset_x" value="-0.01" />
+<xacro:property name="optical_offset_x" value="-0.01" />
     <xacro:property name="baseline" value="${sqrt(calibration.cam1.T_cn_cnm1[0][3]**2 + calibration.cam1.T_cn_cnm1[1][3]**2 + calibration.cam1.T_cn_cnm1[2][3]**2)}"/>
     <link name="${prefix}_camera_center">
       <visual>
-      <material name="oak-d-w-material">
+<material name="oak-d-w-material">
             <color rgba="0.35 0.35 0.35 1"/>
       </material>
@@ -69,4 +69,5 @@
         <camera name="/${prefix}_camera/left">
           <pose>0 ${baseline/2} 0 0 0 0</pose>
+          <horizontal_fov>${2*atan2(calibration.cam0.resolution[0], calibration.cam0.intrinsics[0] + calibration.cam0.intrinsics[1])}</horizontal_fov>
           <image>
             <width>${calibration.cam0.resolution[0]}</width>
@@ -96,4 +97,5 @@
         <camera name="/${prefix}_camera/right">
           <pose>0 -${baseline/2} 0 0 0 0</pose>
+          <horizontal_fov>${2*atan2(calibration.cam0.resolution[0], calibration.cam0.intrinsics[0] + calibration.cam0.intrinsics[1])}</horizontal_fov>
           <image>
             <width>${calibration.cam0.resolution[0]}</width>
@@ -141,4 +143,5 @@
         <visualize>false</visualize>
         <camera name="/${prefix}_camera/depth">
+          <horizontal_fov>${2*atan2(calibration.cam0.resolution[0], calibration.cam0.intrinsics[0] + calibration.cam0.intrinsics[1])}</horizontal_fov>
           <image>
             <width>${calibration.cam0.resolution[0]}</width>
