Commit message: Add pole to marker boxes

File: src/marker_description/urdf/marker1.urdf.xacro (robot description, xacro)
@@ -3,5 +3,13 @@
   <xacro:property name="package" value="marker_description" />
   <xacro:property name="params" value="${xacro.load_yaml('marker.yaml')}" />
-  <xacro:include filename="marker.urdf.xacro" />
-  <xacro:marker size='${params["marker_size"]}' margin='${params["margin"]}' name='marker'/>
+  <xacro:include filename="macros/marker.urdf.xacro" />
+  <xacro:include filename="macros/pole.urdf.xacro" />
+  <xacro:marker size='${params["marker_size"]}' margin='${params["margin"]}' name='marker_box'/>
+  <xacro:pole height='${params["pole_height"]}' radius='${params["pole_radius"]}' name='marker'/>
+  <joint name="marker_pole_joint" type="fixed">
+    <parent link="marker"/>
+    <child link="marker_box"/>
+    <origin xyz="0 0 ${params['pole_height'] + params['marker_size']/2 + params['margin']}" rpy="0 0 0"/>
+    <axis xyz="0 0 0"/>
+  </joint>
 </robot>

File: src/marker_description/urdf/marker2.urdf.xacro (robot description, xacro)
@@ -3,11 +3,13 @@
   <xacro:property name="package" value="marker_description" />
   <xacro:property name="params" value="${xacro.load_yaml('marker.yaml')}" />
-  <xacro:include filename="marker.urdf.xacro" />
-  <link name="marker">
+  <xacro:include filename="macros/marker.urdf.xacro" />
+  <xacro:include filename="macros/pole.urdf.xacro" />
+  <link name="marker_box">
   </link>
   <xacro:marker size='${params["marker_size"]}' margin='${params["margin"]}' name='marker_front'/>
   <xacro:marker size='${params["marker_size"]}' margin='${params["margin"]}' name='marker_back'/>
+  <xacro:pole height='${params["pole_height"]}' radius='${params["pole_radius"]}' name='marker'/>
   <joint name="margin_front_joint" type="fixed">
-    <parent link="marker"/>
+    <parent link="marker_box"/>
     <child link="marker_front"/>
     <origin xyz="0 0 0" rpy="0 0 0"/>
@@ -15,8 +17,14 @@
   </joint>
   <joint name="margin_back_joint" type="fixed">
-    <parent link="marker"/>
+    <parent link="marker_box"/>
     <child link="marker_back"/>
     <origin xyz="0 0 0" rpy="0 0 ${pi}"/>
     <axis xyz="0 0 0"/>
   </joint>
+  <joint name="marker_pole_joint" type="fixed">
+    <parent link="marker"/>
+    <child link="marker_box"/>
+    <origin xyz="0 0 ${params['pole_height'] + params['marker_size']/2 + params['margin']}" rpy="0 0 0"/>
+    <axis xyz="0 0 0"/>
+  </joint>
 </robot>

File: src/marker_description/urdf/marker3.urdf.xacro (robot description, xacro)
@@ -3,14 +3,16 @@
   <xacro:property name="package" value="marker_description" />
   <xacro:property name="params" value="${xacro.load_yaml('marker.yaml')}" />
-  <xacro:include filename="marker.urdf.xacro" />
+  <xacro:include filename="macros/marker.urdf.xacro" />
+  <xacro:include filename="macros/pole.urdf.xacro" />
   <xacro:property name="width" value="${params['marker_size'] + params['margin']*2}" />
   <xacro:property name="radius" value="${width * sqrt(3) / 6}" />
-  <link name="marker">
+  <link name="marker_box">
   </link>
   <xacro:marker size='${params["marker_size"]}' margin='${params["margin"]}' name='marker_front'/>
   <xacro:marker size='${params["marker_size"]}' margin='${params["margin"]}' name='marker_left'/>
   <xacro:marker size='${params["marker_size"]}' margin='${params["margin"]}' name='marker_right'/>
+  <xacro:pole height='${params["pole_height"]}' radius='${params["pole_radius"]}' name='marker'/>
   <joint name="margin_front_joint" type="fixed">
-    <parent link="marker"/>
+    <parent link="marker_box"/>
     <child link="marker_front"/>
     <origin xyz="${radius} 0 0" rpy="0 0 0"/>
@@ -18,5 +20,5 @@
   </joint>
   <joint name="margin_left_joint" type="fixed">
-    <parent link="marker"/>
+    <parent link="marker_box"/>
     <child link="marker_left"/>
     <origin xyz="-${radius * 0.5} ${width / 4} 0" rpy="0 0 ${pi*2/3}"/>
@@ -24,8 +26,14 @@
   </joint>
   <joint name="margin_right_joint" type="fixed">
-    <parent link="marker"/>
+    <parent link="marker_box"/>
     <child link="marker_right"/>
     <origin xyz="-${radius * 0.5} -${width / 4} 0" rpy="0 0 ${-pi*2/3}"/>
     <axis xyz="0 0 0"/>
   </joint>
+  <joint name="marker_pole_joint" type="fixed">
+    <parent link="marker"/>
+    <child link="marker_box"/>
+    <origin xyz="0 0 ${params['pole_height'] + params['marker_size']/2 + params['margin']}" rpy="0 0 0"/>
+    <axis xyz="0 0 0"/>
+  </joint>
 </robot>

File: src/marker_description/urdf/marker4.urdf.xacro (robot description, xacro)
@@ -3,6 +3,7 @@
   <xacro:property name="package" value="marker_description" />
   <xacro:property name="params" value="${xacro.load_yaml('marker.yaml')}" />
-  <xacro:include filename="marker.urdf.xacro" />
-  <link name="marker">
+  <xacro:include filename="macros/marker.urdf.xacro" />
+  <xacro:include filename="macros/pole.urdf.xacro" />
+  <link name="marker_box">
   </link>
   <xacro:marker size='${params["marker_size"]}' margin='${params["margin"]}' name='marker_front'/>
@@ -10,6 +11,7 @@
   <xacro:marker size='${params["marker_size"]}' margin='${params["margin"]}' name='marker_back'/>
   <xacro:marker size='${params["marker_size"]}' margin='${params["margin"]}' name='marker_right'/>
+  <xacro:pole height='${params["pole_height"]}' radius='${params["pole_radius"]}' name='marker'/>
   <joint name="margin_front_joint" type="fixed">
-    <parent link="marker"/>
+    <parent link="marker_box"/>
     <child link="marker_front"/>
     <origin xyz="${params['marker_size']/2 + params['margin']} 0 0" rpy="0 0 0"/>
@@ -17,5 +19,5 @@
   </joint>
   <joint name="margin_left_joint" type="fixed">
-    <parent link="marker"/>
+    <parent link="marker_box"/>
     <child link="marker_left"/>
     <origin xyz="0 ${params['marker_size']/2 + params['margin']} 0" rpy="0 0 ${pi/2}"/>
@@ -23,5 +25,5 @@
   </joint>
   <joint name="margin_back_joint" type="fixed">
-    <parent link="marker"/>
+    <parent link="marker_box"/>
     <child link="marker_back"/>
     <origin xyz="-${params['marker_size']/2 + params['margin']} 0 0" rpy="0 0 ${pi}"/>
@@ -29,8 +31,14 @@
   </joint>
   <joint name="margin_right_joint" type="fixed">
-    <parent link="marker"/>
+    <parent link="marker_box"/>
     <child link="marker_right"/>
     <origin xyz="0 -${params['marker_size']/2 + params['margin']} 0" rpy="0 0 ${-pi/2}"/>
     <axis xyz="0 0 0"/>
   </joint>
+  <joint name="marker_pole_joint" type="fixed">
+    <parent link="marker"/>
+    <child link="marker_box"/>
+    <origin xyz="0 0 ${params['pole_height'] + params['marker_size']/2 + params['margin']}" rpy="0 0 0"/>
+    <axis xyz="0 0 0"/>
+  </joint>
 </robot>
