Commit message: Add artags

File: src/marker_description/urdf/macros/marker.urdf.xacro (robot description, xacro)
@@ -1,4 +1,4 @@
 <robot xmlns:xacro="http://wiki.ros.org/xacro">
-<xacro:macro name="marker" params="size:=0.4 margin:=0.2 name:='marker' image:='marker'">
+<xacro:macro name="marker" params="size:=0.4 margin:=0.2 name:='marker' image:='artag_0'">
   <link name="${name}">
     <visual>

Commit message: Set xacro params with args

File: src/marker_description/urdf/macros/marker.urdf.xacro (robot description, xacro)
@@ -1,8 +1,9 @@
 <robot xmlns:xacro="http://wiki.ros.org/xacro">
-<xacro:macro name="marker" params="size:=0.4 margin:=0.2 name:='marker' image:='artag_0'">
+<xacro:macro name="marker" params="marker_size:=^0.15 margin:=^0.03 name:=^'marker' family:=^'artag' id:=^'0'">
+<xacro:property name="material" value="${family}_${id}" />
   <link name="${name}">
     <visual>
         <geometry>
-          <box size="0.0005 ${size + margin*2} ${size + margin*2}" />
+          <box size="0.0005 ${marker_size + margin*2} ${marker_size + margin*2}" />
         </geometry>
         <origin xyz="0.00025 0 0" rpy="0 0 0"/>
@@ -10,5 +11,5 @@
     <collision>
         <geometry>
-          <box size="0.0005 ${size + margin*2} ${size + margin*2}" />
+          <box size="0.0005 ${marker_size + margin*2} ${marker_size + margin*2}" />
         </geometry>
         <origin xyz="0.00025 0 0" rpy="0 0 0"/>
@@ -19,13 +20,13 @@
     </inertial>
   </link>
-  <link name="${name}_image">
+  <link name="${name}_material">
     <visual>
         <geometry>
-          <box size="0.0005 ${size} ${size}" />
+          <box size="0.0005 ${marker_size} ${marker_size}" />
         </geometry>
     </visual>
     <collision>
         <geometry>
-          <box size="0.0005 ${size} ${size}" />
+          <box size="0.0005 ${marker_size} ${marker_size}" />
         </geometry>
     </collision>
@@ -35,13 +36,13 @@
     </inertial>
   </link>
-  <joint name="${name}_image_joint" type="continuous">
+  <joint name="${name}_material_joint" type="continuous">
     <parent link="${name}"/>
-    <child link="${name}_image"/>
+    <child link="${name}_material"/>
     <origin xyz="0.00075 0 0" rpy="0 0 0"/>
     <axis xyz="0 0 0"/>
     <limit effort="0" velocity="0"/>
   </joint>
-  <gazebo reference="${name}_image">
-    <material>${image}</material>
+  <gazebo reference="${name}_material">
+    <material>${material}</material>
   </gazebo>
   <gazebo reference="${name}">

File: src/marker_description/urdf/marker1.urdf.xacro (robot description, xacro)
@@ -2,13 +2,29 @@
 <robot xmlns:xacro="http://www.ros.org/wiki/xacro" name="marker">
   <xacro:property name="package" value="marker_description" />
-  <xacro:property name="params" value="${xacro.load_yaml('marker.yaml')}" />
+  <xacro:arg name="name" default=""/>
+  <xacro:property name="name" value="$(arg name)" />
+  <xacro:arg name="family" default="artag"/>
+  <xacro:property name="family" value="$(arg family)" />
+  <xacro:arg name="id" default="0"/>
+  <xacro:property name="id" value="${$(arg id)}" />
+  <xacro:arg name="marker_size" default="0.15"/>
+  <xacro:property name="marker_size" value="${$(arg marker_size)}" />
+  <xacro:arg name="margin" default="0.03"/>
+  <xacro:property name="margin" value="${$(arg margin)}" />
+  <xacro:arg name="pole_height" default="0.417"/>
+  <xacro:property name="pole_height" value="${$(arg pole_height)}" />
+  <xacro:arg name="pole_radius" default="0.005"/>
+  <xacro:property name="pole_radius" value="${$(arg pole_radius)}" />
+  <xacro:if value="${name == ''}">
+    <xacro:property name="name" value="${family}_${id}" />
+  </xacro:if>
   <xacro:include filename="macros/marker.urdf.xacro" />
   <xacro:include filename="macros/pole.urdf.xacro" />
-  <xacro:marker size='${params["marker_size"]}' margin='${params["margin"]}' name='marker_box'/>
-  <xacro:pole height='${params["pole_height"]}' radius='${params["pole_radius"]}' name='marker'/>
-  <joint name="marker_pole_joint" type="fixed">
-    <parent link="marker"/>
-    <child link="marker_box"/>
-    <origin xyz="0 0 ${params['pole_height'] + params['marker_size']/2 + params['margin']}" rpy="0 0 0"/>
+  <xacro:marker name='${name}_box'/>
+  <xacro:pole height='${pole_height}' radius='${pole_radius}' name='${name}'/>
+  <joint name="${name}_pole_joint" type="fixed">
+    <parent link="${name}"/>
+    <child link="${name}_box"/>
+    <origin xyz="0 0 ${pole_height + marker_size/2 + margin}" rpy="0 0 0"/>
     <axis xyz="0 0 0"/>
   </joint>

File: src/marker_description/urdf/marker2.urdf.xacro (robot description, xacro)
@@ -2,28 +2,44 @@
 <robot xmlns:xacro="http://www.ros.org/wiki/xacro" name="marker">
   <xacro:property name="package" value="marker_description" />
-  <xacro:property name="params" value="${xacro.load_yaml('marker.yaml')}" />
+  <xacro:arg name="name" default=""/>
+  <xacro:property name="name" value="$(arg name)" />
+  <xacro:arg name="family" default="artag"/>
+  <xacro:property name="family" value="$(arg family)" />
+  <xacro:arg name="id" default="0"/>
+  <xacro:property name="id" value="${$(arg id)}" />
+  <xacro:arg name="marker_size" default="0.15"/>
+  <xacro:property name="marker_size" value="${$(arg marker_size)}" />
+  <xacro:arg name="margin" default="0.03"/>
+  <xacro:property name="margin" value="${$(arg margin)}" />
+  <xacro:arg name="pole_height" default="0.417"/>
+  <xacro:property name="pole_height" value="${$(arg pole_height)}" />
+  <xacro:arg name="pole_radius" default="0.005"/>
+  <xacro:property name="pole_radius" value="${$(arg pole_radius)}" />
+  <xacro:if value="${name == ''}">
+    <xacro:property name="name" value="${family}_${id}" />
+  </xacro:if>
   <xacro:include filename="macros/marker.urdf.xacro" />
   <xacro:include filename="macros/pole.urdf.xacro" />
-  <link name="marker_box">
+  <link name="${name}_box">
   </link>
-  <xacro:marker size='${params["marker_size"]}' margin='${params["margin"]}' name='marker_front'/>
-  <xacro:marker size='${params["marker_size"]}' margin='${params["margin"]}' name='marker_back'/>
-  <xacro:pole height='${params["pole_height"]}' radius='${params["pole_radius"]}' name='marker'/>
+  <xacro:marker name='${name}_front'/>
+  <xacro:marker name='${name}_back'/>
+  <xacro:pole height='${pole_height}' radius='${pole_radius}' name='${name}'/>
   <joint name="margin_front_joint" type="fixed">
-    <parent link="marker_box"/>
-    <child link="marker_front"/>
+    <parent link="${name}_box"/>
+    <child link="${name}_front"/>
     <origin xyz="0 0 0" rpy="0 0 0"/>
     <axis xyz="0 0 0"/>
   </joint>
   <joint name="margin_back_joint" type="fixed">
-    <parent link="marker_box"/>
-    <child link="marker_back"/>
+    <parent link="${name}_box"/>
+    <child link="${name}_back"/>
     <origin xyz="0 0 0" rpy="0 0 ${pi}"/>
     <axis xyz="0 0 0"/>
   </joint>
-  <joint name="marker_pole_joint" type="fixed">
-    <parent link="marker"/>
-    <child link="marker_box"/>
-    <origin xyz="0 0 ${params['pole_height'] + params['marker_size']/2 + params['margin']}" rpy="0 0 0"/>
+  <joint name="${name}_pole_joint" type="fixed">
+    <parent link="${name}"/>
+    <child link="${name}_box"/>
+    <origin xyz="0 0 ${pole_height + marker_size/2 + margin}" rpy="0 0 0"/>
     <axis xyz="0 0 0"/>
   </joint>

File: src/marker_description/urdf/marker3.urdf.xacro (robot description, xacro)
@@ -2,37 +2,53 @@
 <robot xmlns:xacro="http://www.ros.org/wiki/xacro" name="marker">
   <xacro:property name="package" value="marker_description" />
-  <xacro:property name="params" value="${xacro.load_yaml('marker.yaml')}" />
+  <xacro:arg name="name" default=""/>
+  <xacro:property name="name" value="$(arg name)" />
+  <xacro:arg name="family" default="artag"/>
+  <xacro:property name="family" value="$(arg family)" />
+  <xacro:arg name="id" default="0"/>
+  <xacro:property name="id" value="${$(arg id)}" />
+  <xacro:arg name="marker_size" default="0.15"/>
+  <xacro:property name="marker_size" value="${$(arg marker_size)}" />
+  <xacro:arg name="margin" default="0.03"/>
+  <xacro:property name="margin" value="${$(arg margin)}" />
+  <xacro:arg name="pole_height" default="0.417"/>
+  <xacro:property name="pole_height" value="${$(arg pole_height)}" />
+  <xacro:arg name="pole_radius" default="0.005"/>
+  <xacro:property name="pole_radius" value="${$(arg pole_radius)}" />
   <xacro:include filename="macros/marker.urdf.xacro" />
   <xacro:include filename="macros/pole.urdf.xacro" />
-  <xacro:property name="width" value="${params['marker_size'] + params['margin']*2}" />
+  <xacro:property name="width" value="${marker_size + margin*2}" />
   <xacro:property name="radius" value="${width * sqrt(3) / 6}" />
-  <link name="marker_box">
+  <xacro:if value="${name == ''}">
+    <xacro:property name="name" value="${family}_${id}" />
+  </xacro:if>
+  <link name="${name}_box">
   </link>
-  <xacro:marker size='${params["marker_size"]}' margin='${params["margin"]}' name='marker_front'/>
-  <xacro:marker size='${params["marker_size"]}' margin='${params["margin"]}' name='marker_left'/>
-  <xacro:marker size='${params["marker_size"]}' margin='${params["margin"]}' name='marker_right'/>
-  <xacro:pole height='${params["pole_height"]}' radius='${params["pole_radius"]}' name='marker'/>
+  <xacro:marker name='${name}_front'/>
+  <xacro:marker name='${name}_left'/>
+  <xacro:marker name='${name}_right'/>
+  <xacro:pole height='${pole_height}' radius='${pole_radius}' name='${name}'/>
   <joint name="margin_front_joint" type="fixed">
-    <parent link="marker_box"/>
-    <child link="marker_front"/>
+    <parent link="${name}_box"/>
+    <child link="${name}_front"/>
     <origin xyz="${radius} 0 0" rpy="0 0 0"/>
     <axis xyz="0 0 0"/>
   </joint>
   <joint name="margin_left_joint" type="fixed">
-    <parent link="marker_box"/>
-    <child link="marker_left"/>
+    <parent link="${name}_box"/>
+    <child link="${name}_left"/>
     <origin xyz="-${radius * 0.5} ${width / 4} 0" rpy="0 0 ${pi*2/3}"/>
     <axis xyz="0 0 0"/>
   </joint>
   <joint name="margin_right_joint" type="fixed">
-    <parent link="marker_box"/>
-    <child link="marker_right"/>
+    <parent link="${name}_box"/>
+    <child link="${name}_right"/>
     <origin xyz="-${radius * 0.5} -${width / 4} 0" rpy="0 0 ${-pi*2/3}"/>
     <axis xyz="0 0 0"/>
   </joint>
-  <joint name="marker_pole_joint" type="fixed">
-    <parent link="marker"/>
-    <child link="marker_box"/>
-    <origin xyz="0 0 ${params['pole_height'] + params['marker_size']/2 + params['margin']}" rpy="0 0 0"/>
+  <joint name="${name}_pole_joint" type="fixed">
+    <parent link="${name}"/>
+    <child link="${name}_box"/>
+    <origin xyz="0 0 ${pole_height + marker_size/2 + margin}" rpy="0 0 0"/>
     <axis xyz="0 0 0"/>
   </joint>

File: src/marker_description/urdf/marker4.urdf.xacro (robot description, xacro)
@@ -2,42 +2,58 @@
 <robot xmlns:xacro="http://www.ros.org/wiki/xacro" name="marker">
   <xacro:property name="package" value="marker_description" />
-  <xacro:property name="params" value="${xacro.load_yaml('marker.yaml')}" />
+  <xacro:arg name="name" default=""/>
+  <xacro:property name="name" value="$(arg name)" />
+  <xacro:arg name="family" default="artag"/>
+  <xacro:property name="family" value="$(arg family)" />
+  <xacro:arg name="id" default="0"/>
+  <xacro:property name="id" value="${$(arg id)}" />
+  <xacro:arg name="marker_size" default="0.15"/>
+  <xacro:property name="marker_size" value="${$(arg marker_size)}" />
+  <xacro:arg name="margin" default="0.03"/>
+  <xacro:property name="margin" value="${$(arg margin)}" />
+  <xacro:arg name="pole_height" default="0.417"/>
+  <xacro:property name="pole_height" value="${$(arg pole_height)}" />
+  <xacro:arg name="pole_radius" default="0.005"/>
+  <xacro:property name="pole_radius" value="${$(arg pole_radius)}" />
+  <xacro:if value="${name == ''}">
+    <xacro:property name="name" value="${family}_${id}" />
+  </xacro:if>
   <xacro:include filename="macros/marker.urdf.xacro" />
   <xacro:include filename="macros/pole.urdf.xacro" />
-  <link name="marker_box">
+  <link name="${name}_box">
   </link>
-  <xacro:marker size='${params["marker_size"]}' margin='${params["margin"]}' name='marker_front'/>
-  <xacro:marker size='${params["marker_size"]}' margin='${params["margin"]}' name='marker_left'/>
-  <xacro:marker size='${params["marker_size"]}' margin='${params["margin"]}' name='marker_back'/>
-  <xacro:marker size='${params["marker_size"]}' margin='${params["margin"]}' name='marker_right'/>
-  <xacro:pole height='${params["pole_height"]}' radius='${params["pole_radius"]}' name='marker'/>
+  <xacro:marker name='${name}_front'/>
+  <xacro:marker name='${name}_left'/>
+  <xacro:marker name='${name}_back'/>
+  <xacro:marker name='${name}_right'/>
+  <xacro:pole height='${pole_height}' radius='${pole_radius}' name='${name}'/>
   <joint name="margin_front_joint" type="fixed">
-    <parent link="marker_box"/>
-    <child link="marker_front"/>
-    <origin xyz="${params['marker_size']/2 + params['margin']} 0 0" rpy="0 0 0"/>
+    <parent link="${name}_box"/>
+    <child link="${name}_front"/>
+    <origin xyz="${marker_size/2 + margin} 0 0" rpy="0 0 0"/>
     <axis xyz="0 0 0"/>
   </joint>
   <joint name="margin_left_joint" type="fixed">
-    <parent link="marker_box"/>
-    <child link="marker_left"/>
-    <origin xyz="0 ${params['marker_size']/2 + params['margin']} 0" rpy="0 0 ${pi/2}"/>
+    <parent link="${name}_box"/>
+    <child link="${name}_left"/>
+    <origin xyz="0 ${marker_size/2 + margin} 0" rpy="0 0 ${pi/2}"/>
     <axis xyz="0 0 0"/>
   </joint>
   <joint name="margin_back_joint" type="fixed">
-    <parent link="marker_box"/>
-    <child link="marker_back"/>
-    <origin xyz="-${params['marker_size']/2 + params['margin']} 0 0" rpy="0 0 ${pi}"/>
+    <parent link="${name}_box"/>
+    <child link="${name}_back"/>
+    <origin xyz="-${marker_size/2 + margin} 0 0" rpy="0 0 ${pi}"/>
     <axis xyz="0 0 0"/>
   </joint>
   <joint name="margin_right_joint" type="fixed">
-    <parent link="marker_box"/>
-    <child link="marker_right"/>
-    <origin xyz="0 -${params['marker_size']/2 + params['margin']} 0" rpy="0 0 ${-pi/2}"/>
+    <parent link="${name}_box"/>
+    <child link="${name}_right"/>
+    <origin xyz="0 -${marker_size/2 + margin} 0" rpy="0 0 ${-pi/2}"/>
     <axis xyz="0 0 0"/>
   </joint>
-  <joint name="marker_pole_joint" type="fixed">
-    <parent link="marker"/>
-    <child link="marker_box"/>
-    <origin xyz="0 0 ${params['pole_height'] + params['marker_size']/2 + params['margin']}" rpy="0 0 0"/>
+  <joint name="${name}_pole_joint" type="fixed">
+    <parent link="${name}"/>
+    <child link="${name}_box"/>
+    <origin xyz="0 0 ${pole_height + marker_size/2 + margin}" rpy="0 0 0"/>
     <axis xyz="0 0 0"/>
   </joint>
