Commit message: Create package documentation

File: src/marker_description/urdf/macros/pole.urdf.xacro (robot description, xacro)
@@ -2,20 +2,22 @@
 <xacro:macro name="pole" params="height:=0.417 radius:=0.005 name:='marker'">
   <link name="${name}">
-    <visual>
+    <xacro:if value="${height != 0}">
+      <visual>
         <geometry>
           <cylinder length="${height}" radius="${radius}" />
         </geometry>
         <origin xyz="0 0 ${height/2}" rpy="0 0 0"/>
-    </visual>
-    <collision>
+      </visual>
+      <collision>
         <geometry>
           <cylinder length="${height}" radius="${radius}" />
         </geometry>
         <origin xyz="0 0 ${height/2}" rpy="0 0 0"/>
-    </collision>
-    <inertial>
-      <mass value="1.0" />
-      <inertia  ixx="1.0" ixy="0.0"  ixz="0.0"  iyy="1.0"  iyz="0.0"  izz="1.0" />
-    </inertial>
+      </collision>
+      <inertial>
+        <mass value="1.0" />
+        <inertia  ixx="1.0" ixy="0.0"  ixz="0.0"  iyy="1.0"  iyz="0.0"  izz="1.0" />
+      </inertial>
+    </xacro:if>
   </link>
   <gazebo reference="${name}">

File: src/marker_description/urdf/marker.urdf.xacro (robot description, xacro)
@@ -1,5 +1,5 @@
 <?xml version="1.0" encoding="utf-8"?>
 <robot xmlns:xacro="http://www.ros.org/wiki/xacro" name="marker">
-  <xacro:arg name="sides" default="4"/>
+  <xacro:arg name="sides" default="1"/>
   <xacro:if value="${$(arg sides) == 1}">
     <xacro:include filename="marker1.urdf.xacro"></xacro:include>
